File: hardware/voice.kicad_pcb (KiCad board)
At the start: 2 copper layers, 111.8 x 50.8 mm, 56 parts, among them K1 PWR, P1 DATA, P2 OUT, U1 4051, U2 MCP4922-E/P, U3 MCP4922-E/P, U4 TL074, U5 SSM2044, U6 SSM2044

Commit message: hardware project cleanup
Parts:
- C1, C2, C3, C4: value CP1 -> 10u; footprint C1.5V8V -> C1V5
- C21, C22: footprint C1.5V8V -> C1V5
- R1, R2, R3, R4, R5, R6, R8: footprint R4-LARGE_PADS -> R1
- R10, R9: value 68k -> 6k8; footprint R4-LARGE_PADS -> R1
- R11, R12, R13, R14: footprint R4-LARGE_PADS -> R3-LARGE_PADS
- R15, R16: value 2k2 -> 3k3; footprint R4-LARGE_PADS -> R3-LARGE_PADS
- R17, R18: value 18k -> 47k; footprint R4-LARGE_PADS -> R3-LARGE_PADS
- R7: footprint R3-LARGE_PADS -> R1
- moved C1 62.9 mm to (97.2, 69.2)
- moved C6 58.8 mm to (47.0, 27.3), turned to 90 degrees
- moved C5 55.3 mm to (49.5, 27.3), turned to 90 degrees
- moved U2 55.2 mm to (87.0, 59.7), turned to 180 degrees
- moved R2 55.1 mm to (102.2, 63.5), turned to 0 degrees
- moved R1 54.6 mm to (102.2, 66.7), turned to 0 degrees
- moved C2 52.0 mm to (91.4, 69.2)
- moved C10 49.1 mm to (52.1, 27.3), turned to 90 degrees
- moved C24 49.0 mm to (137.2, 24.1), turned to 0 degrees
- moved C8 47.8 mm to (59.7, 27.3), turned to 90 degrees
- moved C7 46.6 mm to (69.8, 27.3), turned to 90 degrees
- moved C9 44.5 mm to (54.6, 27.3), turned to 90 degrees
- moved C11 42.8 mm to (62.2, 27.3), turned to 90 degrees
- moved C12 42.8 mm to (64.8, 27.3), turned to 90 degrees
- moved C3 39.9 mm to (88.9, 40.6)
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Connections:
- P1 pad 1: //LDAC_A -> N-0000041
- P1 pad 10: N-0000035 -> //LDAC_A
- P1 pad 2: //LDAC_B -> N-0000043
- P1 pad 3: /SDI -> N-0000050
- P1 pad 4: /SCK -> N-0000034
- P1 pad 5: //CS -> N-0000042
- P1 pad 6: N-0000043 -> //CS
- P1 pad 7: N-0000036 -> /SCK
- P1 pad 8: N-0000050 -> /SDI
- P1 pad 9: N-0000032 -> //LDAC_B
- U1 pad 10: N-0000036 -> N-0000043
- U1 pad 3: N-0000032 -> N-0000034
- U1 pad 6: N-0000035 -> N-0000042
- U1 pad 9: N-0000043 -> N-0000041
- U4 pad 1: N-0000015 -> N-0000045
- U4 pad 12: N-0000060 -> N-0000061
- U4 pad 13: N-0000045 -> N-0000015
- U4 pad 14: N-0000045 -> N-0000015
- U4 pad 2: N-0000015 -> N-0000045
- U4 pad 3: N-0000061 -> N-0000060
Routing:
- net +5V: track 69.5 -> 247.4 mm, vias 0 -> 1
- net -5V: track 54.5 -> 207.7 mm
- net GND: track 126.2 -> 268.5 mm, vias 0 -> 1
- net N-0000063: track 0.00 -> 99.8 mm, vias 0 -> 2
- net N-0000015: track 0.00 -> 83.7 mm
- net N-0000065: track 0.00 -> 76.2 mm, vias 0 -> 1
- net N-0000060: track 0.00 -> 75.2 mm
- net N-0000064: track 0.00 -> 70.7 mm
- net /SCK: track 0.00 -> 63.0 mm
- net //CS: track 0.00 -> 61.4 mm, vias 0 -> 2
- net N-0000046: track 12.0 -> 72.5 mm
- net N-0000061: track 0.00 -> 55.6 mm
- net N-0000048: track 0.00 -> 54.1 mm
- net N-0000062: track 0.00 -> 53.8 mm, vias 0 -> 1
- net N-0000056: track 0.00 -> 49.0 mm
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Other:
- board size 111.8 x 50.8 mm -> 99.1 x 50.8 mm
- net class Default: clearance 0.762 -> 0.508; via_dia 2.54 -> 2.032
- net class pwr added: clearance 0.508, trace_width 1.27, via_dia 2.032, via_drill 0.508
- rule trace_clearance: 0.762 -> 0.508

Commit message: hardware updates
Parts:
- R1, R2, R3, R4: footprint R1 -> R3-LARGE_PADS
- R17, R18: value 47k -> 18k
- moved C3 5.30 mm to (83.8, 42.2)
- moved R4 4.95 mm to (91.9, 47.0)
- moved R3 3.07 mm to (91.9, 42.2)
- moved R2 2.33 mm to (100.2, 62.4), turned to 90 degrees
- moved R1 1.63 mm to (103.3, 65.4), turned to 90 degrees
Routing:
- net +5V: track 247.4 -> 273.6 mm
- net N-0000046: track 72.5 -> 64.4 mm
- net N-0000017: track 16.5 -> 11.5 mm
- net N-0000048: track 54.1 -> 58.0 mm
- net /SCK: track 63.0 -> 65.5 mm
- net N-0000034: track 20.8 -> 23.2 mm, vias 1 -> 2
- net N-0000019: track 3.17 -> 5.59 mm
- net -5V: track 207.7 -> 210.1 mm
- net (no net): track 0.00 -> 1.93 mm
- net N-0000022: track 10.7 -> 9.20 mm
- net //LDAC_A: track 13.2 -> 14.4 mm, vias 0 -> 1
- net N-0000021: track 3.59 -> 4.83 mm
- net N-0000010: track 5.05 -> 4.23 mm
- net N-000007: track 5.05 -> 4.23 mm
- net N-0000029: track 5.05 -> 4.23 mm
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Other:
- board text added: "2VoiceCard R6"

Commit message: sch: VCFs output resistors change to drive the VCAs harder
Parts:
- R15, R16: value 3k3 -> 8k2
Changed lines of the file:
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@@
       (effects (font (size 1.397 1.27) (thickness 0.2032)))
     )
-    (fp_text value 3k3 (at 0 0 270) (layer F.SilkS) hide
+    (fp_text value 8k2 (at 0 0 270) (layer F.SilkS) hide
       (effects (font (size 1.397 1.27) (thickness 0.2032)))
     )
@@
       (effects (font (size 1.397 1.27) (thickness 0.2032)))
     )
-    (fp_text value 3k3 (at 0 0 270) (layer F.SilkS) hide
+    (fp_text value 8k2 (at 0 0 270) (layer F.SilkS) hide
       (effects (font (size 1.397 1.27) (thickness 0.2032)))
     )
