File: hardware/voice.sch (KiCad schematic (older format))
At the start: 56 parts, among them K1 PWR, P1 DATA, P2 OUT, U1 4051, U2 MCP4922-E/P, U3 MCP4922-E/P, U4 TL074, U5 SSM2044, U6 SSM2044

Commit message: hardware updates
Parts:
- R17, R18: value 47k -> 18k
Changed lines of the file:
@@
 LIBS:contrib
 LIBS:valves
-LIBS:LPC-H1248-EXT1
-LIBS:LPC-H1248-EXT2
-LIBS:SSM2044
-LIBS:SSM2164
 LIBS:voice-cache
 EELAYER 27 0
@@
 Sheet 1 1
 Title "Overcycler voice board schematics"
-Date "15 aug 2013"
+Date "24 aug 2013"
 Rev "1"
 Comp "GliGli's DIY"
@@
 P 9400 3750
 F 0 "R17" V 9480 3750 40  0000 C CNN
-F 1 "47k" V 9407 3751 40  0000 C CNN
+F 1 "18k" V 9407 3751 40  0000 C CNN
 F 2 "~" V 9330 3750 30  0000 C CNN
 F 3 "~" H 9400 3750 30  0000 C CNN
@@
 P 9400 5550
 F 0 "R18" V 9480 5550 40  0000 C CNN
-F 1 "47k" V 9407 5551 40  0000 C CNN
+F 1 "18k" V 9407 5551 40  0000 C CNN
 F 2 "~" V 9330 5550 30  0000 C CNN
 F 3 "~" H 9400 5550 30  0000 C CNN

Commit message: small schematics cleanups / TODO: main/vca board need fixes
Parts:
- R5, R6: Reference R -> (none); Value 220 -> (none)
Changed lines of the file:
@@
 Sheet 1 1
 Title "Overcycler voice board schematics"
-Date "24 aug 2013"
+Date "1 oct 2013"
 Rev "1"
 Comp "GliGli's DIY"
@@
 U 1 1 5208A0F1
 P 4800 3000
-F 0 "R5" V 4850 3050 60  0000 C CNN
-F 1 "220" H 4800 3000 60  0001 C CNN
+F 0 "R5" V 4900 3000 60  0000 C CNN
+F 1 "220" V 4800 3000 60  0000 C CNN
 F 2 "" H 4800 3000 60  0001 C CNN
 F 3 "" H 4800 3000 60  0001 C CNN
-F 4 "R" V 4880 3000 40  0000 C CNN "Reference"
-F 5 "220" V 4807 3001 40  0000 C CNN "Value"
+F 4 "~" V 4880 3000 40  0000 C CNN "Reference"
+F 5 "~" V 4807 3001 40  0000 C CNN "Value"
 F 6 "~" V 4730 3000 30  0000 C CNN "Footprint"
 F 7 "~" H 4800 3000 30  0000 C CNN "Datasheet"
@@
 U 1 1 5208A0FB
 P 4800 4300
-F 0 "R6" V 4850 4350 60  0000 C CNN
-F 1 "220" H 4800 4300 60  0001 C CNN
+F 0 "R6" V 4700 4300 60  0000 C CNN
+F 1 "220" V 4800 4300 60  0000 C CNN
 F 2 "" H 4800 4300 60  0001 C CNN
 F 3 "" H 4800 4300 60  0001 C CNN
-F 4 "R" V 4880 4300 40  0000 C CNN "Reference"
-F 5 "220" V 4807 4301 40  0000 C CNN "Value"
+F 4 "~" V 4900 4300 40  0000 C CNN "Reference"
+F 5 "~" V 4807 4301 40  0000 C CNN "Value"
 F 6 "~" V 4730 4300 30  0000 C CNN "Footprint"
 F 7 "~" H 4800 4300 30  0000 C CNN "Datasheet"

Commit message: sch: VCFs output resistors change to drive the VCAs harder
Parts:
- R15, R16: value 3k3 -> 8k2
Changed lines of the file:
@@
 Sheet 1 1
 Title "Overcycler voice board schematics"
-Date "1 oct 2013"
+Date "29 may 2014"
 Rev "1"
 Comp "GliGli's DIY"
@@
 P 9350 2850
 F 0 "R15" V 9430 2850 40  0000 C CNN
-F 1 "3k3" V 9357 2851 40  0000 C CNN
+F 1 "8k2" V 9357 2851 40  0000 C CNN
 F 2 "~" V 9280 2850 30  0000 C CNN
 F 3 "~" H 9350 2850 30  0000 C CNN
@@
 P 9350 4650
 F 0 "R16" V 9430 4650 40  0000 C CNN
-F 1 "3k3" V 9357 4651 40  0000 C CNN
+F 1 "8k2" V 9357 4651 40  0000 C CNN
 F 2 "~" V 9280 4650 30  0000 C CNN
 F 3 "~" H 9350 4650 30  0000 C CNN
