File: hardware/overcycler.sch (KiCad schematic (older format))
At the start: 24 parts

Commit message: mainboard schema WIP
Parts:
- removed D?: 1N5819, ~, symbol DIODESCH
- removed J? (x5): JACK_2P, ~, symbol JACK_2P
- removed P?: DIN_5, symbol DIN_5
- removed U?: SSM2164, MODULE, symbol SSM2164
- removed U?: LPC-H1248-EXT1, MODULE, symbol LPC-H1248-EXT1
- removed U?: LPC-H1248-EXT2, MODULE, symbol LPC-H1248-EXT2
- removed U?: 4051, symbol 4051
- removed U?: 7805, ~, symbol 7805
- removed U?: 7905, ~, symbol 7905
- added C?: 2.2u, ~, symbol CP1
- added P?: LPC_P1, symbol CONN_33
- added P?: LPC_P2, symbol CONN_33
- added P?: FT232, symbol CONN_6
- added P?: SDCARD, symbol CONN_7
- added P?: CARD0_CMD_PWR, symbol CONN_14
- added P?: VOICE_OUT, symbol CONN_2
- added P?: MIDI_IN, symbol CONN_2
- added P?: SCREEN, symbol CONN_5
- added P?: TEN_POTS, symbol CONN_12
- added P?: CARD1_CMD_PWR, symbol CONN_14
- added P?: CARD2_CMD_PWR, symbol CONN_14
- added P?: VCA_CMD_PWR, symbol CONN_9
- added SW?: RESET, ~, symbol SW_PUSH
- added U?: LM1084IT-3.3/NOPB, TO-220, symbol LM1084IT-3.3/NOPB
- added U?: LM1084IT-5.0/NOPB, TO-220, symbol LM1084IT-5.0/NOPB
- added U?: LM2990-5.0/NOPB, TO-220, symbol LM7905CT
- added U? (x2): 4053, symbol 4053
- C?: value 2200u -> 3300u
Connections:
- net labels added: +3.3V
- net labels removed: +V_UNREG, VCC
- wire segments 27 -> 207
Other:
- moved on the sheet: U?A

Commit message: sch update
Parts:
- removed P?: VOICE_OUT, symbol CONN_2
- removed U? (x4): TL074, symbol TL074
- added C1, C2, C3, C9: 100n, ~, symbol C
- added D3: 1N5819, ~, symbol DIODESCH
- added OC1: 6N139, optocoupler-DIL08, symbol 6N139
- added P12: FOOT_IN, symbol CONN_2
- added R1: 33k, ~, symbol R
- added R2: 270, ~, symbol R
- added R3, R6: 4k7, ~, symbol R
- added R4: 100k, ~, symbol R
- added R5: 220, ~, symbol R
- added RV1: 10k, ~, symbol POT
- added U3: MCP4921-E/P, DIP8, symbol MCP4921-E/P
- C6, C8: renamed from C?; value 2.2u -> 6u8
- C7: renamed from C?; value 2.2u -> 4u7
- P1: renamed from P?; footprint (none) -> ~
- P11: renamed from P?; value CONN_2 -> AC_IN
- gave numbers to parts that had none: 20
Connections:
- net labels added: AC_IN, FOOT_IN, MIDI_IN, UNR+, UNR-
- wire segments 207 -> 298
Other:
- moved on the sheet: P13

Commit message: mainboard almost ok
Parts:
- removed P9: TEN_POTS, symbol CONN_12
- added P9: TEN_POTS, symbol CONN_6X2
Connections:
- wire segments 298 -> 310
Changed lines of the file:
@@
 Sheet 1 1
 Title "Overcycler main board schematics"
-Date "21 aug 2013"
+Date "22 aug 2013"
 Rev "1"
 Comp "GliGli's DIY"
@@
 $EndComp
 $Comp
-L CONN_12 P9
-U 1 1 521411A0
-P 5550 2600
-F 0 "P9" V 5500 2600 60  0000 C CNN
-F 1 "TEN_POTS" V 5600 2600 60  0000 C CNN
-F 2 "" H 5550 2600 60  0000 C CNN
-F 3 "" H 5550 2600 60  0000 C CNN
-	1    5550 2600
-	1    0    0    -1
-$EndComp
-$Comp
 L +3.3V #PWR014
 U 1 1 52142117
@@
 L GND #PWR016
 U 1 1 52153743
-P 6750 6900
-F 0 "#PWR016" H 6750 6900 30  0001 C CNN
-F 1 "GND" H 6750 6830 30  0001 C CNN
-F 2 "" H 6750 6900 60  0000 C CNN
-F 3 "" H 6750 6900 60  0000 C CNN
-	1    6750 6900
+P 7100 7000
+F 0 "#PWR016" H 7100 7000 30  0001 C CNN
+F 1 "GND" H 7100 6930 30  0001 C CNN
+F 2 "" H 7100 7000 60  0000 C CNN
+F 3 "" H 7100 7000 60  0000 C CNN
+	1    7100 7000
 	1    0    0    -1
 $EndComp
@@
 L -5V #PWR018
 U 1 1 52153759
-P 6950 6900
-F 0 "#PWR018" H 6950 7040 20  0001 C CNN
-F 1 "-5V" H 6950 7010 30  0000 C CNN
-F 2 "" H 6950 6900 60  0000 C CNN
-F 3 "" H 6950 6900 60  0000 C CNN
-	1    6950 6900
+P 6750 6900
+F 0 "#PWR018" H 6750 7040 20  0001 C CNN
+F 1 "-5V" H 6750 7010 30  0000 C CNN
+F 2 "" H 6750 6900 60  0000 C CNN
+F 3 "" H 6750 6900 60  0000 C CNN
+	1    6750 6900
 	1    0    0    -1
 $EndComp
@@
 	2900 3150 2900 3350
 Wire Wire Line
-	4400 3350 2900 3350
+	2900 3350 4400 3350
 Connection ~ 3650 3350
 Wire Wire Line
@@
 	4400 5100 2900 5100
 Wire Wire Line
-	2900 4400 2900 5100
+	2900 5100 2900 4400
 Wire Wire Line
 	2900 4900 2950 4900
@@
 	4400 4700 4350 4700
 Wire Wire Line
-	4400 1850 4400 3350
+	4400 3350 4400 1950
 Wire Wire Line
 	4400 2950 4350 2950
@@
 	4350 2650 5200 2650
 Wire Wire Line
-	4350 2750 5200 2750
+	4350 2750 6050 2750
 Wire Wire Line
 	4350 3800 4650 3800
@@
 	4650 3800 4650 2850
 Wire Wire Line
-	4650 2850 5200 2850
+	4650 2850 6150 2850
 Wire Wire Line
 	4350 3900 4750 3900
@@
 	4750 3900 4750 2950
 Wire Wire Line
-	4750 2950 5200 2950
+	4750 2950 6250 2950
 Wire Wire Line
 	4350 4100 4850 4100
@@
 	4850 4100 4850 3050
 Wire Wire Line
-	4850 3050 5200 3050
+	4850 3050 6350 3050
 Wire Wire Line
 	4350 4200 4950 4200
@@
 	4950 4200 4950 3150
 Wire Wire Line
-	4950 3150 5200 3150
-Wire Wire Line
-	4400 1850 5150 1850
-Wire Wire Line
-	5150 2050 5200 2050
+	4950 3150 6450 3150
 Connection ~ 4400 2950
-Wire Wire Line
-	5150 1850 5150 2050
 Wire Wire Line
 	5200 2150 5050 2150
@@
 	2950 7250 2950 7150
 Wire Wire Line
-	2950 7150 6950 7150
+	2950 7150 6750 7150
 Wire Wire Line
 	2850 7250 2850 7100
@@
 	1650 6250 1650 7250
 Wire Wire Line
-	6950 6900 6950 7250
-Wire Wire Line
-	6850 6850 6850 7250
-Wire Wire Line
 	4850 6900 4850 7250
 Wire Wire Line
@@
 Wire Wire Line
 	6650 6900 6650 7250
-Wire Wire Line
-	6750 7100 6750 7250
 Wire Wire Line
 	8350 6450 8450 6450
@@
 	8450 6850 8450 6550
 Wire Wire Line
-	6850 6850 6750 6850
-Wire Wire Line
-	6750 6850 6750 6900
-Connection ~ 6950 7150
-Wire Wire Line
 	1500 7250 1500 6650
 Wire Wire Line
@@
 	1400 7050 1400 6500
 Wire Wire Line
-	2850 7100 6850 7100
+	1600 7100 6950 7100
 Connection ~ 4350 7100
 Connection ~ 5850 7100
-Connection ~ 6750 7100
 Connection ~ 6850 7100
 Wire Wire Line
@@
 Text Label 8000 2150 3    60   ~ 0
 UNR-
+$Comp
+L CONN_6X2 P9
+U 1 1 52164F61
+P 5600 2400
+F 0 "P9" H 5600 2750 60  0000 C CNN
+F 1 "TEN_POTS" V 5600 2400 60  0000 C CNN
+F 2 "" H 5600 2400 60  0000 C CNN
+F 3 "" H 5600 2400 60  0000 C CNN
+	1    5600 2400
+	1    0    0    -1
+$EndComp
+Wire Wire Line
+	4400 1950 6050 1950
+Wire Wire Line
+	6050 1950 6050 2150
+Wire Wire Line
+	6050 2150 6000 2150
+Wire Wire Line
+	6050 2750 6050 2650
+Wire Wire Line
+	6050 2650 6000 2650
+Wire Wire Line
+	6150 2850 6150 2550
+Wire Wire Line
+	6150 2550 6000 2550
+Wire Wire Line
+	6250 2950 6250 2450
+Wire Wire Line
+	6250 2450 6000 2450
+Wire Wire Line
+	6350 3050 6350 2350
+Wire Wire Line
+	6350 2350 6000 2350
+Wire Wire Line
+	6450 3150 6450 2250
+Wire Wire Line
+	6450 2250 6000 2250
+Wire Wire Line
+	6750 6900 6750 7250
+Connection ~ 6750 7150
+Wire Wire Line
+	6850 7100 6850 7250
+Wire Wire Line
+	6950 6900 6950 7250
+Wire Wire Line
+	6950 6900 7100 6900
+Wire Wire Line
+	7100 6900 7100 7000
+Connection ~ 6950 7100
+Wire Wire Line
+	1050 6850 1600 6850
+Wire Wire Line
+	1600 6850 1600 7100
+Connection ~ 2850 7100
 $EndSCHEMATC

Commit message: mainboard ok
Connections:
- net GND: no longer P5.6 (P6)
Changed lines of the file:
@@
 Wire Wire Line
 	3400 1450 3400 1050
-Wire Wire Line
-	3500 1100 3500 1050
 Connection ~ 2650 1100
 Wire Wire Line
 	3200 1100 3200 1050
-Connection ~ 3200 1100
 Wire Wire Line
 	3300 1050 3300 1200
@@
 Wire Wire Line
 	4500 1100 4500 1050
-Connection ~ 3500 1100
 Wire Wire Line
 	4400 1050 4400 1100
-Connection ~ 4400 1100
 Wire Wire Line
 	4300 1050 4300 1200
@@
 	2900 3150 2900 3350
 Wire Wire Line
-	2900 3350 4400 3350
+	4400 3350 2900 3350
 Connection ~ 3650 3350
 Wire Wire Line
@@
 	4400 5100 2900 5100
 Wire Wire Line
-	2900 5100 2900 4400
+	2900 4400 2900 5100
 Wire Wire Line
 	2900 4900 2950 4900
@@
 	4400 4700 4350 4700
 Wire Wire Line
-	4400 3350 4400 1950
+	4400 1950 4400 3350
 Wire Wire Line
 	4400 2950 4350 2950
@@
 	4250 7050 4250 7250
 Wire Wire Line
-	4350 7250 4350 7100
+	4350 7100 4350 7250
 Wire Wire Line
 	1950 7250 1950 6950
@@
 	1600 6850 1600 7100
 Connection ~ 2850 7100
+Connection ~ 4400 1100
+Connection ~ 3200 1100
 $EndSCHEMATC

Commit message: schematics fixes
Connections:
- net at P4.6 (P6), P6.6 (P6), P8.6 (P6)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: now also P2.31 (P31); no longer P2.30 (P30)
- net at P4.7 (P7), P6.7 (P7), P8.7 (P7)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: now also P2.30 (P30); no longer P2.31 (P31)
Changed lines of the file:
@@
 Sheet 1 1
 Title "Overcycler main board schematics"
-Date "22 aug 2013"
-Rev "1"
+Date "24 sep 2013"
+Rev "2"
 Comp "GliGli's DIY"
-Comment1 "inverser sck/ssel"
-Comment2 "largeur lpc"
-Comment3 "espacement ports cards"
+Comment1 ""
+Comment2 ""
+Comment3 ""
 Comment4 ""
 $EndDescr
@@
 	1550 7450 1550 6700
 Wire Wire Line
-	1050 7250 1500 7250
-Wire Wire Line
-	1050 7150 1450 7150
+	1050 7250 1450 7250
 Wire Wire Line
 	1050 7050 1400 7050
@@
 	8450 6850 8450 6550
 Wire Wire Line
-	1500 7250 1500 6650
-Wire Wire Line
-	1450 7150 1450 6600
+	1500 7150 1500 6650
+Wire Wire Line
+	1450 7250 1450 6600
 Wire Wire Line
 	1400 7050 1400 6500
@@
 Connection ~ 4400 1100
 Connection ~ 3200 1100
+Wire Wire Line
+	1050 7150 1500 7150
 $EndSCHEMATC

Commit message: hw: fix for potmux noise
Connections:
- net +3.3V: now also U1.16 (VDD), U2.16 (VDD)
- net +5V: no longer U1.16 (VDD), U2.16 (VDD)
Changed lines of the file:
@@
 Sheet 1 1
 Title "Overcycler main board schematics"
-Date "24 sep 2013"
+Date "30 mar 2014"
 Rev "2"
 Comp "GliGli's DIY"
@@
 $EndComp
 $Comp
-L +5V #PWR012
-U 1 1 521401B5
-P 3650 1900
-F 0 "#PWR012" H 3650 1990 20  0001 C CNN
-F 1 "+5V" H 3650 1990 30  0000 C CNN
-F 2 "" H 3650 1900 60  0000 C CNN
-F 3 "" H 3650 1900 60  0000 C CNN
-	1    3650 1900
-	1    0    0    -1
-$EndComp
-$Comp
-L +5V #PWR013
-U 1 1 521401BB
-P 3650 3650
-F 0 "#PWR013" H 3650 3740 20  0001 C CNN
-F 1 "+5V" H 3650 3740 30  0000 C CNN
-F 2 "" H 3650 3650 60  0000 C CNN
-F 3 "" H 3650 3650 60  0000 C CNN
-	1    3650 3650
-	1    0    0    -1
-$EndComp
-$Comp
 L +3.3V #PWR014
 U 1 1 52142117
@@
 	2900 3150 2900 3350
 Wire Wire Line
-	4400 3350 2900 3350
+	2900 3350 4400 3350
 Connection ~ 3650 3350
 Wire Wire Line
@@
 	4400 5100 2900 5100
 Wire Wire Line
-	2900 4400 2900 5100
+	2900 5100 2900 4400
 Wire Wire Line
 	2900 4900 2950 4900
@@
 	4400 4700 4350 4700
 Wire Wire Line
-	4400 1950 4400 3350
+	4400 3350 4400 1950
 Wire Wire Line
 	4400 2950 4350 2950
@@
 	3650 3650 3650 3750
 Wire Wire Line
-	3650 1900 3650 2000
+	3650 1850 3650 2000
 Wire Wire Line
 	4500 5000 4350 5000
@@
 	5200 2150 5050 2150
 Wire Wire Line
-	5050 2150 5050 1750
+	5050 1750 5050 3650
 Wire Wire Line
 	2500 2650 1350 2650
@@
 Wire Wire Line
 	1050 7150 1500 7150
+Wire Wire Line
+	3650 1850 5050 1850
+Connection ~ 5050 1850
+Wire Wire Line
+	5050 3650 3650 3650
+Connection ~ 5050 2150
 $EndSCHEMATC

Commit message: sch: fix mainboard footswitch resistor value
Parts:
- R4: value 100k -> 10k
Changed lines of the file:
@@
 Sheet 1 1
 Title "Overcycler main board schematics"
-Date "30 mar 2014"
+Date "9 sep 2014"
 Rev "2"
 Comp "GliGli's DIY"
@@
 P 10300 5850
 F 0 "R4" V 10380 5850 40  0000 C CNN
-F 1 "100k" V 10307 5851 40  0000 C CNN
+F 1 "10k" V 10307 5851 40  0000 C CNN
 F 2 "~" V 10230 5850 30  0000 C CNN
 F 3 "~" H 10300 5850 30  0000 C CNN
