File: hardware/overcycler.sch (KiCad schematic (older format))
At the start: 40 parts, among them P1 LPC_P1, P10 VCA_CMD_PWR, P11 AC_IN, P12 FOOT_IN, P13 MIDI_IN, P2 LPC_P2, P3 FT232, P4 CARD0_CMD_PWR, P5 SDCARD, P6 CARD1_CMD_PWR, P7 SCREEN, P8 CARD2_CMD_PWR, P9 TEN_POTS, SW1 RESET, U1 4053, U2 4053, U3 MCP4921-E/P, U4 LM1084IT-5.0/NOPB, U5 LM2990-5.0/NOPB, U6 LM1084IT-3.3/NOPB

Commit message: hw: revised mainboard
Parts:
- added C10, C11: 100n, ~, symbol C
- added P14: VCA_SPI, symbol CONN_5
- C4: value 3300u -> 10000u
- C5: value 2200u -> 10000u
Connections:
- net +3.3V: now also C10.1, C11.1
- net GND: now also C10.2, C11.2
- net at P2.30 (P30), P4.7 (P7), P6.7 (P7)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: now also P14.2
- net at P2.31 (P31), P4.6 (P6), P6.6 (P6)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: now also P14.3
- net at P2.33 (P33), P4.8 (P8), P6.8 (P8)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: now also P14.1
- net at P4.4 (P4), P6.4 (P4), P8.4 (P4)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: no longer P10.4 (P4)
