File: hardware/vca.sch (KiCad schematic (older format))
At the start: 59 parts

Commit message: adding vca board schematics
Parts:
- removed C?: CP1, ~, symbol CP1
- removed C? (x2): 560p, ~, symbol C
- removed P?: CARD_0, symbol CONN_2
- removed R?: R, ~, symbol R
- removed R? (x10): 33k, ~, symbol R
- removed R? (x8): 3k3, ~, symbol R
- removed R? (x2): 470, ~, symbol R
- removed U? (x7): TL082, symbol TL082
- removed U? (x7): TL074, symbol TL074
- added C1, C19, C2, C20, C23, C24: 470p, ~, symbol C
- added C10, C11, C12, C29, C30, C31, C32, C9: 100p, ~, symbol C
- added C17, C18, C21, C22, C25, C26: 100n, ~, symbol C
- added C27, C28: 47u, ~, symbol CP1
- added P10: CARD_2, symbol CONN_2
- added P11: OUT_MAIN, symbol CONN_4
- added P12: OUT_GND, symbol CONN_3
- added P2: CARD_0, symbol CONN_2
- added P4: OUT_0, symbol CONN_2
- added P5: OUT_1, symbol CONN_2
- added P6: OUT_2, symbol CONN_2
- added P7: OUT_3, symbol CONN_2
- added P8: OUT_4, symbol CONN_2
- added P9: OUT_5, symbol CONN_2
- added R1, R13, R14, R15, R16, R3, R34, R35, R36, R37: 10k, ~, symbol R
- added R10, R30, R31, R32, R33, R9: 470, ~, symbol R
- added R17, R18, R20, R29, R4, R5: 33k, ~, symbol R
- added R19, R6: 7.5k, ~, symbol R
- added R2, R22, R27: 82k, ~, symbol R
- added R21, R28: 47k, ~, symbol R
- added R23, R26: 56k, ~, symbol R
- added R24, R25: 68k, ~, symbol R
- added unit 3 of U1
- added unit 1 of U1
- added unit 4 of U1
- added U10: NE5532, symbol TL082
- added U2, U6, U9: TL082, symbol TL082
- added unit 2 of U5
- added U7: TL074, symbol TL074
- added U8: SSM2164, MODULE, symbol SSM2164
- C3, C4: renamed from C?; value 560p -> 470p
- gave numbers to parts that had none: 18
Connections:
- net +5V: now also U5.8 (V+), C17.1, C21.1, C25.1, C27.1, R19.2, R6.2, U1.4 (V+), U1.4 (V+), U1.4 (V+), U10.8 (V+), U10.8 (V+), U2.8 (V+), U2.8 (V+), U5.8 (V+), U6.8 (V+), U6.8 (V+), U7.4 (V+), U7.4 (V+), U7.4 (V+), U7.4 (V+), U8.16 (V+), U9.8 (V+), U9.8 (V+)
- net -5V: now also P1.7 (P7), U5.4 (V-), C18.2, C22.2, C26.2, C28.2, R2.1, U1.11 (V-), U1.11 (V-), U1.11 (V-), U10.4 (V-), U10.4 (V-), U2.4 (V-), U2.4 (V-), U5.4 (V-), U6.4 (V-), U6.4 (V-), U7.11 (V-), U7.11 (V-), U7.11 (V-), U7.11 (V-), U8.9 (V-), U9.4 (V-), U9.4 (V-); no longer P1.9 (P9)
- net GND: now also P1.9 (P9), C1.2, C17.2, C18.1, C19.2, C2.2, C20.2, C21.2, C22.1, C23.2, C24.2, C25.2, C26.1, C27.2, C28.1, P11.2 (P2), P11.3 (P3), P12.1 (P1), P12.2 (PM), P12.3 (P3), U8.8 (GND); no longer P1.7 (P7)
- net at C8.1, U3.1 (X4): now also U7.12 (+)
- net at C13.1, U3.12 (X3): now also U1.5 (+)
- net at C16.1, U3.13 (X0): now also U1.12 (+); no longer U1.3 (+)
- net at C15.1, U3.14 (X1): now also U1.3 (+)
- net at C14.1, U3.15 (X2): now also U1.10 (+)
- net at C6.1, U3.2 (X6): now also U7.5 (+)
- net at U3.3 (X): now also R3.2, U2.1; no longer P1.4 (P4)
- net at C5.1, U3.4 (X7): now also U7.3 (+)
- net at C7.1, U3.5 (X5): now also U7.10 (+)
- net at U4.1 (MODE): now also R6.1
- net at U4.10 (IIN3): now also R4.2, R9.1
- net at U4.11 (VC3): now also U1.8, U1.9 (-)
- net at U4.12 (IOUT3): now also U5.5 (+)
- net at U4.13 (IOUT4): now also U5.3 (+)
- net at U4.14 (VC4): now also U1.6 (-), U1.7
- net at U4.15 (IIN4): now also R10.1, R5.2
- net at U4.3 (VC1): now also U1.13 (-), U1.14
- net at U4.4 (IOUT1): now also U6.3 (+)
- net at U4.5 (IOUT2): now also U6.5 (+)
- net at U4.6 (VC2): now also U1.1, U1.2 (-)
- net at U5.1: now also C9.2, P7.2 (PM), R13.2
- net at U5.2 (-): now also C9.1, R13.1
- new net: P1.4 (P4), U2.5 (+)
- new net: C10.1, R14.1, U5.6 (-)
- new net: C10.2, P6.2 (PM), R14.2, U5.7
- new net: C11.1, R15.1, U6.6 (-)
- new net: C11.2, P5.2 (PM), R15.2, U6.7
- new net: C12.2, P4.2 (PM), R16.2, U6.1
- new net: C12.1, R16.1, U6.2 (-)
- new net: P2.1 (P1), R4.1
- new net: P2.2 (PM), R5.1
- new net: C2.1, R10.2
- new net: C1.1, R9.2
- new net: P7.1 (P1), R25.1, R26.1
- new net: R22.2, R24.2, R26.2, R28.2, R29.2, R33.1, U8.7 (IIN2)
- new net: P8.1 (P1), R27.1, R28.1
- new net: R20.2, R21.2, R23.2, R25.2, R27.2, R32.1, U8.2 (IIN1)
- new net: P9.1 (P1), R29.1
- new net: P6.1 (P1), R23.1, R24.1
- new net: P5.1 (P1), R21.1, R22.1
- new net: P4.1 (P1), R20.1
- new net: R1.2, R2.2, U2.3 (+)
- new net: R1.1, U2.6 (-), U2.7
- new net: R19.1, U8.1 (MODE)
- new net: R3.1, U2.2 (-)
- new net: R17.2, R30.1, U8.10 (IIN3)
- new net: U7.13 (-), U7.14, U8.11 (VC3)
- new net: U8.12 (IOUT3), U9.5 (+)
- new net: U8.13 (IOUT4), U9.3 (+)
- new net: U7.8, U7.9 (-), U8.14 (VC4)
- new net: R18.2, R31.1, U8.15 (IIN4)
- new net: U7.6 (-), U7.7, U8.3 (VC1)
- new net: U10.5 (+), U8.4 (IOUT1)
- new net: U10.3 (+), U8.5 (IOUT2)
- new net: U7.1, U7.2 (-), U8.6 (VC2)
- new net: C29.2, P9.2 (PM), R34.2, U9.1
- new net: C29.1, R34.1, U9.2 (-)
- new net: C30.1, R35.1, U9.6 (-)
- new net: C30.2, P8.2 (PM), R35.2, U9.7
- new net: C31.2, P11.4 (P4), R36.2, U10.1
- new net: C31.1, R36.1, U10.2 (-)
- new net: C32.1, R37.1, U10.6 (-)
- new net: C32.2, P11.1 (P1), R37.2, U10.7
- new net: P10.1 (P1), R17.1
- new net: P10.2 (PM), R18.1
- new net: C20.1, R31.2
- new net: C19.1, R30.2
- new net: C24.1, R33.2
- new net: C23.1, R32.2
Other:
- moved on the sheet: C13, C14, C15, C16, C3, C4, C5, C6, C7, C8, P1, P3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

Commit message: schematics fixes
Parts:
- R22, R27: value 82k -> 150k
Connections:
- net GND: now also U10.3 (+), U10.5 (+), U5.3 (+), U5.5 (+), U6.3 (+), U6.5 (+), U9.3 (+), U9.5 (+)
- net at U4.12 (IOUT3): now also C10.1, R14.1, U5.6 (-); no longer U5.5 (+)
- net at U4.13 (IOUT4): now also C9.1, R13.1, U5.2 (-); no longer U5.3 (+)
- net at U4.4 (IOUT1): now also C12.1, R16.1, U6.2 (-); no longer U6.3 (+)
- net at U4.5 (IOUT2): now also C11.1, R15.1, U6.6 (-); no longer U6.5 (+)
- net at U8.12 (IOUT3): now also C30.1, R35.1, U9.6 (-); no longer U9.5 (+)
- net at U8.13 (IOUT4): now also C29.1, R34.1, U9.2 (-); no longer U9.3 (+)
- net at U8.4 (IOUT1): now also C32.1, R37.1, U10.6 (-); no longer U10.5 (+)
- net at U8.5 (IOUT2): now also C31.1, R36.1, U10.2 (-); no longer U10.3 (+)
Changed lines of the file:
@@
 Sheet 1 1
 Title "VCA  / Mixer board schematics"
-Date "21 sep 2013"
-Rev "2"
+Date "24 sep 2013"
+Rev "3"
 Comp "GliGli's DIY"
 Comment1 ""
@@
 P 8000 6450
 F 0 "R27" V 8080 6450 40  0000 C CNN
-F 1 "82k" V 8007 6451 40  0000 C CNN
+F 1 "150k" V 8007 6451 40  0000 C CNN
 F 2 "~" V 7930 6450 30  0000 C CNN
 F 3 "~" H 8000 6450 30  0000 C CNN
@@
 P 8000 5400
 F 0 "R22" V 8080 5400 40  0000 C CNN
-F 1 "82k" V 8007 5401 40  0000 C CNN
+F 1 "150k" V 8007 5401 40  0000 C CNN
 F 2 "~" V 7930 5400 30  0000 C CNN
 F 3 "~" H 8000 5400 30  0000 C CNN
@@
 	10200 1250 10200 1450
 Wire Wire Line
-	9650 1450 10250 1450
-Wire Wire Line
-	9650 1450 9650 1050
-Wire Wire Line
-	9650 1050 9700 1050
+	8650 1450 10250 1450
+Wire Wire Line
+	9550 1050 9700 1050
 Connection ~ 10200 1450
 Wire Wire Line
@@
 	10200 2300 10200 2500
 Wire Wire Line
-	9650 2500 10250 2500
-Wire Wire Line
-	9650 2500 9650 2100
-Wire Wire Line
-	9650 2100 9700 2100
+	9550 2500 10250 2500
 Connection ~ 10200 2500
 Wire Wire Line
@@
 	10200 3350 10200 3550
 Wire Wire Line
-	9650 3550 10250 3550
-Wire Wire Line
-	9650 3150 9650 3550
-Wire Wire Line
-	9650 3150 9700 3150
+	9550 3550 10250 3550
+Wire Wire Line
+	9550 3150 9700 3150
 Connection ~ 10200 3550
 Wire Wire Line
@@
 	9650 4600 9650 4200
 Wire Wire Line
-	9650 4200 9700 4200
+	9550 4200 9700 4200
 Connection ~ 10200 4600
 Wire Wire Line
@@
 	9550 1650 8750 1650
 Wire Wire Line
-	8650 4000 9700 4000
-Wire Wire Line
-	9550 3700 9550 2950
-Wire Wire Line
-	9550 2950 9700 2950
-Wire Wire Line
-	9700 1900 9550 1900
-Wire Wire Line
-	9550 1900 9550 1650
-Wire Wire Line
-	8650 2000 8650 1300
-Wire Wire Line
-	8650 1300 9550 1300
-Wire Wire Line
-	9550 1300 9550 850
-Wire Wire Line
-	9550 850  9700 850
+	8650 4000 9550 4000
+Wire Wire Line
+	9550 3700 9550 3150
+Wire Wire Line
+	9550 1650 9550 2500
+Wire Wire Line
+	8650 2000 8650 1450
 Wire Wire Line
 	3100 950  3150 950
@@
 	4900 1250 4900 1450
 Wire Wire Line
-	4350 1450 4950 1450
-Wire Wire Line
-	4350 1450 4350 1050
-Wire Wire Line
-	4350 1050 4400 1050
+	3350 1450 4950 1450
+Wire Wire Line
+	4250 1050 4400 1050
 Connection ~ 4900 1450
 Wire Wire Line
@@
 	4900 2300 4900 2500
 Wire Wire Line
-	4350 2500 4950 2500
-Wire Wire Line
-	4350 2500 4350 2100
-Wire Wire Line
-	4350 2100 4400 2100
+	4250 2500 4950 2500
+Wire Wire Line
+	4250 2100 4400 2100
 Connection ~ 4900 2500
 Wire Wire Line
@@
 	4900 3350 4900 3550
 Wire Wire Line
-	4350 3550 4950 3550
-Wire Wire Line
-	4350 3150 4350 3550
-Wire Wire Line
-	4350 3150 4400 3150
+	4250 3550 4950 3550
+Wire Wire Line
+	4250 3150 4400 3150
 Connection ~ 4900 3550
 Wire Wire Line
@@
 	4350 4600 4350 4200
 Wire Wire Line
-	4350 4200 4400 4200
+	4250 4200 4400 4200
 Connection ~ 4900 4600
 Wire Wire Line
@@
 	4250 1650 3450 1650
 Wire Wire Line
-	3350 4000 4400 4000
-Wire Wire Line
-	4250 3700 4250 2950
-Wire Wire Line
-	4250 2950 4400 2950
-Wire Wire Line
-	4400 1900 4250 1900
-Wire Wire Line
-	4250 1900 4250 1650
-Wire Wire Line
-	3350 2000 3350 1300
-Wire Wire Line
-	3350 1300 4250 1300
-Wire Wire Line
-	4250 1300 4250 850
-Wire Wire Line
-	4250 850  4400 850
+	3350 4000 4250 4000
+Wire Wire Line
+	4250 1650 4250 2500
+Wire Wire Line
+	3350 2000 3350 1450
 Connection ~ 4950 6550
 Connection ~ 4750 6650
@@
 	1150 5900 1150 5850
 Connection ~ 1150 5850
+Wire Wire Line
+	4250 4000 4250 4200
+Connection ~ 4350 4200
+Wire Wire Line
+	4250 3700 4250 3150
+Connection ~ 4250 3550
+Connection ~ 4250 2100
+Wire Wire Line
+	4250 1450 4250 1050
+Connection ~ 4250 1450
+Wire Wire Line
+	9550 2100 9700 2100
+Connection ~ 9550 2100
+Wire Wire Line
+	9550 1450 9550 1050
+Connection ~ 9550 1450
+Connection ~ 9550 3550
+Wire Wire Line
+	9550 4000 9550 4200
+Connection ~ 9650 4200
+$Comp
+L GND #PWR?
+U 1 1 524163BA
+P 4350 900
+F 0 "#PWR?" H 4350 900 30  0001 C CNN
+F 1 "GND" H 4350 830 30  0001 C CNN
+F 2 "" H 4350 900 60  0000 C CNN
+F 3 "" H 4350 900 60  0000 C CNN
+	1    4350 900
+	1    0    0    -1
+$EndComp
+Wire Wire Line
+	4350 900  4350 850
+Wire Wire Line
+	4350 850  4400 850
+$Comp
+L GND #PWR?
+U 1 1 52416635
+P 4350 1950
+F 0 "#PWR?" H 4350 1950 30  0001 C CNN
+F 1 "GND" H 4350 1880 30  0001 C CNN
+F 2 "" H 4350 1950 60  0000 C CNN
+F 3 "" H 4350 1950 60  0000 C CNN
+	1    4350 1950
+	1    0    0    -1
+$EndComp
+$Comp
+L GND #PWR?
+U 1 1 5241663B
+P 4350 3000
+F 0 "#PWR?" H 4350 3000 30  0001 C CNN
+F 1 "GND" H 4350 2930 30  0001 C CNN
+F 2 "" H 4350 3000 60  0000 C CNN
+F 3 "" H 4350 3000 60  0000 C CNN
+	1    4350 3000
+	1    0    0    -1
+$EndComp
+$Comp
+L GND #PWR?
+U 1 1 52416641
+P 4350 4050
+F 0 "#PWR?" H 4350 4050 30  0001 C CNN
+F 1 "GND" H 4350 3980 30  0001 C CNN
+F 2 "" H 4350 4050 60  0000 C CNN
+F 3 "" H 4350 4050 60  0000 C CNN
+	1    4350 4050
+	1    0    0    -1
+$EndComp
+$Comp
+L GND #PWR?
+U 1 1 52416647
+P 9650 900
+F 0 "#PWR?" H 9650 900 30  0001 C CNN
+F 1 "GND" H 9650 830 30  0001 C CNN
+F 2 "" H 9650 900 60  0000 C CNN
+F 3 "" H 9650 900 60  0000 C CNN
+	1    9650 900
+	1    0    0    -1
+$EndComp
+$Comp
+L GND #PWR?
+U 1 1 5241664D
+P 9650 1950
+F 0 "#PWR?" H 9650 1950 30  0001 C CNN
+F 1 "GND" H 9650 1880 30  0001 C CNN
+F 2 "" H 9650 1950 60  0000 C CNN
+F 3 "" H 9650 1950 60  0000 C CNN
+	1    9650 1950
+	1    0    0    -1
+$EndComp
+$Comp
+L GND #PWR?
+U 1 1 52416653
+P 9650 3000
+F 0 "#PWR?" H 9650 3000 30  0001 C CNN
+F 1 "GND" H 9650 2930 30  0001 C CNN
+F 2 "" H 9650 3000 60  0000 C CNN
+F 3 "" H 9650 3000 60  0000 C CNN
+	1    9650 3000
+	1    0    0    -1
+$EndComp
+$Comp
+L GND #PWR?
+U 1 1 52416659
+P 9650 4050
+F 0 "#PWR?" H 9650 4050 30  0001 C CNN
+F 1 "GND" H 9650 3980 30  0001 C CNN
+F 2 "" H 9650 4050 60  0000 C CNN
+F 3 "" H 9650 4050 60  0000 C CNN
+	1    9650 4050
+	1    0    0    -1
+$EndComp
+Wire Wire Line
+	9650 3000 9650 2950
+Wire Wire Line
+	9650 2950 9700 2950
+Wire Wire Line
+	9650 1950 9650 1900
+Wire Wire Line
+	9650 1900 9700 1900
+Wire Wire Line
+	9650 900  9650 850
+Wire Wire Line
+	9650 850  9700 850
+Wire Wire Line
+	4350 3000 4350 2950
+Wire Wire Line
+	4350 2950 4400 2950
+Wire Wire Line
+	4350 1950 4350 1900
+Wire Wire Line
+	4350 1900 4400 1900
+Wire Wire Line
+	4350 4050 4350 4000
+Wire Wire Line
+	4350 4000 4400 4000
+Wire Wire Line
+	9650 4050 9650 4000
+Wire Wire Line
+	9650 4000 9700 4000
 $EndSCHEMATC

Commit message: hardware: VCA board R4 (fully working version)
Parts:
- removed R19, R6: 7.5k, ~, symbol R
- added R38, R39: 1k, ~, symbol R
- U10: value NE5532 -> TL082
Connections:
- net at C31.2, R36.2, U10.1: now also R39.2; no longer P11.4 (P4)
- net at C32.2, R37.2, U10.7: now also R38.2; no longer P11.1 (P1)
- new net: P11.1 (P1), R38.1
- new net: P11.4 (P4), R39.1
Other:
- moved on the sheet: P11, P12

Commit message: hw: new LM13700-based VCA / Mixer board schematics
Parts:
- removed C10, C11, C12, C29, C30, C9: 100p, ~, symbol C
- removed C13, C14, C15, C16, C8: 47n, ~, symbol C
- removed C19, C20, C4: 470p, ~, symbol C
- removed P10: CARD_2, symbol CONN_2
- removed P2: CARD_0, symbol CONN_2
- removed U1, U7: TL074, symbol TL074
- removed U2, U5, U6, U9: TL082, symbol TL082
- removed U3: 4051, symbol 4051
- removed U4, U8: SSM2164, MODULE, symbol SSM2164
- added C10, C11, C12, C13, C14, C9: 100u, ~, symbol CP1
- added C25: 1u, ~, symbol CP1
- added C26: 100n, ~, symbol C
- added C4, C8: 22u, ~, symbol CP1
- added IC1, IC2, IC3, IC4: LM13700, symbol LM13700
- added P2: VCA_SPI, symbol CONN_5
- added P4: CARD_23, symbol CONN_2
- added P5: CARD_45, symbol CONN_2
- added R19, R20, R21, R22: 1k, ~, symbol R
- added R23, R24, R25, R26, R27, R28, R29: 6k8, ~, symbol R
- added R36: 33k, ~, symbol R
- added R37, R38, R39, R40, R41, R42, R6: 4k7, ~, symbol R
- added R57: 100k, ~, symbol R
- added RV1, RV2, RV3, RV4, RV5, RV6, RV7, RV8: 1k, ~, symbol POT
- added U1, U2, U3, U4: MCP4922-E/P, DIP14, symbol MCP4922-E/P
- added U5: 74HCT139, ~, symbol 74LS139
- C1, C2, C3: value 470p -> 470n
- C23, C24: value 470p -> 100n
- C5, C6, C7: value 47n -> 470n
- P10: renamed from P6; value OUT_2 -> OUT_0
- P11: renamed from P7; value OUT_3 -> OUT_1
- P12: renamed from P8; value OUT_4 -> OUT_3
- P3: value CARD_1 -> CARD_01
- P8: renamed from P4; value OUT_0 -> OUT_4
- P9: renamed from P5; value OUT_1 -> OUT_2
- R1, R3: value 10k -> 4k7
- R10, R11, R12, R9: value 470 -> 1k
- R17, R18: value 33k -> 10k
- R2: value 82k -> 4k7
- R30: value 470 -> 6k8
- R31, R32, R33: value 470 -> 33k
- R34, R35: value 10k -> 33k
- R4, R5, R7, R8: value 33k -> 4k7
- R53: renamed from R36; value 10k -> 47k
- R54: renamed from R37; value 10k -> 47k
- renumbered C31 to C15, C32 to C16, C21 to C19, C22 to C20, C25 to C21, C26 to C22, P9 to P13, P11 to P6, P12 to P7, R20 to R43, R21 to R44, R22 to R45, R23 to R46, R24 to R47, R25 to R48, R26 to R49, R27 to R50, R28 to R51, R29 to R52, R38 to R55, R39 to R56, U10 to U6
Connections:
- net +5V: now also C23.1, R30.2, C26.1, IC1.11 (V+), IC1.11 (V+), IC2.11 (V+), IC2.11 (V+), IC3.11 (V+), IC3.11 (V+), IC4.11 (V+), IC4.11 (V+), R23.2, R24.2, R25.2, R26.2, R27.2, R28.2, R29.2, R57.1, U1.1 (VDD), U1.9 (~SHDN~), U2.1 (VDD), U2.9 (~SHDN~), U3.1 (VDD), U3.9 (~SHDN~), U4.1 (VDD), U4.9 (~SHDN~), U5.13 (A1), U5.14 (A0), U5.15 (E), U5.16 (VCC), U5.16 (VCC)
- net -5V: now also C1.2, C2.2, C24.2, C3.2, C5.2, C6.2, C7.2, R10.2, R11.2, R12.2, R9.2, C4.2, C8.2, IC1.6 (V-), IC1.6 (V-), IC2.6 (V-), IC2.6 (V-), IC3.6 (V-), IC3.6 (V-), IC4.6 (V-), IC4.6 (V-), R19.2, R20.2, R21.2, R22.2, R37.2, R38.2, R39.2, R40.2, R41.2, R42.2; no longer R2.1
- net GND: now also C24.1, R31.2, R32.2, R33.2, R34.2, R35.2, C25.2, C26.2, R36.2, RV1.2, RV2.2, RV3.2, RV4.2, RV5.2, RV6.2, RV7.2, RV8.2, U1.12 (AVSS), U2.12 (AVSS), U3.12 (AVSS), U4.12 (AVSS), U5.8 (GND), U5.8 (GND); no longer C1.2, C2.2, C24.2, C3.2, C5.2, C6.2, C7.2
- net at P1.2 (P2): now also U5.3 (A1)
- net at P1.3 (P3): now also U5.2 (A0)
- net at C6.1: now also R4.2, IC2.1 (Iabc), R20.1
- net at R3.2: now also C2.1, R10.1, IC2.16 (Iabc)
- net at C5.1: now also R2.2, IC1.1 (Iabc), R19.1
- net at C7.1: now also IC3.1 (Iabc), R21.1, R6.2
- net at P1.5 (P5): now also U5.1 (E)
- net at R9.1: now also C1.1, R1.2, IC1.16 (Iabc); no longer R4.2
- net at R14.1: now also IC1.3 (+), RV2.3
- net at R13.1: now also IC1.14 (+), RV1.3
- net at R5.2: now also C3.1, R11.1, IC3.16 (Iabc); no longer R10.1
- net at R7.2: now also R12.1, C4.1, IC4.16 (Iabc); no longer R11.1
- net at R16.1: now also IC2.3 (+), RV4.3
- net at R15.1: now also IC2.14 (+), RV3.3
- net at R8.2: now also C8.1, IC4.1 (Iabc), R22.1; no longer R12.1
- net at P11.2 (PM): now also C10.2; no longer R13.2
- net at P3.1 (P1): now also R13.2; no longer R7.1
- net at P3.2 (PM): now also R14.2; no longer R8.1
- net at P10.2 (PM): now also C9.2; no longer R14.2
- net at P9.2 (PM): now also C11.2; no longer R15.2
- net at P8.2 (PM): now also C13.2; no longer R16.2
- net at R4.1: now also U2.10 (VoutB)
- net at R5.1: now also U3.14 (VoutA)
- net at R45.2, R47.2, R49.2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: now also IC4.3 (+), RV8.3; no longer R33.1
- net at R43.2, R44.2, R46.2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: now also IC4.14 (+), RV7.3; no longer R32.1
- net at R1.1: now also U1.14 (VoutA)
- net at R3.1: now also U2.14 (VoutA)
- net at R17.2: now also P5.1 (P1); no longer R30.1
- net at R35.1: now also IC3.10 (buffer_in), IC3.12 (out)
- net at R34.1: now also IC2.5 (out), IC2.7 (buffer_in)
- net at R31.1: now also IC1.10 (buffer_in), IC1.12 (out); no longer R18.2
- net at C16.1, R54.1, U6.6 (-): now also IC4.5 (out)
- net at C15.1, R53.1, U6.2 (-): now also IC4.12 (out)
- net at P13.2 (PM): now also C14.2; no longer R34.2
- net at P12.2 (PM): now also C12.2; no longer R35.2
- net at R17.1: now also IC3.14 (+), RV5.3
- net at R18.1: now also IC3.3 (+), RV6.3
- new net: P2.1, U1.5 (SDI), U2.5 (SDI), U3.5 (SDI), U4.5 (SDI)
- new net: P2.2, U1.4 (SCK), U2.4 (SCK), U3.4 (SCK), U4.4 (SCK)
- new net: P2.3, U1.3 (~CS~), U2.3 (~CS~), U3.3 (~CS~), U4.3 (~CS~)
- new net: R2.1, U1.10 (VoutB)
- new net: U1.8 (~LDAC~), U5.4 (O0)
- new net: IC1.13 (-), RV1.1
- new net: IC1.15 (bias), R23.1
- new net: C9.1, IC1.9 (buffer_out), R37.1
- new net: U2.8 (~LDAC~), U5.5 (O1)
- new net: U3.8 (~LDAC~), U5.6 (O2)
- new net: U4.8 (~LDAC~), U5.7 (O3)
- new net: IC1.2 (bias), R24.1
- new net: IC1.4 (-), RV2.1
- new net: IC1.5 (out), IC1.7 (buffer_in), R32.1
- new net: C10.1, IC1.8 (buffer_out), R38.1
- new net: IC2.10 (buffer_in), IC2.12 (out), R33.1
- new net: IC2.13 (-), RV3.1
- new net: IC2.15 (bias), R25.1
- new net: C11.1, IC2.9 (buffer_out), R39.1
- new net: IC2.2 (bias), R26.1
- new net: IC2.4 (-), RV4.1
- new net: C12.1, IC2.8 (buffer_out), R40.1
- new net: P4.1 (P1), R15.2
- new net: P4.2 (PM), R16.2
- new net: R6.1, U3.10 (VoutB)
- new net: IC3.13 (-), RV5.1
- new net: IC3.15 (bias), R27.1
- new net: C13.1, IC3.9 (buffer_out), R41.1
- new net: IC3.2 (bias), R28.1
- new net: IC3.4 (-), RV6.1
- new net: IC3.5 (out), IC3.7 (buffer_in), R36.1
- new net: C14.1, IC3.8 (buffer_out), R42.1
- new net: P5.2 (PM), R18.2
- new net: R8.1, U4.10 (VoutB)
- new net: R7.1, U4.14 (VoutA)
- new net: IC4.13 (-), RV7.1
- new net: IC4.15 (bias), R29.1
- new net: IC4.2 (bias), R30.1
- new net: IC4.4 (-), RV8.1
- new net VAA: C25.1, R57.2, U1.11 (VrefB), U1.13 (VrefA), U2.11 (VrefB), U2.13 (VrefA), U3.11 (VrefB), U3.13 (VrefA), U4.11 (VrefB), U4.13 (VrefA)
Other:
- moved on the sheet: C15, C16, C17, C18, C19, C20, C21, C22, C27, C28, P1, P10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

Commit message: hw: LM13700 vca board wip
Parts:
- added C29, C30, C31, C32: 100n, ~, symbol C
Connections:
- net +5V: now also C29.1, C30.1, C31.1, C32.1
- net GND: now also C29.2, C30.2, C31.2, C32.2
- net at IC4.14 (+), R43.2, R44.2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: now also RV7.1; no longer RV7.3
- net at IC1.13 (-): now also RV1.3; no longer RV1.1
- net at IC1.14 (+), R13.1: now also RV1.1; no longer RV1.3
- net at IC2.13 (-): now also RV3.3; no longer RV3.1
- net at IC2.14 (+), R15.1: now also RV3.1; no longer RV3.3
- net at IC3.13 (-): now also RV5.3; no longer RV5.1
- net at IC3.14 (+), R17.1: now also RV5.1; no longer RV5.3
- net at IC4.13 (-): now also RV7.3; no longer RV7.1
Other:
- moved on the sheet: C27, C28

Commit message: sh: LM13700 vca board routing finished
Connections:
- net +5V: now also U5.1 (E), U5.2 (A0), U5.3 (A1); no longer U5.13 (A1), U5.14 (A0), U5.15 (E)
- net at P1.2 (P2): now also U5.13 (A1); no longer U5.3 (A1)
- net at P1.3 (P3): now also U5.14 (A0); no longer U5.2 (A0)
- net at P1.5 (P5): now also U5.15 (E); no longer U5.1 (E)
- net at U1.8 (~LDAC~): now also U5.12 (O0); no longer U5.4 (O0)
- net at U2.8 (~LDAC~): now also U5.11 (O1); no longer U5.5 (O1)
- net at U3.8 (~LDAC~): now also U5.10 (O2); no longer U5.6 (O2)
- net at U4.8 (~LDAC~): now also U5.9 (O3); no longer U5.7 (O3)
Changed lines of the file:
@@
 $Comp
 L 74LS139 U5
-U 1 1 5415B781
+U 2 1 5415B781
 P 2500 10650
 F 0 "U5" H 2500 10750 60  0000 C CNN
@@
 F 2 "~" H 2500 10650 60  0000 C CNN
 F 3 "~" H 2500 10650 60  0000 C CNN
-	1    2500 10650
+	2    2500 10650
 	1    0    0    -1
 $EndComp
@@
 $Comp
 L 74LS139 U5
-U 2 1 5416807B
+U 1 1 5416807B
 P 5000 10650
 F 0 "U5" H 5000 10750 60  0000 C CNN
@@
 F 2 "~" H 5000 10650 60  0000 C CNN
 F 3 "~" H 5000 10650 60  0000 C CNN
-	2    5000 10650
-	1    0    0    -1
-$EndComp
+	1    5000 10650
+	1    0    0    -1
+$EndComp
