File: hardware/overcycler.kicad_pcb (KiCad board)
At the start: 2 copper layers, 99.1 x 104.1 mm, 42 parts, among them P1 LPC_P1, P10 VCA_CMD_PWR, P11 AC_IN, P12 FOOT_IN, P13 MIDI_IN, P2 LPC_P2, P3 FT232, P4 CARD0_CMD_PWR, P5 SDCARD, P6 CARD1_CMD_PWR, P7 SCREEN, P8 CARD2_CMD_PWR, P9 TEN_POTS, SW1 RESET, U1 4053, U2 4053, U3 MCP4921-E/P, U4 LM1084IT-5.0/NOPB, U5 LM2990-5.0/NOPB, U6 LM1084IT-3.3/NOPB

Commit message: mainboard almost ok
Parts:
- removed C2: 100n, C2
- P9: footprint SIL-12 -> pin_array_6x2
- moved U2 91.9 mm to (31.8, 120.0), turned to 270 degrees
- moved R5 83.3 mm to (33.0, 134.6), turned to 0 degrees
- moved SW1 80.7 mm to (61.0, 43.2), turned to 90 degrees
- moved P13 79.6 mm to (38.7, 141.6), turned to 270 degrees
- moved P3 77.4 mm to (42.5, 40.0), turned to 180 degrees
- moved C1 75.2 mm to (27.9, 88.3), turned to 270 degrees
- moved D3 72.3 mm to (43.8, 134.6), turned to 180 degrees
- moved OC1 66.4 mm to (50.8, 141.6), turned to 270 degrees
- moved C9 60.4 mm to (103.5, 116.8)
- moved R3 57.3 mm to (63.5, 141.6), turned to 180 degrees
- moved R2 56.4 mm to (63.5, 145.4), turned to 180 degrees
- moved P12 56.1 mm to (105.4, 112.4), turned to 0 degrees
- moved P5 54.8 mm to (27.9, 47.6), turned to 90 degrees
- moved R4 53.2 mm to (93.3, 116.2)
- moved P2 52.4 mm to (76.2, 78.1), turned to 270 degrees
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Connections:
- P10 pad 7: GND -> -5V
- P10 pad 9: -5V -> GND
- P2 pad 27: (no net) -> GND
- P9 pad 1: GND -> +3.3V
- P9 pad 10: N-0000010 (its old number) -> N-0000027
- P9 pad 11: N-0000011 (its old number) -> N-0000025
- P9 pad 12: N-000002 (its old number) -> N-0000026
- P9 pad 2: +3.3V -> GND
- P9 pad 4: N-000005 -> N-0000034
- P9 pad 5: N-000006 (its old number) -> N-0000022
- P9 pad 6: N-000007 -> N-000005
- P9 pad 7: N-000003 (its old number) -> N-0000023
- P9 pad 8: N-000008 -> N-0000028
- P9 pad 9: N-000009 (its old number) -> N-0000020
- U1 pad 1: N-000007 -> N-0000020
- U1 pad 13: N-000005 -> N-0000022
- U1 pad 2: N-000006 (its old number) -> N-0000023
- U1 pad 3: N-000008 -> N-0000026
- U1 pad 5: N-000003 (its old number) -> N-0000025
- U2 pad 1: N-000002 (its old number) -> N-0000034
- U2 pad 12: N-000009 (its old number) -> N-0000027
- U2 pad 13: N-0000010 (its old number) -> N-0000028
- U2 pad 2: N-0000011 (its old number) -> N-000005
Routing:
- net GND: track 0.00 -> 592.9 mm
- net +5V: track 0.00 -> 423.0 mm, vias 0 -> 5
- net +3.3V: track 0.00 -> 245.3 mm, vias 0 -> 2
- net N-0000045: track 0.00 -> 136.4 mm, vias 0 -> 3
- net -5V: track 0.00 -> 124.9 mm, vias 0 -> 2
- net N-0000040: track 0.00 -> 110.0 mm, vias 0 -> 1
- net N-000003: track 0.00 -> 109.1 mm, vias 0 -> 2
- net N-000002: track 0.00 -> 104.7 mm, vias 0 -> 2
- net N-000004: track 0.00 -> 101.6 mm, vias 0 -> 1
- net N-000001: track 0.00 -> 101.4 mm, vias 0 -> 3
- net N-0000024: track 0.00 -> 97.5 mm
- net /UNR+: track 0.00 -> 95.7 mm
- net N-0000041: track 0.00 -> 93.7 mm, vias 0 -> 3
- net N-000006: track 0.00 -> 93.0 mm, vias 0 -> 2
- net N-0000035: track 0.00 -> 92.5 mm, vias 0 -> 1
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Other:
- board size 99.1 x 104.1 mm -> 99.1 x 109.2 mm
- net class ac removed
- net class pwr removed

Commit message: mainboard ok
Parts:
- added C2: 100n, C2, F.Cu at (224.2, 73.4)
- moved HOLE1 5.30 mm to (33.0, 55.0)
- moved HOLE2 1.92 mm to (33.0, 142.0)
Connections:
- P5 pad 6: GND -> (no net)
Routing:
- net GND: track 592.9 -> 581.2 mm
- net +5V: track 423.0 -> 415.3 mm, vias 5 -> 4
- net N-0000057: track 36.9 -> 34.3 mm
- net N-0000056: track 28.6 -> 30.9 mm
- net N-0000058: track 35.7 -> 33.8 mm, vias 2 -> 1
- net N-0000059: track 30.1 -> 31.6 mm
Other:
- board text added: "GliGli's DIY OverCycler"

Commit message: hardware updates
Parts:
- U4, U5, U6: footprint TO220_VERT -> TO220_VERT_FIXED
- moved C2 102.3 mm to (127.0, 41.3), turned to 90 degrees
- moved U5 1.91 mm to (100.3, 144.8)
- moved U6 1.91 mm to (76.2, 144.8)
- moved HOLE1 1.00 mm to (33.0, 56.0)
- moved HOLE2 1.00 mm to (33.0, 143.0)
- moved C5 0.64 mm to (109.2, 137.8)
- moved U4 0.64 mm to (118.1, 144.8)
- moved R2 0.51 mm to (64.0, 145.4)
- moved R3 0.51 mm to (64.0, 141.6)
Routing:
- net /UNR+: track 95.7 -> 67.1 mm
- net GND: track 581.2 -> 602.9 mm
- net +3.3V: track 245.3 -> 264.5 mm
- net -5V: track 124.9 -> 138.8 mm
- net /UNR-: track 30.7 -> 25.5 mm
- net N-000008: track 5.61 -> 9.92 mm
- net /MIDI_IN: track 44.6 -> 47.9 mm
- net N-0000044: track 81.7 -> 84.8 mm
- net +5V: track 415.3 -> 416.4 mm, vias 4 -> 3
Other:
- net class Default: clearance 0.508 -> 0.4826
- rule trace_clearance: 0.508 -> 0.4826
- board text added: "OverCycler MainBoard R3"
- board text removed: "GliGli's DIY OverCycler"

Commit message: schematics fixes
Connections:
- P2 pad 30: N-000005 -> N-000004
- P2 pad 31: N-000004 -> N-000005
Routing:
- net N-000005: track 93.0 -> 96.7 mm
- net N-000004: track 101.6 -> 99.7 mm
Other:
- board text added: "OverCycler MainBoard R4"
- board text removed: "OverCycler MainBoard R3"

Commit message: hw: fix for potmux noise
Connections:
- U1 pad 16: +5V -> +3.3V
- U2 pad 16: +5V -> +3.3V
Routing:
- net +5V: track 416.4 -> 341.3 mm, vias 3 -> 2
- net +3.3V: track 264.5 -> 339.6 mm, vias 2 -> 3

Commit message: sch: fix mainboard footswitch resistor value
Parts:
- R4: value 100k -> 10k
Routing:
- net +5V: track 341.3 -> 311.8 mm
- net +3.3V: track 339.6 -> 369.2 mm
Changed lines of the file:
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@@
       (effects (font (size 1.397 1.27) (thickness 0.2032)))
     )
-    (fp_text value 100k (at 0 0) (layer F.SilkS) hide
+    (fp_text value 10k (at 0 0) (layer F.SilkS) hide
       (effects (font (size 1.397 1.27) (thickness 0.2032)))
     )
@@
   (segment (start 48.387 92.2727) (end 48.387 100.3303) (width 0.762) (layer B.Cu) (net 1))
   (segment (start 49.6573 91.0024) (end 48.387 92.2727) (width 0.762) (layer B.Cu) (net 1))
+  (segment (start 45.5927 61.4951) (end 45.5927 81.28) (width 0.762) (layer F.Cu) (net 1))
+  (segment (start 49.6573 81.28) (end 49.6573 91.0024) (width 0.762) (layer B.Cu) (net 1))
   (segment (start 116.84 70.485) (end 116.84 40.030398) (width 2.032) (layer B.Cu) (net 2))
   (segment (start 116.865398 40.005) (end 116.84 40.005) (width 2.032) (layer B.Cu) (net 2))
@@
   (segment (start 47.625 81.28) (end 49.6573 81.28) (width 0.762) (layer B.Cu) (net 2))
   (segment (start 47.625 81.28) (end 45.5927 81.28) (width 0.762) (layer F.Cu) (net 2))
-  (segment (start 45.5927 61.4951) (end 45.5927 81.28) (width 0.762) (layer F.Cu) (net 2))
   (segment (start 52.5777 48.2819) (end 52.5777 48.26) (width 0.762) (layer B.Cu) (net 2))
   (segment (start 47.641 53.2186) (end 52.5777 48.2819) (width 0.762) (layer B.Cu) (net 2))
   (segment (start 54.61 48.26) (end 52.5777 48.26) (width 0.762) (layer B.Cu) (net 2))
-  (segment (start 49.6573 81.28) (end 49.6573 91.0024) (width 0.762) (layer B.Cu) (net 2))
   (segment (start 83.0535 118.8765) (end 83.0535 124.333) (width 0.762) (layer B.Cu) (net 2))
   (segment (start 89.535 112.395) (end 83.0535 118.8765) (width 0.762) (layer B.Cu) (net 2))

Commit message: hw: revised mainboard
Parts:
- removed C1, C2: 100n, C2
- added C10: 100n, C2, F.Cu at (31.8, 132.1)
- added C11: 100n, C2, F.Cu at (36.8, 60.3)
- added P14: VCA_SPI, SIL-5, F.Cu at (114.3, 81.3)
- C4: value 3300u -> 10000u
- C5: value 2200u -> 10000u
- C6, C7, C8: footprint C1.5V8V -> C1V8
- RV1: footprint RV2 -> RV2X1.5
- moved SW1 70.8 mm to (43.2, 111.8)
- moved C8 25.2 mm to (64.5, 135.9), turned to 0 degrees
- moved C7 8.89 mm to (98.4, 128.3)
- moved P10 7.18 mm to (114.3, 101.6)
- moved D2 5.72 mm to (106.7, 122.6)
- moved P11 5.72 mm to (116.8, 121.3)
- moved D1 5.71 mm to (106.7, 118.7)
- moved U2 3.42 mm to (33.0, 116.8), turned to 90 degrees
- moved C4 3.24 mm to (87.6, 134.6)
- moved C5 3.17 mm to (109.2, 134.6)
- moved R1 2.88 mm to (104.1, 105.4)
- moved R4 2.62 mm to (92.7, 113.7)
- moved R6 2.62 mm to (92.7, 109.9)
- moved P12 2.62 mm to (104.8, 109.9)
- moved C9 2.54 mm to (103.5, 114.3)
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Connections:
- P10 pad 4: N-0000042 (its old number) -> (no net)
- P4 pad 4: N-0000042 (its old number) -> N-0000045
- P6 pad 4: N-0000042 (its old number) -> N-0000045
- P8 pad 4: N-0000042 (its old number) -> N-0000045
- U3 pad 8: N-0000042 (its old number) -> N-0000045
Routing:
- net GND: track 602.9 -> 475.0 mm, vias 0 -> 2
- net N-0000042 (its old number): track 93.7 -> 0.00 mm, vias 3 -> 0
- net N-0000045: track 0.00 -> 68.7 mm, vias 0 -> 1
- net +3.3V: track 369.2 -> 313.6 mm
- net N-0000027: track 20.1 -> 72.3 mm
- net N-0000042: track 136.4 -> 90.7 mm, vias 3 -> 2
- net +5V: track 311.8 -> 269.2 mm
- net N-000005: track 31.1 -> 64.6 mm, vias 1 -> 0
- net N-0000043: track 84.8 -> 61.4 mm
- net N-0000036: track 50.8 -> 29.1 mm
- net N-000006: track 37.6 -> 53.0 mm
- net N-0000049: track 74.0 -> 58.7 mm
- net N-0000033: track 97.5 -> 82.9 mm
- net N-000003: track 18.8 -> 33.4 mm
- net /AC_IN: track 23.2 -> 10.2 mm
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Other:
- net class Default: via_dia 2.032 -> 1.524
- net class pwr added: clearance 0.4826, trace_width 1.524, via_dia 2.032, via_drill 0.508
- board text added: "OverCycler MainBoard R5"
- board text removed: "OverCycler MainBoard R4"
