File: hardware/overcycler2.sch (KiCad schematic (older format))
At the start: 104 parts

Commit message: simulated master mixer output -- sch fixes
Parts:
- removed R? (x2): 47k, ~, symbol R
- R? (x2): value 10k -> 8k2
Connections:
- net GND: now also P?.3 (P3); no longer P?.5 (P5)
- net at R?.1, U?.1: now also P?.4 (P4); no longer P?.3 (P3)
- net at U?.3 (+): now also P?.5 (P5); no longer P?.4 (P4)
Changed lines of the file:
@@
 LIBS:contrib
 LIBS:valves
-LIBS:TLV1543
-LIBS:ok-ic-analog
-LIBS:SSM2044
-LIBS:LTC1660
-LIBS:hardware-cache
-LIBS:vca-cache
+LIBS:overcycler2-cache
 EELAYER 27 0
 EELAYER END
@@
 Sheet 1 1
 Title "LM13700-based VCA  / Mixer board schematics"
-Date "9 sep 2015"
+Date "10 sep 2015"
 Rev "5"
 Comp "GliGli's DIY"
@@
 	12850 4350 12850 3950
 Wire Wire Line
-	12700 3950 12850 3950
-Wire Wire Line
 	12850 3950 12900 3950
 Wire Wire Line
-	12700 5050 12850 5050
-Wire Wire Line
 	12850 5050 12900 5050
 Wire Wire Line
@@
 	11950 6250 11950 6050
 Wire Wire Line
-	11950 6050 12500 6050
-Wire Wire Line
-	12500 6050 12600 6050
+	11950 6050 12300 6050
 Wire Wire Line
-	12500 6050 12500 6150
+	12300 6050 12600 6050
 Wire Wire Line
 	12600 6050 12600 6150
-Connection ~ 12500 6050
 $Comp
 L GND #PWR?
@@
 P 11800 4350
 F 0 "R?" V 11880 4350 40  0000 C CNN
-F 1 "10k" V 11807 4351 40  0000 C CNN
+F 1 "8k2" V 11807 4351 40  0000 C CNN
 F 2 "~" V 11730 4350 30  0000 C CNN
 F 3 "~" H 11800 4350 30  0000 C CNN
@@
 P 11800 5450
 F 0 "R?" V 11880 5450 40  0000 C CNN
-F 1 "10k" V 11807 5451 40  0000 C CNN
+F 1 "8k2" V 11807 5451 40  0000 C CNN
 F 2 "~" V 11730 5450 30  0000 C CNN
 F 3 "~" H 11800 5450 30  0000 C CNN
@@
 	12050 5450 12100 5450
 Wire Wire Line
-	12100 5450 12300 5450
+	12100 5450 12400 5450
 Wire Wire Line
 	11550 5450 11000 5450
@@
 	0    -1   -1   0
 $EndComp
-$Comp
-L R R?
-U 1 1 55F1104E
-P 12700 4200
-F 0 "R?" V 12780 4200 40  0000 C CNN
-F 1 "47k" V 12707 4201 40  0000 C CNN
-F 2 "~" V 12630 4200 30  0000 C CNN
-F 3 "~" H 12700 4200 30  0000 C CNN
-	1    12700 4200
-	-1   0    0    -1
-$EndComp
-$Comp
-L R R?
-U 1 1 55F11054
-P 12700 5300
-F 0 "R?" V 12780 5300 40  0000 C CNN
-F 1 "47k" V 12707 5301 40  0000 C CNN
-F 2 "~" V 12630 5300 30  0000 C CNN
-F 3 "~" H 12700 5300 30  0000 C CNN
-	1    12700 5300
-	-1   0    0    -1
-$EndComp
-$Comp
-L GND #PWR?
-U 1 1 55F1106E
-P 12700 5600
-F 0 "#PWR?" H 12700 5600 30  0001 C CNN
-F 1 "GND" H 12700 5530 30  0001 C CNN
-F 2 "" H 12700 5600 60  0000 C CNN
-F 3 "" H 12700 5600 60  0000 C CNN
-	1    12700 5600
-	1    0    0    -1
-$EndComp
-$Comp
-L GND #PWR?
-U 1 1 55F11074
-P 12700 4500
-F 0 "#PWR?" H 12700 4500 30  0001 C CNN
-F 1 "GND" H 12700 4430 30  0001 C CNN
-F 2 "" H 12700 4500 60  0000 C CNN
-F 3 "" H 12700 4500 60  0000 C CNN
-	1    12700 4500
-	1    0    0    -1
-$EndComp
-Connection ~ 12850 3950
-Wire Wire Line
-	12700 4450 12700 4500
-Wire Wire Line
-	12700 5550 12700 5600
-Connection ~ 12850 5050
-Wire Wire Line
-	12900 3750 12450 3750
-Wire Wire Line
-	12450 3750 12450 5850
-Wire Wire Line
-	12450 5850 12200 5850
-Wire Wire Line
-	12200 5850 12200 6150
 Wire Wire Line
-	12400 6150 12400 5950
+	12300 3750 12900 3750
 Wire Wire Line
-	12400 5950 12550 5950
+	12200 5950 12200 6150
 Wire Wire Line
-	12550 5950 12550 4850
-Wire Wire Line
-	12550 4850 12900 4850
-Wire Wire Line
-	12300 5450 12300 6150
+	12500 4850 12900 4850
 Connection ~ 12100 5450
 Wire Wire Line
-	12100 6150 12100 5750
+	12100 6150 12100 5850
 Wire Wire Line
-	12100 5750 12200 5750
+	12200 4350 12200 5750
 Wire Wire Line
-	12200 5750 12200 4350
+	12200 5750 12200 5850
 Connection ~ 12100 4350
 $Comp
@@
 Text Label 7650 2850 0    60   ~ 0
 DAC_VREF
+Wire Wire Line
+	12500 4850 12500 6150
+Wire Wire Line
+	12400 5450 12400 6150
+Wire Wire Line
+	12300 6050 12300 6150
+Connection ~ 12300 6050
+Wire Wire Line
+	12300 3750 12300 5950
+Wire Wire Line
+	12300 5950 12200 5950
+Wire Wire Line
+	12200 5850 12100 5850
 $EndSCHEMATC

Commit message: working VC noise gen -- sch tweaks
Parts:
- removed C?: 100u, ~, symbol CP1
- removed R? (x8): 10k, ~, symbol R
- added C? (x2): 100u, ~, symbol CP1
- added C? (x11): 100n, ~, symbol C
- added C? (x3): 10n, ~, symbol C
- added D? (x4): 1N4148, ~, symbol DIODE
- added Q?: BC547, TO92, symbol BC547
- added R?: 47k, ~, symbol R
- added R?: 1k, ~, symbol R
- added R? (x2): 100k, ~, symbol R
- added R?: 4k7, ~, symbol R
- added R? (x2): 470, ~, symbol R
- added R?: 2M2, ~, symbol R
- added R? (x3): 10k, ~, symbol R
- added R?: 27k, ~, symbol R
- added R?: 1M, ~, symbol R
- added RR?: 10k, ~, symbol RR8
- added U? (x4): TL074, symbol TL074
- C? (x3): value 100n -> 10n
Connections:
- net VDD is gone; now on net +3.3V: U?.16 (VDD)
- net VSS is gone; now on net GND: U?.8 (VSS)
- net +3.3V: now also C?.1, RR?.1 (COM)
- net +5V: now also C?.1, C?.1, C?.1, C?.1, C?.1, C?.1, C?.1, C?.1, C?.1, R?.2, U?.4 (V+), U?.4 (V+), U?.4 (V+), U?.4 (V+)
- net -5V: now also C?.2, C?.2, C?.2, Q?.2 (B), U?.11 (V-), U?.11 (V-), U?.11 (V-), U?.11 (V-)
- net GND: now also C?.1, C?.1, C?.1, C?.2, C?.2, C?.2, C?.2, C?.2, C?.2, C?.2, C?.2, C?.2, C?.2, C?.2, R?.1, R?.1, R?.1, U?.3 (+)
- net NOISE: now also C?.2
- net SPI_DAC0: now also RR?.2
- net SPI_DAC1: now also RR?.3
- net SPI_DAC2: now also RR?.4
- net SPI_DAC3: now also RR?.5
- net SPI_DAC4: now also RR?.6
- net SPI_DAC5: now also RR?.7
- net SPI_DAC6: now also RR?.8
- net SPI_DAC7: now also RR?.9
- net DAC_MIXN: now reaches U?.15 (VOUTH)
- net DAC_MIXN: now also R?.2
- new net: R?.1, R?.2, U?.1, U?.2 (-)
- new net: R?.1, R?.2, U?.3 (+)
- new net: R?.2, R?.2, U?.1
- new net: R?.1, R?.2, U?.2 (-) (x2)
- new net: C?.2, R?.2, U?.3 (+)
- new net: R?.1, R?.2, U?.1
- new net: R?.2, R?.2, U?.2 (-)
- new net: C?.1, R?.2, U?.1
- new net: D?.1 (A), D?.2 (K), R?.1, U?.3 (+)
- new net: C?.1, Q?.3 (E), R?.1
- new net: C?.1, R?.1
- new net: D?.1 (A), D?.2 (K) (x2)
- new net: D?.1 (A), R?.1
- new net: D?.2 (K), R?.1
Other:
- moved on the sheet: C?, P?, R?, U?, U?A

Commit message: DAC / mixer / filter sch ok
Parts:
- C? (x2): value 100u -> 22u
- R?: value 4k7 -> 6k8
- R?: value 8k2 -> 5k6
Changed lines of the file:
@@
 P 6350 8350
 F 0 "R?" V 6430 8350 40  0000 C CNN
-F 1 "4k7" V 6357 8351 40  0000 C CNN
+F 1 "6k8" V 6357 8351 40  0000 C CNN
 F 2 "~" V 6280 8350 30  0000 C CNN
 F 3 "~" H 6350 8350 30  0000 C CNN
@@
 P 8200 9450
 F 0 "R?" V 8280 9450 40  0000 C CNN
-F 1 "8k2" V 8207 9451 40  0000 C CNN
+F 1 "5k6" V 8207 9451 40  0000 C CNN
 F 2 "~" V 8130 9450 30  0000 C CNN
 F 3 "~" H 8200 9450 30  0000 C CNN
@@
 P 4900 8600
 F 0 "C?" H 4950 8700 50  0000 L CNN
-F 1 "100u" H 4950 8500 50  0000 L CNN
+F 1 "22u" H 4950 8500 50  0000 L CNN
 F 2 "~" H 4900 8600 60  0000 C CNN
 F 3 "~" H 4900 8600 60  0000 C CNN
@@
 P 4900 8900
 F 0 "C?" H 4950 9000 50  0000 L CNN
-F 1 "100u" H 4950 8800 50  0000 L CNN
+F 1 "22u" H 4950 8800 50  0000 L CNN
 F 2 "~" H 4900 8900 60  0000 C CNN
 F 3 "~" H 4900 8900 60  0000 C CNN

Commit message: vcf range adjustments
Parts:
- R?: value 470 -> 390
- R?: value 6k8 -> 5k6
- R?: value 5k6 -> 6k8
- R?: value 18k -> 15k
Changed lines of the file:
@@
 Sheet 1 1
 Title "OverCycler 2 full board"
-Date "11 sep 2015"
+Date "12 sep 2015"
 Rev "5"
 Comp "GliGli's DIY"
@@
 P 8700 9050
 F 0 "R?" V 8780 9050 40  0000 C CNN
-F 1 "470" V 8707 9051 40  0000 C CNN
+F 1 "390" V 8707 9051 40  0000 C CNN
 F 2 "~" V 8630 9050 30  0000 C CNN
 F 3 "~" H 8700 9050 30  0000 C CNN
@@
 P 6350 8350
 F 0 "R?" V 6430 8350 40  0000 C CNN
-F 1 "6k8" V 6357 8351 40  0000 C CNN
+F 1 "5k6" V 6357 8351 40  0000 C CNN
 F 2 "~" V 6280 8350 30  0000 C CNN
 F 3 "~" H 6350 8350 30  0000 C CNN
@@
 P 8200 9450
 F 0 "R?" V 8280 9450 40  0000 C CNN
-F 1 "5k6" V 8207 9451 40  0000 C CNN
+F 1 "6k8" V 8207 9451 40  0000 C CNN
 F 2 "~" V 8130 9450 30  0000 C CNN
 F 3 "~" H 8200 9450 30  0000 C CNN
@@
 P 9050 9350
 F 0 "R?" V 9130 9350 40  0000 C CNN
-F 1 "18k" V 9057 9351 40  0000 C CNN
+F 1 "15k" V 9057 9351 40  0000 C CNN
 F 2 "~" V 8980 9350 30  0000 C CNN
 F 3 "~" H 9050 9350 30  0000 C CNN

Commit message: vca range adjustments -- vca spice model update
Parts:
- C?: value 100u -> 33u
- R?: value 27k -> 22k
Connections:
- net OUT_V0: now also C?.1; no longer C?.2
- net at IC?.9 (buffer_out), R?.1: now also C?.2; no longer C?.1
Changed lines of the file:
@@
 P 9300 8100
 F 0 "C?" H 9350 8200 50  0000 L CNN
-F 1 "100u" H 9350 8000 50  0000 L CNN
+F 1 "33u" H 9350 8000 50  0000 L CNN
 F 2 "~" H 9300 8100 60  0000 C CNN
 F 3 "~" H 9300 8100 60  0000 C CNN
@@
 P 11250 8800
 F 0 "R?" V 11330 8800 40  0000 C CNN
-F 1 "27k" V 11257 8801 40  0000 C CNN
+F 1 "22k" V 11257 8801 40  0000 C CNN
 F 2 "~" V 11180 8800 30  0000 C CNN
 F 3 "~" H 11250 8800 30  0000 C CNN
@@
 F 3 "~" H 12100 8500 60  0000 C CNN
 	1    12100 8500
-	0    -1   1    0
-$EndComp
-$Comp
+	0    1    -1   0
+$EndComp
+$Comp

Commit message: output range adjustments -- output spice model update
Parts:
- R? (x2): value 8k2 -> 12k
Changed lines of the file:
@@
 P 13400 3350
 F 0 "R?" V 13480 3350 40  0000 C CNN
-F 1 "8k2" V 13407 3351 40  0000 C CNN
+F 1 "12k" V 13407 3351 40  0000 C CNN
 F 2 "~" V 13330 3350 30  0000 C CNN
 F 3 "~" H 13400 3350 30  0000 C CNN
@@
 P 13400 4450
 F 0 "R?" V 13480 4450 40  0000 C CNN
-F 1 "8k2" V 13407 4451 40  0000 C CNN
+F 1 "12k" V 13407 4451 40  0000 C CNN
 F 2 "~" V 13330 4450 30  0000 C CNN
 F 3 "~" H 13400 4450 30  0000 C CNN

Commit message: output stage can be pushed a little harder without clipping
Parts:
- R? (x2): value 12k -> 15k
Changed lines of the file:
@@
 P 13400 3350
 F 0 "R?" V 13480 3350 40  0000 C CNN
-F 1 "12k" V 13407 3351 40  0000 C CNN
+F 1 "15k" V 13407 3351 40  0000 C CNN
 F 2 "~" V 13330 3350 30  0000 C CNN
 F 3 "~" H 13400 3350 30  0000 C CNN
@@
 P 13400 4450
 F 0 "R?" V 13480 4450 40  0000 C CNN
-F 1 "12k" V 13407 4451 40  0000 C CNN
+F 1 "15k" V 13407 4451 40  0000 C CNN
 F 2 "~" V 13330 4450 30  0000 C CNN
 F 3 "~" H 13400 4450 30  0000 C CNN

Commit message: hierarchical sheet for voice
Parts:
- removed C? (x3): 10n, ~, symbol C
- removed C?: 820p, ~, symbol C
- removed C?: 33u, ~, symbol CP1
- removed C? (x2): 22u, ~, symbol CP1
- removed C?: 470n, ~, symbol C
- removed C?: 100u, ~, symbol CP1
- removed IC?: LM13700, symbol LM13700
- removed R?: 220, ~, symbol R
- removed R?: 390, ~, symbol R
- removed R?: 5k6, ~, symbol R
- removed R?: 6k8, ~, symbol R
- removed R?: 15k, ~, symbol R
- removed R? (x3): 4k7, ~, symbol R
- removed R? (x2): 15k, symbol R
- removed R?: 22k, symbol R
- removed R?: 220, symbol R
- removed R?: 820, ~, symbol R
- removed R?: 22k, ~, symbol R
- removed R?: 10k, ~, symbol R
- removed RV?: 1k, ~, symbol POT
- removed U?: SSM2044, MODULE, symbol SSM2044
- removed U?: MCP4922-E/P, DIP14, symbol MCP4922-E/P
- U2: renamed from U?; value 4051 -> 74HCT4051
- gave numbers to parts that had none: 97
Connections:
- net DAC_MIXN: now also U4.14 (VOUTG); no longer U4.15 (VOUTH)
- net DAC_RES: now also U4.15 (VOUTH); no longer U4.14 (VOUTG)
- net GND: now also U5.10 (+), U6.5 (+); no longer U5.3 (+), U6.3 (+)
- net at R22.1, R24.1, R26.1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: now also U6.6 (-); no longer U6.2 (-)
- net at C31.1, R32.1: now also U6.9 (-); no longer U6.2 (-)
- net at C31.2, R32.2, R35.2: now also U6.8; no longer U6.1
- net at C32.1, R33.1: now also U6.13 (-); no longer U6.2 (-)
- net at C32.2, R33.2, R34.2: now also U6.14; no longer U6.1
- net at P9.2 (P2): now also U6.10 (+); no longer U6.3 (+)
- net at P9.4 (P4), R31.1: now also U6.7; no longer U6.1
- net at P9.5 (P5): now also U6.12 (+); no longer U6.3 (+)
- net at R12.1, R15.2: now also U5.6 (-), U5.7; no longer U5.1, U5.2 (-)
- net at R11.2, R9.1: now also U5.5 (+); no longer U5.3 (+)
- net at R14.1, R17.2: now also U5.8; no longer U5.1
- net at R12.2, R14.2: now also U5.9 (-); no longer U5.2 (-)
- net at C23.1, R19.2: now also U5.14; no longer U5.1
- net at R18.2, R19.1: now also U5.13 (-); no longer U5.2 (-)
- net at D3.2 (K), D4.1 (A), R16.1: now also U5.12 (+); no longer U5.3 (+)
- net SPI_DAC0 renamed SPI_CS0
- net SPI_DAC1 renamed SPI_CS1
- net SPI_DAC2 renamed SPI_CS2
- net SPI_DAC3 renamed SPI_CS3
- net SPI_DAC4 renamed SPI_CS4
- net SPI_DAC5 renamed SPI_CS5
- net SPI_DAC6 renamed SPI_CS6
- net SPI_DAC7 renamed SPI_CS7
