File: hardware/overcycler2.sch (KiCad schematic (older format))
At the start: 98 parts, among them P1 LPC_P1, P2 LPC_P2, P3 FT232, P4 PANEL, P5 SDCARD, P6 MIDI_IN, P7 FOOT_IN, P8 AC_IN, P9 AUDIO_OUT, Q1 BC547, SW1 RESET, U1 TLV1543, U2 74HCT4051, U3 LTC1660, U4 LTC1660, U5 TL074, U6 TL074, U7 LM1084IT-5.0/NOPB, U8 LM2990-5.0/NOPB, U9 LM1084IT-3.3/NOPB

Commit message: better pcb placement -- sch fixes
Parts:
- removed U9: LM1084IT-3.3/NOPB, TO-220, symbol LM1084IT-3.3/NOPB
- added R126: 220, ~, symbol R
- added R127: 120, ~, symbol R
- added U9: LM1084IT-ADJ/NOPB, TO-220, symbol LM1084IT-ADJ/NOPB
Connections:
- wire segments 339 -> 340
Other:
- moved on the sheet: C24, C25, C26, C27, C28, C29, C30, C33, D6, D7, P8, U7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

Commit message: better pcb placement
Changed lines of the file:
@@
 	1    0    0    -1
 $EndComp
-Text Label 3200 3750 0    60   ~ 0
+Text Label 3200 4150 0    60   ~ 0
 P_0
-Text Label 3200 3850 0    60   ~ 0
+Text Label 3200 4050 0    60   ~ 0
 P_1
 Text Label 3200 3950 0    60   ~ 0
 P_2
-Text Label 3200 4050 0    60   ~ 0
+Text Label 3200 3850 0    60   ~ 0
 P_3
-Text Label 3200 4150 0    60   ~ 0
+Text Label 3200 3750 0    60   ~ 0
 P_4
 Text Label 2050 4550 2    60   ~ 0

Commit message: autorouted pcb
Changed lines of the file:
@@
 	1    0    0    -1
 $EndComp
-Text Label 3200 4150 0    60   ~ 0
+Text Label 3200 3750 0    60   ~ 0
 P_0
-Text Label 3200 4050 0    60   ~ 0
+Text Label 3200 3850 0    60   ~ 0
 P_1
 Text Label 3200 3950 0    60   ~ 0
 P_2
-Text Label 3200 3850 0    60   ~ 0
+Text Label 3200 4050 0    60   ~ 0
 P_3
-Text Label 3200 3750 0    60   ~ 0
+Text Label 3200 4150 0    60   ~ 0
 P_4
 Text Label 2050 4550 2    60   ~ 0

Commit message: board v2 -- dac addressing fixes
Parts:
- removed RR1: 10k, ~, symbol RR8
- removed U2: 74HCT4051, symbol 4051
- added C88: 2u2, ~, symbol CP1
- added R128: 10k, ~, symbol R
- added U2: 74HC138, ~, symbol 74LS138
- C24, C25: value 10000u -> 10000u 16v
Connections:
- wire segments 340 -> 339
Other:
- moved on the sheet: P3, P5, SW1

Commit message: sch/pcb: making the noise generator a lot more resilient to 50hz ripple
Parts:
- added C95: 100u, ~, symbol CP1
- added R129: 10k, ~, symbol R
Connections:
- net -5V: now also R129.2; no longer Q1.2 (B)
- net GND: now also C95.2
- new net: C95.1, Q1.2 (B), R129.1

Commit message: sch/pcb: whoops! one cap was backwards
Connections:
- net GND: now also C95.1; no longer C95.2
- net at Q1.2 (B), R129.1: now also C95.2; no longer C95.1
Changed lines of the file:
@@
 F 3 "~" H 7150 6000 60  0000 C CNN
 	1    7150 6000
-	1    0    0    -1
+	-1   0    0    1
 $EndComp
 $Comp
