File: hardware/overcycler2.sch (KiCad schematic (older format))
At the start: 103 parts, among them P1 LPC_P1, P2 LPC_P2, P3 FT232, P4 PANEL, P5 SDCARD, P6 MIDI_IN, P7 FOOT_IN, P8 AC_IN, P9 AUDIO_OUT, Q1 BC547, SW1 RESET, U1 TLV1543, U2 74HC138, U3 LTC1660, U4 LTC1660, U5 TL074, U6 TL074, U7 LM1084IT-5.0/NOPB, U8 LM2990-5.0/NOPB, U9 LM1084IT-ADJ/NOPB

Commit message: sch: adding notes in case someone wants to build it
Other:
- note added: "1: left master volume to pot\n2: left master volume from pot\n3: master volume ground\n4: right master volume to pot\n5: right master volume from pot\n6: master jacks ground\n7: left master jack\n8: right master jack"
- note added: "All capacitors should be minimum 16V unless specified\nAll polarized capacitors are electrolytic\nAll unpolarised capacitors are film\nAll resistors are 5% 1/4w\nData entry potentiometers are 4.7k linear taper\nMaster volume potentiometer is 47k dual audio taper"
- note added: "Pin 1 is DIN socket pin 4\nPin 2 is DIN socket pin 5"
- note added: "Select Q1 for\n0.3Vpp..0.4Vpp\nof noise at U5.1\nR6 value can be \nadjusted if need be"
- note added: "Solder a microSD to SD adapter using a pin strip\nPins are per SD specifications"
- note added: "Use mininum 7.5VAC 1A power supply\nHigher voltage may overheat the regulators"
Changed lines of the file:
@@
 Wire Wire Line
 	7150 6200 7150 6350
+Text Notes 7500 6150 0    60   ~ 0
+Select Q1 for\n0.3Vpp..0.4Vpp\nof noise at U5.1\nR6 value can be \nadjusted if need be
+Text Notes 12100 6900 0    60   ~ 0
+All capacitors should be minimum 16V unless specified\nAll polarized capacitors are electrolytic\nAll unpolarised capacitors are film\nAll resistors are 5% 1/4w\nData entry potentiometers are 4.7k linear taper\nMaster volume potentiometer is 47k dual audio taper
+Text Notes 14500 5100 0    60   ~ 0
+1: left master volume to pot\n2: left master volume from pot\n3: master volume ground\n4: right master volume to pot\n5: right master volume from pot\n6: master jacks ground\n7: left master jack\n8: right master jack
+Text Notes 5800 1700 0    60   ~ 0
+Pin 1 is DIN socket pin 4\nPin 2 is DIN socket pin 5
+Text Notes 4000 600  0    60   ~ 0
+Solder a microSD to SD adapter using a pin strip\nPins are per SD specifications
+Text Notes 10400 850  0    60   ~ 0
+Use mininum 7.5VAC 1A power supply\nHigher voltage may overheat the regulators
 $EndSCHEMATC

Commit message: pcb r4, one resistor was missing
Parts:
- added R130: 10k, ~, symbol R
Connections:
- net +3.3V: now also R130.1
- net ADC_CLK: now also R130.2

Commit message: hw: fixing unconnected SPI_MOSI/SPI_SCK (pcb r5)
Changed lines of the file:
@@
 Sheet 1 7
 Title "OverCycler 2 full board"
-Date "21 sep 2015"
-Rev "8"
+Date "23 sep 2015"
+Rev "9"
 Comp "GliGli's DIY"
 Comment1 ""
@@
 Text Label 1050 7300 0    60   ~ 0
 SPI_SSEL
-Text Label 1050 7200 0    60   ~ 0
-SPI_SCK
-Text Label 1050 7500 0    60   ~ 0
-SPI_MOSI
 Text Label 6200 2600 0    60   ~ 0
 SPI_CS0
@@
 	1    0    0    -1
 $EndComp
-Text Label 6350 4800 0    60   ~ 0
-SPI_MOSI
-Text Label 4850 4800 2    60   ~ 0
-SPI_SCK
 Text Label 4850 4700 2    60   ~ 0
 SPI_CS6
@@
 	1    0    0    -1
 $EndComp
-Text Label 4850 6000 2    60   ~ 0
-SPI_SCK
 Text Label 4850 5800 2    60   ~ 0
 DAC_VREF
@@
 Text Label 4850 5900 2    60   ~ 0
 SPI_CS7
-Text Label 6350 6000 0    60   ~ 0
-SPI_MOSI
 $Comp
 L R R26
@@
 	4050 4150 4050 4200
 Connection ~ 3650 4150
+Text GLabel 1050 7500 2    39   Output ~ 0
+SPI_MOSI
+Text GLabel 1450 7200 2    39   Output ~ 0
+SPI_SCK
+Wire Wire Line
+	1050 7200 1450 7200
+Text GLabel 4850 4800 0    39   Input ~ 0
+SPI_SCK
+Text GLabel 4850 6000 0    39   Input ~ 0
+SPI_SCK
+Text GLabel 6350 6000 2    39   Input ~ 0
+SPI_MOSI
+Text GLabel 6350 4800 2    39   Input ~ 0
+SPI_MOSI
 $EndSCHEMATC

Commit message: hw: lower value pullup for  ADC_CLK, makes the adc work much better
Parts:
- R130: value 10k -> 1k
Changed lines of the file:
@@
 Sheet 1 7
 Title "OverCycler 2 full board"
-Date "23 sep 2015"
-Rev "9"
+Date "24 sep 2015"
+Rev "10"
 Comp "GliGli's DIY"
 Comment1 ""
@@
 P 4050 4450
 F 0 "R130" V 4130 4450 40  0000 C CNN
-F 1 "10k" V 4057 4451 40  0000 C CNN
+F 1 "1k" V 4057 4451 40  0000 C CNN
 F 2 "~" V 3980 4450 30  0000 C CNN
 F 3 "~" H 4050 4450 30  0000 C CNN

Commit message: hw: adjusted noise generator resistor value
Parts:
- R6: value 47k -> 470k
Changed lines of the file:
@@
 Sheet 1 7
 Title "OverCycler 2 full board"
-Date "26 sep 2015"
-Rev "11"
+Date "27 sep 2015"
+Rev "12"
 Comp "GliGli's DIY"
 Comment1 ""
@@
 P 7750 5050
 F 0 "R6" V 7830 5050 40  0000 C CNN
-F 1 "47k" V 7757 5051 40  0000 C CNN
+F 1 "470k" V 7757 5051 40  0000 C CNN
 F 2 "~" V 7680 5050 30  0000 C CNN
 F 3 "~" H 7750 5050 30  0000 C CNN

Commit message: changed VCNoise level (3M3 diode input res)
Parts:
- R16: value 2M2 -> 3M3
Changed lines of the file:
@@
 EESchema Schematic File Version 2
 LIBS:power
+LIBS:device
+LIBS:transistors
+LIBS:conn
+LIBS:linear
+LIBS:regul
+LIBS:74xx
+LIBS:cmos4000
+LIBS:adc-dac
+LIBS:memory
+LIBS:xilinx
+LIBS:special
+LIBS:microcontrollers
+LIBS:dsp
+LIBS:microchip
+LIBS:analog_switches
+LIBS:motorola
+LIBS:texas
+LIBS:intel
+LIBS:audio
+LIBS:interface
+LIBS:digital-audio
+LIBS:philips
+LIBS:display
+LIBS:cypress
+LIBS:siliconi
+LIBS:opto
+LIBS:atmel
+LIBS:contrib
+LIBS:valves
 LIBS:overcycler2-cache
 EELAYER 27 0
@@
 Sheet 1 7
 Title "OverCycler 2 full board"
-Date "12 jan 2020"
+Date "25 aug 2021"
 Rev "12"
 Comp "GliGli's DIY"
@@
 P 10350 5350
 F 0 "R16" V 10430 5350 40  0000 C CNN
-F 1 "2M2" V 10357 5351 40  0000 C CNN
+F 1 "3M3" V 10357 5351 40  0000 C CNN
 F 2 "~" V 10280 5350 30  0000 C CNN
 F 3 "~" H 10350 5350 30  0000 C CNN
