File: hardware/voice2.sch (KiCad schematic (older format))
At the start: 28 parts, among them IC1 LM13700, U10 MCP4922-E/P, U11 SSM2044

Commit message: adding overcycler2 netlist/cmp/empty pcb
Connections:
- net at C41.2, R47.2, R48.2: now also IC1.16 (Iabc); no longer IC1.1 (Iabc)
- net at R46.2, RV2.1: now also IC1.14 (+); no longer IC1.3 (+)
- net at RV2.3: now also IC1.13 (-); no longer IC1.4 (-)
- net at C42.2, R50.1: now also IC1.9 (buffer_out); no longer IC1.8 (buffer_out)
- new net: IC1.10 (buffer_in), IC1.12 (out), R49.1
