File: hardware/voice2.sch (KiCad schematic (older format))
At the start: 28 parts, among them IC1 LM13700, U10 MCP4922-E/P, U11 SSM2044

Commit message: better pcb routing -- adding slew rate limiter caps for VCF Fc
Parts:
- added C88: 1u, ~, symbol CP1
Connections:
- net GND: now also C88.2
- net at R41.2, R43.2, R45.2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: now also C88.1
- net at C41.2, R47.2, R48.2: now also IC1.16 (Iabc); no longer IC1.1 (Iabc)
- net at R46.2, RV2.1: now also IC1.14 (+); no longer IC1.3 (+)
- net at RV2.3: now also IC1.13 (-); no longer IC1.4 (-)
- net at C42.2, R50.1: now also IC1.9 (buffer_out); no longer IC1.8 (buffer_out)
- new net: IC1.10 (buffer_in), IC1.12 (out), R49.1
Other:
- moved on the sheet: R75

Commit message: board v2 -- dac addressing fixes
Parts:
- removed C88: 1u, ~, symbol CP1
- added C89: 470n, ~, symbol C
Connections:
- net GND: now also C89.2
- net at R41.2, R43.2, R45.2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: now also C89.1

Commit message: sch/pcb: making the noise generator a lot more resilient to 50hz ripple
Connections:
- net at RV2.3: now also IC1.4 (-); no longer IC1.13 (-)
- net at R46.2, RV2.1: now also IC1.3 (+); no longer IC1.14 (+)
- net at C41.2, R47.2, R48.2: now also IC1.1 (Iabc); no longer IC1.16 (Iabc)
- net at C42.2, R50.1: now also IC1.8 (buffer_out); no longer IC1.9 (buffer_out)
- new net: IC1.5 (out), IC1.7 (buffer_in), R49.1

Commit message: now compensating resonance volume loss with the pre-filter mixer -- sch changes to accomodate this before that, cranking up the resonance made the filter/vca lose its overdrive, which was totally counter intuitive
Parts:
- R39, R42: value 220 -> 1k
- R40: value 5k6 -> 22k
Connections:
- net at C41.2, R47.2, R48.2: now also IC1.16 (Iabc); no longer IC1.1 (Iabc)
- net at R46.2, RV2.1: now also IC1.14 (+); no longer IC1.3 (+)
- net at RV2.3: now also IC1.13 (-); no longer IC1.4 (-)
- net at C42.2, R50.1: now also IC1.9 (buffer_out); no longer IC1.8 (buffer_out)
- new net: IC1.10 (buffer_in), IC1.12 (out), R49.1

Commit message: sch: adding notes in case someone wants to build it
Connections:
- net at RV2.3: now also IC1.4 (-); no longer IC1.13 (-)
- net at R46.2, RV2.1: now also IC1.3 (+); no longer IC1.14 (+)
- net at C41.2, R47.2, R48.2: now also IC1.1 (Iabc); no longer IC1.16 (Iabc)
- net at C42.2, R50.1: now also IC1.8 (buffer_out); no longer IC1.9 (buffer_out)
- new net: IC1.5 (out), IC1.7 (buffer_in), R49.1
Other:
- note added: "Adjust RV2 to reduce DC offset at IC1.12\nbetween VCA fully open and fully closed\n(set OscA,OscB,Noise volume to zero)"
- note added: "Notes refer to voice #0, but apply to all other voices too"
- note added: "Use film capacitors for C36..C39,\npreferably within 1% of theoretical value."

Commit message: hw: fixing unconnected SPI_MOSI/SPI_SCK (pcb r5)
Connections:
- net at C41.2, R47.2, R48.2: now also IC1.16 (Iabc); no longer IC1.1 (Iabc)
- net at R46.2, RV2.1: now also IC1.14 (+); no longer IC1.3 (+)
- net at RV2.3: now also IC1.13 (-); no longer IC1.4 (-)
- net at C42.2, R50.1: now also IC1.9 (buffer_out); no longer IC1.8 (buffer_out)
- new net: IC1.10 (buffer_in), IC1.12 (out), R49.1
