File: hardware/voice2.sch (KiCad schematic (older format))
At the start: 29 parts, among them IC1 LM13700, U10 MCP4922-E/P, U11 SSM2044

Commit message: hw: VCF resonance adjumstments
Parts:
- R39, R42: value 1k -> 820
- R40: value 22k -> 15k
Connections:
- net at RV2.3: now also IC1.4 (-); no longer IC1.13 (-)
- net at R46.2, RV2.1: now also IC1.3 (+); no longer IC1.14 (+)
- net at C41.2, R47.2, R48.2: now also IC1.1 (Iabc); no longer IC1.16 (Iabc)
- net at C42.2, R50.1: now also IC1.8 (buffer_out); no longer IC1.9 (buffer_out)
- new net: IC1.5 (out), IC1.7 (buffer_in), R49.1

Commit message: hardware: voice sch clarification
Connections:
- net -5V: now also R45.2; no longer R45.1
- net GND: now also C89.1, R43.2; no longer C89.2, R43.1
- net at C41.2, R47.2, R48.2: now also IC1.16 (Iabc); no longer IC1.1 (Iabc)
- net at R46.2, RV2.1: now also IC1.14 (+); no longer IC1.3 (+)
- net at RV2.3: now also IC1.13 (-); no longer IC1.4 (-)
- net at C42.2, R50.1: now also IC1.9 (buffer_out); no longer IC1.8 (buffer_out)
- new net: C89.2, R41.2, R43.1, R45.1, U11.13 (FREQ_CTL)
- new net: IC1.10 (buffer_in), IC1.12 (out), R49.1
Other:
- moved on the sheet: C41, C89, R39, R41, R43, R45, R47, R48

Commit message: hw: fixed voice tuning note
Connections:
- net at RV2.3: now also IC1.4 (-); no longer IC1.13 (-)
- net at R46.2, RV2.1: now also IC1.3 (+); no longer IC1.14 (+)
- net at C41.2, R47.2, R48.2: now also IC1.1 (Iabc); no longer IC1.16 (Iabc)
- net at C42.2, R50.1: now also IC1.8 (buffer_out); no longer IC1.9 (buffer_out)
- new net: IC1.5 (out), IC1.7 (buffer_in), R49.1
Other:
- note added: "Adjust RV2 to reduce DC offset at IC1.5 or IC1.12\nbetween VCA fully open and fully closed\n(set OscA,OscB,Noise volume to zero)"
- note removed: "Adjust RV2 to reduce DC offset at IC1.12\nbetween VCA fully open and fully closed\n(set OscA,OscB,Noise volume to zero)"
