File: hardware/overcycler2.kicad_pcb (KiCad board)
At the start: 2 copper layers, 215.9 x 152.4 mm, 263 parts, among them IC1 LM13700, IC2 LM13700, IC3 LM13700, P1 LPC_P1, P2 LPC_P2, P3 FT232, P4 PANEL, P5 SDCARD, P6 MIDI_IN, P7 FOOT_IN, P8 AC_IN, P9 AUDIO_OUT, Q1 BC547, SW1 RESET, U1 TLV1543, U10 MCP4922-E/P, U11 SSM2044, U12 MCP4922-E/P, U13 SSM2044, U14 MCP4922-E/P, U15 SSM2044, U16 MCP4922-E/P, U17 SSM2044, U18 MCP4922-E/P, U19 SSM2044, U2 74HCT4051, U20 MCP4922-E/P, U21 SSM2044, U3 LTC1660, U4 LTC1660, U5 TL074, U6 TL074, U7 LM1084IT-5.0/NOPB, U8 LM2990-5.0/NOPB, U9 LM1084IT-3.3/NOPB

Commit message: better pcb placement -- sch fixes
Parts:
- added HOLE1: P***, 1pin, F.Cu at (29.2, 29.2)
- added HOLE2: P***, 1pin, F.Cu at (29.2, 176.5)
- added HOLE3: P***, 1pin, F.Cu at (229.9, 176.5)
- added HOLE4: P***, 1pin, F.Cu at (229.9, 29.2)
- added R126: 220, R3-LARGE_PADS, F.Cu at (34.3, 68.6)
- added R127: 120, R3-LARGE_PADS, F.Cu at (36.2, 61.0)
- U9: value LM1084IT-3.3/NOPB -> LM1084IT-ADJ/NOPB
- moved R10 43.3 mm to (217.8, 110.5), turned to 180 degrees
- moved D5 41.2 mm to (217.8, 126.4), turned to 0 degrees
- moved R17 39.9 mm to (217.8, 129.5), turned to 180 degrees
- moved D4 35.0 mm to (217.8, 123.2), turned to 180 degrees
- moved R4 33.7 mm to (61.6, 170.8)
- moved C13 31.9 mm to (64.8, 172.1)
- moved U3 31.3 mm to (78.1, 170.8)
- moved D3 29.1 mm to (217.8, 120.0), turned to 0 degrees
- moved R15 28.3 mm to (217.8, 113.7), turned to 180 degrees
- moved D2 23.8 mm to (217.8, 116.8), turned to 180 degrees
- moved C5 23.6 mm to (228.0, 112.4), turned to 270 degrees
- moved C19 22.0 mm to (99.1, 151.1), turned to 270 degrees
- moved C14 22.0 mm to (99.1, 30.5), turned to 270 degrees
- moved C15 22.0 mm to (99.1, 54.6), turned to 270 degrees
- moved C16 22.0 mm to (99.1, 78.7), turned to 270 degrees
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Connections:
- P1 pad 4: N-00000116 -> N-0000060
- P2 pad 21: /KP_1_R1 -> /KP_4_R4
- P2 pad 22: /KP_2_R2 -> /KP_3_R3
- P2 pad 23: /KP_3_R3 -> /KP_2_R2
- P2 pad 24: /KP_4_R4 -> /KP_1_R1
- P4 pad 20: /KP_2_R2 -> /KP_5_C1
- P4 pad 21: /KP_3_R3 -> /KP_2_R2
- P4 pad 22: /KP_4_R4 -> /KP_6_C2
- P4 pad 23: /KP_5_C1 -> /KP_3_R3
- P4 pad 24: /KP_6_C2 -> /KP_7_C3
- P4 pad 25: /KP_7_C3 -> /KP_4_R4
- SW1 pad 1: GND -> N-0000060
- SW1 pad 2: N-00000116 -> GND
- U9 pad 1: GND -> N-0000064
Routing:
- added copper zone on B.Cu, net GND
Other:
- board size 215.9 x 152.4 mm -> 208.3 x 154.9 mm
- net class Default: via_dia 1.016 -> 1.27
- net class pwr2: clearance 0.635 -> 0.4826

Commit message: better pcb placement (first full autoroute)
Parts:
- moved C13 22.9 mm to (77.5, 153.0), turned to 180 degrees
- moved U3 16.6 mm to (87.0, 156.8), turned to 90 degrees
- moved U4 12.6 mm to (69.2, 164.5), turned to 90 degrees
- moved R4 11.2 mm to (53.3, 178.4), turned to 0 degrees
- moved C12 6.35 mm to (59.7, 160.7), turned to 180 degrees
- moved C2 4.96 mm to (54.6, 175.3), turned to 180 degrees
- moved C1 3.17 mm to (55.9, 170.8), turned to 180 degrees
- moved C34 2.54 mm to (118.7, 30.5)
- moved C35 2.54 mm to (118.7, 40.6)
- moved C43 2.54 mm to (118.7, 54.6)
- moved C44 2.54 mm to (118.7, 64.8)
- moved C52 2.54 mm to (118.7, 78.7)
- moved C53 2.54 mm to (118.7, 88.9)
- moved C61 2.54 mm to (118.7, 102.9)
- moved C62 2.54 mm to (118.7, 113.0)
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
Commit message: better pcb placement
Parts:
- moved R33 10.6 mm to (220.3, 41.9), turned to 180 degrees
- moved R31 7.67 mm to (220.3, 66.0), turned to 180 degrees
- moved R104 5.39 mm to (158.8, 142.2), turned to 270 degrees
- moved R119 5.39 mm to (158.8, 166.4), turned to 270 degrees
- moved R44 5.39 mm to (158.8, 45.7), turned to 270 degrees
- moved R74 5.39 mm to (158.8, 94.0), turned to 270 degrees
- moved R89 5.39 mm to (158.8, 118.1), turned to 270 degrees
- moved R59 5.39 mm to (158.8, 69.8), turned to 270 degrees
- moved C40 3.81 mm to (175.3, 30.5)
- moved C49 3.81 mm to (175.3, 54.6)
- moved C58 3.81 mm to (175.3, 78.7)
- moved C67 3.81 mm to (175.3, 102.2)
- moved C76 3.81 mm to (175.3, 127.0)
- moved C85 3.81 mm to (175.3, 151.1)
- moved R106 3.81 mm to (185.4, 127.0)
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Connections:
- P4 pad 32: /P_0 -> /P_4
- P4 pad 34: /P_1 -> /P_3
- P4 pad 38: /P_3 -> /P_1
- P4 pad 40: /P_4 -> /P_0

Commit message: autorouted pcb
Parts:
- moved R100 22.5 mm to (160.0, 141.6), turned to 90 degrees
- moved R40 22.5 mm to (160.0, 45.1), turned to 90 degrees
- moved R85 22.5 mm to (160.0, 117.5), turned to 90 degrees
- moved R115 22.5 mm to (160.0, 165.7), turned to 90 degrees
- moved R55 22.4 mm to (160.0, 69.2), turned to 90 degrees
- moved R70 22.4 mm to (160.0, 93.3), turned to 90 degrees
- moved R84 11.7 mm to (127.6, 99.7)
- moved R99 11.7 mm to (127.6, 123.8)
- moved R39 11.7 mm to (127.6, 27.3)
- moved R114 11.7 mm to (127.6, 148.0)
- moved R54 11.7 mm to (127.6, 51.4)
- moved R69 11.7 mm to (127.6, 75.6)
- moved C22 7.24 mm to (62.2, 108.0), turned to 90 degrees
- moved C72 4.07 mm to (160.0, 131.4)
- moved C81 4.07 mm to (160.0, 155.6)
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Connections:
- P4 pad 32: /P_4 -> /P_0
- P4 pad 34: /P_3 -> /P_1
- P4 pad 38: /P_1 -> /P_3
- P4 pad 40: /P_0 -> /P_4
Routing:
- net +5V: track 0.00 -> 983.3 mm
- net -5V: track 0.00 -> 889.3 mm
- net +3.3V: track 0.00 -> 308.8 mm, vias 0 -> 1
- net NOISE: track 0.00 -> 254.6 mm, vias 0 -> 1
- net DAC_RES: track 0.00 -> 251.5 mm
- net DAC_MIXB: track 0.00 -> 232.0 mm
- net /Voice #1/DAC_VCA: track 0.00 -> 196.2 mm, vias 0 -> 1
- net /Voice #2/DAC_VCA: track 0.00 -> 195.7 mm
- net /Voice #0/DAC_VCA: track 0.00 -> 187.2 mm, vias 0 -> 2
- net /DAC_MIXN: track 0.00 -> 179.4 mm
- net DAC_MIXA: track 0.00 -> 178.5 mm
- net /Voice #0/DAC_FC: track 0.00 -> 177.0 mm, vias 0 -> 2
- net /Voice #4/SPI_CS: track 0.00 -> 157.5 mm, vias 0 -> 1
- net /Voice #3/DAC_VCA: track 0.00 -> 144.5 mm, vias 0 -> 1
- net /SPI_CS7: track 0.00 -> 142.9 mm, vias 0 -> 1
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- added copper zone on F.Cu, net GND
Other:
- net class Default: via_dia 1.27 -> 1.524; via_drill 0.508 -> 0.8128
- net class pwr: via_drill 0.508 -> 0.8128
- net class pwr2: via_drill 0.508 -> 0.8128
- board text added: "OverCycler 2 board R1 Bottom"
- board text added: "OverCycler 2 board R1 Top"

Commit message: better pcb routing -- adding slew rate limiter caps for VCF Fc
Parts:
- added C88: 1u, C1V5, F.Cu at (139.1, 40.6)
- added C89: 1u, C1V5, F.Cu at (139.1, 64.8)
- added C90: 1u, C1V5, F.Cu at (139.1, 88.9)
- added C91: 1u, C1V5, F.Cu at (139.1, 113.0)
- added C92: 1u, C1V5, F.Cu at (139.1, 137.2)
- added C93: 1u, C1V5, F.Cu at (139.1, 161.3)
- moved C16 2.54 mm to (101.6, 80.0)
- moved C17 2.54 mm to (101.6, 104.1)
- moved C18 2.54 mm to (101.6, 128.3)
- moved C21 2.54 mm to (66.0, 38.1)
- moved U2 2.54 mm to (79.4, 39.4)
- moved C15 2.54 mm to (101.6, 55.9)
- moved C19 2.54 mm to (101.6, 152.4)
- moved R20 2.54 mm to (220.3, 95.9)
- moved R21 2.54 mm to (220.3, 83.2)
- moved R22 2.54 mm to (220.3, 86.4)
- moved R23 2.54 mm to (220.3, 70.5)
- moved R24 2.54 mm to (220.3, 73.7)
- moved R25 2.54 mm to (220.3, 76.8)
- moved R26 2.54 mm to (220.3, 80.0)
- moved R27 2.54 mm to (220.3, 89.5)
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Routing:
- net +5V: track 983.3 -> 0.00 mm
- net -5V: track 889.3 -> 0.00 mm
- net +3.3V: track 308.8 -> 0.00 mm, vias 1 -> 0
- net NOISE: track 254.6 -> 0.00 mm, vias 1 -> 0
- net DAC_RES: track 251.5 -> 0.00 mm
- net DAC_MIXB: track 232.0 -> 0.00 mm
- net /Voice #1/DAC_VCA: track 196.2 -> 0.00 mm, vias 1 -> 0
- net /Voice #2/DAC_VCA: track 195.7 -> 0.00 mm
- net /Voice #0/DAC_VCA: track 187.2 -> 0.00 mm, vias 2 -> 0
- net /DAC_MIXN: track 179.4 -> 0.00 mm
- net DAC_MIXA: track 178.5 -> 0.00 mm
- net /Voice #0/DAC_FC: track 177.0 -> 0.00 mm, vias 2 -> 0
- net /Voice #4/SPI_CS: track 157.5 -> 0.00 mm, vias 1 -> 0
- net /Voice #3/DAC_VCA: track 144.5 -> 0.00 mm, vias 1 -> 0
- net /SPI_CS7: track 142.9 -> 0.00 mm, vias 1 -> 0
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Other:
- net class Default: trace_width 0.762 -> 0.635; via_dia 1.524 -> 1.651
- net class pwr: via_dia 1.778 -> 1.651
- rule trace_min: 0.254 -> 0.635
- rule via_min_drill: 0.508 -> 0.762
- rule via_min_size: 0.889 -> 1.651

Commit message: board v2 -- dac addressing fixes
Parts:
- removed RR1: 10k, SIL-9
- added C94: 470n, C2, F.Cu at (138.4, 160.7)
- added R128: 10k, R3-LARGE_PADS, F.Cu at (65.4, 42.5)
- C24, C25: value 10000u -> 10000u 16v
- C88: value 1u -> 2u2
- C89, C90, C91, C92, C93: value 1u -> 470n; footprint C1V5 -> C2
- U2: value 74HCT4051 -> 74HC138
- moved C88 79.6 mm to (59.7, 46.4)
- moved C90 24.8 mm to (138.4, 64.1)
- moved C91 24.8 mm to (138.4, 88.3)
- moved C92 24.8 mm to (138.4, 112.4)
- moved C89 24.8 mm to (138.4, 40.0)
- moved C93 24.8 mm to (138.4, 136.5)
- moved R40 21.6 mm to (139.7, 47.0), turned to 0 degrees
- moved R55 21.6 mm to (139.7, 71.1), turned to 0 degrees
- moved R70 21.6 mm to (139.7, 95.2), turned to 0 degrees
- moved R85 21.6 mm to (139.7, 119.4), turned to 0 degrees
- moved R100 21.6 mm to (139.7, 143.5), turned to 0 degrees
- moved R115 21.6 mm to (139.7, 167.6), turned to 0 degrees
- moved U4 20.5 mm to (87.0, 154.3)
- moved U3 18.5 mm to (69.2, 161.9)
- moved SW1 15.4 mm to (59.7, 38.7), turned to 90 degrees
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Connections:
- C88 pad 1: N-00000173 -> N-0000070
- C89 pad 1: N-00000200 -> N-00000173
- C90 pad 1: N-00000223 -> N-00000200
- C91 pad 1: N-00000247 -> N-00000223
- C92 pad 1: N-00000271 -> N-00000247
- C93 pad 1: N-00000295 -> N-00000271
- P1 pad 4: N-0000060 (its old number) -> N-0000070
- SW1 pad 1: N-0000060 (its old number) -> GND
- SW1 pad 2: GND -> N-0000070
- U2 pad 1: /Voice #4/SPI_CS -> /SPI_MUX_A
- U2 pad 10: /SPI_MUX_B -> /Voice #5/SPI_CS
- U2 pad 11: /SPI_MUX_A -> /Voice #4/SPI_CS
- U2 pad 13: /Voice #0/SPI_CS -> /Voice #2/SPI_CS
- U2 pad 15: /Voice #2/SPI_CS -> /Voice #0/SPI_CS
- U2 pad 2: /SPI_CS6 -> /SPI_MUX_B
- U2 pad 3: /SPI_SSEL -> /SPI_MUX_C
- U2 pad 4: /SPI_CS7 -> /SPI_SSEL
- U2 pad 5: /Voice #5/SPI_CS -> GND
- U2 pad 6: GND -> +3.3V
- U2 pad 7: GND -> /SPI_CS7
- U2 pad 9: /SPI_MUX_C -> /SPI_CS6
- U3 pad 14: DAC_MIXA -> /DAC_MIXN
- U3 pad 15: DAC_MIXB -> DAC_RES
- U4 pad 14: /DAC_MIXN -> DAC_MIXA
- U4 pad 15: DAC_RES -> DAC_MIXB
Routing:
- net +5V: track 0.00 -> 993.5 mm, vias 0 -> 1
- net -5V: track 0.00 -> 746.8 mm
- net +3.3V: track 0.00 -> 288.0 mm, vias 0 -> 2
- net NOISE: track 0.00 -> 265.1 mm
- net /Voice #0/DAC_VCA: track 0.00 -> 227.2 mm
- net DAC_RES: track 0.00 -> 221.2 mm, vias 0 -> 1
- net DAC_MIXA: track 0.00 -> 202.8 mm
- net /Voice #2/DAC_VCA: track 0.00 -> 196.1 mm
- net /Voice #1/DAC_VCA: track 0.00 -> 191.8 mm
- net /DAC_MIXN: track 0.00 -> 183.1 mm
- net DAC_MIXB: track 0.00 -> 177.7 mm, vias 0 -> 2
- net /LCD_DB4: track 0.00 -> 168.6 mm
- net /SPI_CS6: track 0.00 -> 160.7 mm, vias 0 -> 3
- net /Voice #0/DAC_FC: track 0.00 -> 160.0 mm
- net /Voice #1/DAC_FC: track 0.00 -> 159.1 mm, vias 0 -> 3
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Other:
- board size 208.3 x 154.9 mm -> 208.3 x 151.1 mm
- board text added: "OverCycler 2 board R2 Bottom"
- board text added: "OverCycler 2 board R2 Top"
- board text removed: "OverCycler 2 board R1 Bottom"
- board text removed: "OverCycler 2 board R1 Top"

Commit message: pcb: back to square one, can't rely on gound plane
Parts:
- moved C21 20.9 mm to (90.8, 43.8), turned to 0 degrees
- moved C12 16.9 mm to (69.2, 172.1), turned to 0 degrees
- moved C13 16.9 mm to (87.0, 164.5), turned to 0 degrees
- moved R32 9.88 mm to (223.5, 38.1), turned to 180 degrees
- moved C22 7.85 mm to (54.6, 106.0), turned to 180 degrees
- moved R30 7.62 mm to (227.3, 55.2), turned to 270 degrees
- moved RV1 6.48 mm to (36.8, 106.0), turned to 180 degrees
- moved U3 3.18 mm to (69.2, 158.8)
- moved U4 3.18 mm to (87.0, 151.1)
- moved C15 1.27 mm to (102.9, 55.9)
- moved C16 1.27 mm to (102.9, 80.0)
- moved C17 1.27 mm to (102.9, 104.1)
- moved C18 1.27 mm to (102.9, 128.3)
- moved C19 1.27 mm to (102.9, 152.4)
- moved C34 1.27 mm to (118.7, 30.5)
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Routing:
- net +5V: track 993.5 -> 0.00 mm, vias 1 -> 0
- net -5V: track 746.8 -> 0.00 mm
- net +3.3V: track 288.0 -> 0.00 mm, vias 2 -> 0
- net NOISE: track 265.1 -> 0.00 mm
- net /Voice #0/DAC_VCA: track 227.2 -> 0.00 mm
- net DAC_RES: track 221.2 -> 0.00 mm, vias 1 -> 0
- net DAC_MIXA: track 202.8 -> 0.00 mm
- net /Voice #2/DAC_VCA: track 196.1 -> 0.00 mm
- net /Voice #1/DAC_VCA: track 191.8 -> 0.00 mm
- net /DAC_MIXN: track 183.1 -> 0.00 mm
- net DAC_MIXB: track 177.7 -> 0.00 mm, vias 2 -> 0
- net /LCD_DB4: track 168.6 -> 0.00 mm
- net /SPI_CS6: track 160.7 -> 0.00 mm, vias 3 -> 0
- net /Voice #0/DAC_FC: track 160.0 -> 0.00 mm
- net /Voice #1/DAC_FC: track 159.1 -> 0.00 mm, vias 3 -> 0
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- removed copper zone on B.Cu, net GND
- removed copper zone on F.Cu, net GND
Other:
- board size 208.3 x 151.1 mm -> 208.3 x 152.4 mm
- rule trace_min: 0.635 -> 0.025
- rule via_min_size: 1.651 -> 0.065
- board text added: "OverCycler 2 board R2 bottom"
- board text added: "OverCycler 2 board R2 top"
- board text removed: "OverCycler 2 board R2 Bottom"
- board text removed: "OverCycler 2 board R2 Top"

Commit message: rev3 pcb
Parts:
- moved R122 19.0 mm to (174.6, 148.0)
- moved C10 18.4 mm to (195.6, 132.1), turned to 90 degrees
- moved R92 17.8 mm to (174.6, 101.0)
- moved C8 17.5 mm to (195.6, 85.1), turned to 90 degrees
- moved C49 17.0 mm to (182.9, 69.8)
- moved C6 16.7 mm to (195.6, 38.1), turned to 90 degrees
- moved R62 16.5 mm to (174.6, 54.0)
- moved C67 16.5 mm to (182.9, 116.8)
- moved R124 15.9 mm to (193.0, 154.9), turned to 270 degrees
- moved R94 15.3 mm to (193.0, 108.0), turned to 270 degrees
- moved R64 14.9 mm to (193.0, 61.0), turned to 270 degrees
- moved C85 14.8 mm to (182.9, 163.8)
- moved R79 14.5 mm to (193.0, 86.4), turned to 90 degrees
- moved R109 14.3 mm to (193.0, 133.3), turned to 90 degrees
- moved C7 13.9 mm to (195.6, 62.2), turned to 90 degrees
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Routing:
- net GND: track 0.00 -> 1701.5 mm, vias 0 -> 3
- net +5V: track 0.00 -> 1051.7 mm, vias 0 -> 3
- net -5V: track 0.00 -> 873.3 mm, vias 0 -> 3
- net +3.3V: track 0.00 -> 264.0 mm, vias 0 -> 2
- net NOISE: track 0.00 -> 262.7 mm
- net /Voice #0/DAC_VCA: track 0.00 -> 222.2 mm, vias 0 -> 1
- net DAC_RES: track 0.00 -> 217.0 mm, vias 0 -> 2
- net /Voice #1/DAC_VCA: track 0.00 -> 213.1 mm, vias 0 -> 1
- net DAC_MIXA: track 0.00 -> 182.6 mm
- net /Voice #5/DAC_VCA: track 0.00 -> 176.2 mm
- net /Voice #2/DAC_VCA: track 0.00 -> 171.8 mm, vias 0 -> 1
- net DAC_MIXB: track 0.00 -> 165.1 mm
- net /Voice #3/DAC_VCA: track 0.00 -> 163.6 mm, vias 0 -> 1
- net /DAC_MIXN: track 0.00 -> 162.5 mm
- net /Voice #0/DAC_FC: track 0.00 -> 154.7 mm, vias 0 -> 1
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Other:
- board text added: "OverCycler 2 board R3 bottom"
- board text added: "OverCycler 2 board R3 top"
- board text removed: "OverCycler 2 board R2 bottom"
- board text removed: "OverCycler 2 board R2 top"
