File: hardware/overcycler2.kicad_pcb (KiCad board)
At the start: 2 copper layers, 208.3 x 152.4 mm, 276 parts, among them IC1 LM13700, IC2 LM13700, IC3 LM13700, P1 LPC_P1, P2 LPC_P2, P3 FT232, P4 PANEL, P5 SDCARD, P6 MIDI_IN, P7 FOOT_IN, P8 AC_IN, P9 AUDIO_OUT, Q1 BC547, SW1 RESET, U1 TLV1543, U10 MCP4922-E/P, U11 SSM2044, U12 MCP4922-E/P, U13 SSM2044, U14 MCP4922-E/P, U15 SSM2044, U16 MCP4922-E/P, U17 SSM2044, U18 MCP4922-E/P, U19 SSM2044, U2 74HC138, U20 MCP4922-E/P, U21 SSM2044, U3 LTC1660, U4 LTC1660, U5 TL074, U6 TL074, U7 LM1084IT-5.0/NOPB, U8 LM2990-5.0/NOPB, U9 LM1084IT-ADJ/NOPB

Commit message: pcb r3 ok!
Parts:
- moved C12 1.69 mm to (70.5, 173.2)
- moved R4 0.95 mm to (55.9, 169.9)
Routing:
- net GND: track 1701.5 -> 1723.9 mm, vias 3 -> 4
- net +5V: track 1051.7 -> 1056.2 mm, vias 3 -> 4
- net /LCD_DB4: track 103.0 -> 107.0 mm
- net /DAC_VREF: track 78.6 -> 75.5 mm
- net DAC_RES: track 217.0 -> 219.1 mm
- net N-0000081: track 51.3 -> 52.7 mm
- net /LCD_RW: track 88.0 -> 89.2 mm
- net /DAC_MIXN: track 162.5 -> 161.9 mm
- added copper zone on B.Cu, net GND
- added copper zone on F.Cu, net GND

Commit message: sch/pcb: making the noise generator a lot more resilient to 50hz ripple
Parts:
- added C95: 100u, C1.5V8V, F.Cu at (228.0, 128.0)
- added R129: 10k, R3-LARGE_PADS, F.Cu at (224.2, 170.2)
- moved C23 8.10 mm to (228.0, 118.3)
- moved C5 3.81 mm to (228.0, 108.6), turned to 90 degrees
- moved R19 3.24 mm to (224.8, 137.2)
- moved Q1 3.18 mm to (229.9, 167.6)
Connections:
- Q1 pad 2: -5V -> N-0000064
Routing:
- net N-0000064: track 0.00 -> 43.9 mm
- net N-000003: track 15.3 -> 23.4 mm
- net GND: track 1723.9 -> 1727.9 mm
- net N-0000031: track 9.94 -> 13.1 mm
- net -5V: track 873.3 -> 876.4 mm
- net N-000002: track 7.67 -> 5.71 mm
- net NOISE: track 262.7 -> 261.1 mm

Commit message: sch/pcb: whoops! one cap was backwards
Parts:
- turned C95 to 270 degrees
Connections:
- C95 pad 1: N-0000064 -> GND
- C95 pad 2: GND -> N-0000064
Changed lines of the file:
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@@
   )
   (module C1.5V8V (layer F.Cu)
-    (at 227.965 127.9525 90)
-    (fp_text reference C95 (at 0 2.286 90) (layer F.SilkS)
+    (at 227.965 127.9525 270)
+    (fp_text reference C95 (at 0 2.286 270) (layer F.SilkS)
       (effects (font (size 1.016 1.016) (thickness 0.2032)))
     )
-    (fp_text value 100u (at 0 -2.286 90) (layer F.SilkS)
+    (fp_text value 100u (at 0 -2.286 270) (layer F.SilkS)
       (effects (font (size 1.016 1.016) (thickness 0.2032)))
     )
-    (fp_text user + (at -3.429 -0.127 90) (layer F.SilkS)
+    (fp_text user + (at -3.429 -0.127 270) (layer F.SilkS)
       (effects (font (size 1.524 1.524) (thickness 0.3048)))
     )
     (fp_circle (center 0 0) (end 0 4.445) (layer F.SilkS) (width 0.381))
-    (pad 1 thru_hole rect (at -1.905 0 90) (size 1.524 1.524) (drill 0.8128)
+    (pad 1 thru_hole rect (at -1.905 0 270) (size 1.524 1.524) (drill 0.8128)
+      (layers *.Cu *.Mask F.SilkS)
+      (net 77 GND)
+    )
+    (pad 2 thru_hole circle (at 1.905 0 270) (size 1.651 1.651) (drill 0.8128)
       (layers *.Cu *.Mask F.SilkS)
       (net 244 N-0000064)
-    )
-    (pad 2 thru_hole circle (at 1.905 0 90) (size 1.651 1.651) (drill 0.8128)
-      (layers *.Cu *.Mask F.SilkS)
-      (net 77 GND)
     )
     (model discret/c_vert_c1v8.wrl
@@
   (segment (start 130.6692 159.4808) (end 122.9194 167.2306) (width 0.635) (layer B.Cu) (net 76))
   (segment (start 116.68125 173.03865) (end 122.4893 167.2306) (width 0.635) (layer F.Cu) (net 76))
-  (segment (start 227.965 126.0475) (end 230.98125 126.0475) (width 1.524) (layer F.Cu) (net 77))
   (segment (start 227.965 106.68) (end 230.98125 109.69625) (width 1.524) (layer F.Cu) (net 77))
   (segment (start 230.98125 148.11375) (end 227.965 151.13) (width 1.524) (layer F.Cu) (net 77))
-  (segment (start 230.98125 109.69625) (end 230.98125 126.0475) (width 1.524) (layer F.Cu) (net 77))
-  (segment (start 230.98125 126.0475) (end 230.98125 148.11375) (width 1.524) (layer F.Cu) (net 77))
   (segment (start 210.97875 108.55325) (end 211.0105 108.55325) (width 1.524) (layer B.Cu) (net 77))
   (segment (start 212.88375 106.68) (end 227.965 106.68) (width 1.524) (layer B.Cu) (net 77))
@@
   (segment (start 28.473 90.1881) (end 28.473 86.2343) (width 1.524) (layer B.Cu) (net 77))
   (segment (start 29.7249 91.44) (end 28.473 90.1881) (width 1.524) (layer B.Cu) (net 77))
+  (segment (start 227.965 126.0475) (end 230.98125 126.0475) (width 1.524) (layer F.Cu) (net 77))
+  (segment (start 230.98125 109.69625) (end 230.98125 126.0475) (width 1.524) (layer F.Cu) (net 77))
+  (segment (start 230.98125 126.0475) (end 230.98125 148.11375) (width 1.524) (layer F.Cu) (net 77))
   (segment (start 221.615 110.49) (end 227.965 110.49) (width 0.635) (layer B.Cu) (net 78))
   (segment (start 226.4356 162.8194) (end 227.965 161.29) (width 0.635) (layer F.Cu) (net 79))
@@
   (segment (start 68.344 70.721) (end 68.344 35.4796) (width 0.635) (layer F.Cu) (net 243))
   (segment (start 65.405 73.66) (end 68.344 70.721) (width 0.635) (layer F.Cu) (net 243))
+  (segment (start 227.965 129.8575) (end 227.965 139.7) (width 0.635) (layer B.Cu) (net 244))
+  (segment (start 227.965 139.7) (end 231.775 143.51) (width 0.635) (layer B.Cu) (net 244))
   (segment (start 224.155 166.37) (end 228.6 166.37) (width 0.635) (layer B.Cu) (net 244))
-  (segment (start 227.965 129.8575) (end 227.965 139.7) (width 0.635) (layer B.Cu) (net 244))
   (segment (start 231.775 163.195) (end 228.6 166.37) (width 0.635) (layer B.Cu) (net 244))
   (segment (start 231.775 143.51) (end 231.775 163.195) (width 0.635) (layer B.Cu) (net 244))
-  (segment (start 227.965 139.7) (end 231.775 143.51) (width 0.635) (layer B.Cu) (net 244))
   (segment (start 62.23 42.545) (end 62.23 34.925) (width 0.635) (layer F.Cu) (net 245))
   (segment (start 60.96 53.975) (end 60.96 46.355) (width 0.635) (layer F.Cu) (net 245))

Commit message: now compensating resonance volume loss with the pre-filter mixer -- sch changes to accomodate this before that, cranking up the resonance made the filter/vca lose its overdrive, which was totally counter intuitive
Parts:
- R100, R115, R40, R55, R70, R85: value 5k6 -> 22k
- R102, R114, R117, R39, R42, R54, R57, R69, R72, R84, R87, R99: value 220 -> 1k
Changed lines of the file:
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@@
       (effects (font (size 1.397 1.27) (thickness 0.2032)))
     )
-    (fp_text value 220 (at 0 0) (layer F.SilkS) hide
+    (fp_text value 1k (at 0 0) (layer F.SilkS) hide
       (effects (font (size 1.397 1.27) (thickness 0.2032)))
     )
@@
       (effects (font (size 1.397 1.27) (thickness 0.2032)))
     )
-    (fp_text value 5k6 (at 0 0) (layer F.SilkS) hide
+    (fp_text value 22k (at 0 0) (layer F.SilkS) hide
       (effects (font (size 1.397 1.27) (thickness 0.2032)))
     )
@@
       (effects (font (size 1.397 1.27) (thickness 0.2032)))
     )
-    (fp_text value 220 (at 0 0) (layer F.SilkS) hide
+    (fp_text value 1k (at 0 0) (layer F.SilkS) hide
       (effects (font (size 1.397 1.27) (thickness 0.2032)))
     )
@@
       (effects (font (size 1.397 1.27) (thickness 0.2032)))
     )
-    (fp_text value 220 (at 0 0) (layer F.SilkS) hide
+    (fp_text value 1k (at 0 0) (layer F.SilkS) hide
       (effects (font (size 1.397 1.27) (thickness 0.2032)))
     )
@@
       (effects (font (size 1.397 1.27) (thickness 0.2032)))
     )
-    (fp_text value 5k6 (at 0 0) (layer F.SilkS) hide
+    (fp_text value 22k (at 0 0) (layer F.SilkS) hide
       (effects (font (size 1.397 1.27) (thickness 0.2032)))
     )
@@
       (effects (font (size 1.397 1.27) (thickness 0.2032)))
     )
-    (fp_text value 220 (at 0 0) (layer F.SilkS) hide
+    (fp_text value 1k (at 0 0) (layer F.SilkS) hide
       (effects (font (size 1.397 1.27) (thickness 0.2032)))
     )
@@
       (effects (font (size 1.397 1.27) (thickness 0.2032)))
     )
-    (fp_text value 220 (at 0 0) (layer F.SilkS) hide
+    (fp_text value 1k (at 0 0) (layer F.SilkS) hide
       (effects (font (size 1.397 1.27) (thickness 0.2032)))
     )
@@
       (effects (font (size 1.397 1.27) (thickness 0.2032)))
     )
-    (fp_text value 220 (at 0 0) (layer F.SilkS) hide
+    (fp_text value 1k (at 0 0) (layer F.SilkS) hide
       (effects (font (size 1.397 1.27) (thickness 0.2032)))
     )
@@
       (effects (font (size 1.397 1.27) (thickness 0.2032)))
     )
-    (fp_text value 5k6 (at 0 0) (layer F.SilkS) hide
+    (fp_text value 22k (at 0 0) (layer F.SilkS) hide
       (effects (font (size 1.397 1.27) (thickness 0.2032)))
     )
@@
       (effects (font (size 1.397 1.27) (thickness 0.2032)))
     )
-    (fp_text value 220 (at 0 0) (layer F.SilkS) hide
+    (fp_text value 1k (at 0 0) (layer F.SilkS) hide
       (effects (font (size 1.397 1.27) (thickness 0.2032)))
     )
@@
       (effects (font (size 1.397 1.27) (thickness 0.2032)))
     )
-    (fp_text value 5k6 (at 0 0) (layer F.SilkS) hide
+    (fp_text value 22k (at 0 0) (layer F.SilkS) hide
       (effects (font (size 1.397 1.27) (thickness 0.2032)))
     )
@@
       (effects (font (size 1.397 1.27) (thickness 0.2032)))
     )
-    (fp_text value 220 (at 0 0) (layer F.SilkS) hide
+    (fp_text value 1k (at 0 0) (layer F.SilkS) hide
       (effects (font (size 1.397 1.27) (thickness 0.2032)))
     )
@@
       (effects (font (size 1.397 1.27) (thickness 0.2032)))
     )
-    (fp_text value 220 (at 0 0) (layer F.SilkS) hide
+    (fp_text value 1k (at 0 0) (layer F.SilkS) hide
       (effects (font (size 1.397 1.27) (thickness 0.2032)))
     )
@@
       (effects (font (size 1.397 1.27) (thickness 0.2032)))
     )
-    (fp_text value 220 (at 0 0) (layer F.SilkS) hide
+    (fp_text value 1k (at 0 0) (layer F.SilkS) hide
       (effects (font (size 1.397 1.27) (thickness 0.2032)))
     )
@@
       (effects (font (size 1.397 1.27) (thickness 0.2032)))
     )
-    (fp_text value 220 (at 0 0) (layer F.SilkS) hide
+    (fp_text value 1k (at 0 0) (layer F.SilkS) hide
       (effects (font (size 1.397 1.27) (thickness 0.2032)))
     )
@@
       (effects (font (size 1.397 1.27) (thickness 0.2032)))
     )
-    (fp_text value 5k6 (at 0 0) (layer F.SilkS) hide
+    (fp_text value 22k (at 0 0) (layer F.SilkS) hide
       (effects (font (size 1.397 1.27) (thickness 0.2032)))
     )
@@
       (effects (font (size 1.397 1.27) (thickness 0.2032)))
     )
-    (fp_text value 5k6 (at 0 0) (layer F.SilkS) hide
+    (fp_text value 22k (at 0 0) (layer F.SilkS) hide
       (effects (font (size 1.397 1.27) (thickness 0.2032)))
     )
@@
       (effects (font (size 1.397 1.27) (thickness 0.2032)))
     )
-    (fp_text value 220 (at 0 0) (layer F.SilkS) hide
+    (fp_text value 1k (at 0 0) (layer F.SilkS) hide
       (effects (font (size 1.397 1.27) (thickness 0.2032)))
     )

Commit message: pcb r4, one resistor was missing
Parts:
- added R130: 10k, R3-LARGE_PADS, F.Cu at (61.0, 94.1)
Routing:
- net +3.3V: track 264.0 -> 270.9 mm
- net /ADC_CLK: track 52.5 -> 53.4 mm
Other:
- board text added: "OverCycler 2 board R4 bottom"
- board text added: "OverCycler 2 board R4 top"
- board text removed: "OverCycler 2 board R3 bottom"
- board text removed: "OverCycler 2 board R3 top"
