File: hardware/overcycler2.kicad_pcb (KiCad board)
At the start: 2 copper layers, 208.3 x 152.4 mm, 279 parts, among them IC1 LM13700, IC2 LM13700, IC3 LM13700, P1 LPC_P1, P2 LPC_P2, P3 FT232, P4 PANEL, P5 SDCARD, P6 MIDI_IN, P7 FOOT_IN, P8 AC_IN, P9 AUDIO_OUT, Q1 BC547, SW1 RESET, U1 TLV1543, U10 MCP4922-E/P, U11 SSM2044, U12 MCP4922-E/P, U13 SSM2044, U14 MCP4922-E/P, U15 SSM2044, U16 MCP4922-E/P, U17 SSM2044, U18 MCP4922-E/P, U19 SSM2044, U2 74HC138, U20 MCP4922-E/P, U21 SSM2044, U3 LTC1660, U4 LTC1660, U5 TL074, U6 TL074, U7 LM1084IT-5.0/NOPB, U8 LM2990-5.0/NOPB, U9 LM1084IT-ADJ/NOPB

Commit message: pcb r4 cleanup
Routing:
- net /ADC_CLK: vias 1 -> 0
Changed lines of the file:
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@@
     (links 662)
     (no_connects 0)
-    (area 25.349999 25.349999 233.730001 177.850001)
+    (area 20.935245 24.638 246.251785 177.9016)
     (thickness 1.6)
     (drawings 8)
-    (tracks 2183)
+    (tracks 2182)
     (zones 0)
     (modules 279)
@@
   (gr_line (start 25.4 176.53) (end 25.4 25.4) (angle 90) (layer Edge.Cuts) (width 0.1))
   (gr_line (start 233.68 25.4) (end 233.68 176.53) (angle 90) (layer Edge.Cuts) (width 0.1))
-  (gr_text "OverCycler 2 board R4 top" (at 228.6 87.15375 90) (layer F.Cu)
+  (gr_text "OverCycler 2 board R4 top" (at 230.02875 87.15375 90) (layer F.Cu)
     (effects (font (size 2.5 1.5) (thickness 0.375)))
   )
-  (gr_text "OverCycler 2 board R4 bottom" (at 228.6 85.24875 90) (layer B.Cu)
+  (gr_text "OverCycler 2 board R4 bottom" (at 230.02875 85.24875 90) (layer B.Cu)
     (effects (font (size 2.5 1.5) (thickness 0.375)) (justify mirror))
   )
@@
   (segment (start 59.113 101.9175) (end 59.113 99.79575) (width 0.635) (layer F.Cu) (net 6))
   (segment (start 59.113 99.79575) (end 60.96 97.94875) (width 0.635) (layer F.Cu) (net 6))
-  (via (at 60.96 97.94875) (size 1.651) (layers F.Cu B.Cu) (net 6))
   (segment (start 60.96 97.94875) (end 61.11875 97.79) (width 0.635) (layer B.Cu) (net 6))
   (segment (start 61.11875 97.79) (end 64.135 97.79) (width 0.635) (layer B.Cu) (net 6))

Commit message: hw: fixing unconnected SPI_MOSI/SPI_SCK (pcb r5)
Connections:
- P2 pad 30: /SPI_SCK -> SPI_SCK
- P2 pad 33: /SPI_MOSI -> SPI_MOSI
- U3 pad 8: /SPI_SCK -> SPI_SCK
- U3 pad 9: /SPI_MOSI -> SPI_MOSI
- U4 pad 8: /SPI_SCK -> SPI_SCK
- U4 pad 9: /SPI_MOSI -> SPI_MOSI
Routing:
- net SPI_SCK: track 139.4 -> 201.4 mm
- net SPI_MOSI: track 134.8 -> 188.9 mm
- net /SPI_SCK: track 40.8 -> 0.00 mm
- net /SPI_MOSI: track 35.8 -> 0.00 mm
- net /SPI_CS6: track 134.1 -> 140.3 mm
- net +5V: track 1056.2 -> 1054.9 mm
Other:
- board text added: "OverCycler 2 board R5 bottom"
- board text added: "OverCycler 2 board R5 top"
- board text removed: "OverCycler 2 board R4 bottom"
- board text removed: "OverCycler 2 board R4 top"

Commit message: hw: lower value pullup for  ADC_CLK, makes the adc work much better
Parts:
- R130: value 10k -> 1k
Changed lines of the file:
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@@
       (effects (font (size 1.397 1.27) (thickness 0.2032)))
     )
-    (fp_text value 10k (at 0 0 270) (layer F.SilkS) hide
+    (fp_text value 1k (at 0 0 270) (layer F.SilkS) hide
       (effects (font (size 1.397 1.27) (thickness 0.2032)))
     )

Commit message: hw: VCF resonance adjumstments
Parts:
- R100, R115, R40, R55, R70, R85: value 22k -> 15k
- R102, R114, R117, R39, R42, R54, R57, R69, R72, R84, R87, R99: value 1k -> 820
Changed lines of the file:
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@@
       (effects (font (size 1.397 1.27) (thickness 0.2032)))
     )
-    (fp_text value 1k (at 0 0) (layer F.SilkS) hide
+    (fp_text value 820 (at 0 0) (layer F.SilkS) hide
       (effects (font (size 1.397 1.27) (thickness 0.2032)))
     )
@@
       (effects (font (size 1.397 1.27) (thickness 0.2032)))
     )
-    (fp_text value 22k (at 0 0) (layer F.SilkS) hide
+    (fp_text value 15k (at 0 0) (layer F.SilkS) hide
       (effects (font (size 1.397 1.27) (thickness 0.2032)))
     )
@@
       (effects (font (size 1.397 1.27) (thickness 0.2032)))
     )
-    (fp_text value 1k (at 0 0) (layer F.SilkS) hide
+    (fp_text value 820 (at 0 0) (layer F.SilkS) hide
       (effects (font (size 1.397 1.27) (thickness 0.2032)))
     )
@@
       (effects (font (size 1.397 1.27) (thickness 0.2032)))
     )
-    (fp_text value 1k (at 0 0) (layer F.SilkS) hide
+    (fp_text value 820 (at 0 0) (layer F.SilkS) hide
       (effects (font (size 1.397 1.27) (thickness 0.2032)))
     )
@@
       (effects (font (size 1.397 1.27) (thickness 0.2032)))
     )
-    (fp_text value 22k (at 0 0) (layer F.SilkS) hide
+    (fp_text value 15k (at 0 0) (layer F.SilkS) hide
       (effects (font (size 1.397 1.27) (thickness 0.2032)))
     )
@@
       (effects (font (size 1.397 1.27) (thickness 0.2032)))
     )
-    (fp_text value 1k (at 0 0) (layer F.SilkS) hide
+    (fp_text value 820 (at 0 0) (layer F.SilkS) hide
       (effects (font (size 1.397 1.27) (thickness 0.2032)))
     )
@@
       (effects (font (size 1.397 1.27) (thickness 0.2032)))
     )
-    (fp_text value 1k (at 0 0) (layer F.SilkS) hide
+    (fp_text value 820 (at 0 0) (layer F.SilkS) hide
       (effects (font (size 1.397 1.27) (thickness 0.2032)))
     )
@@
       (effects (font (size 1.397 1.27) (thickness 0.2032)))
     )
-    (fp_text value 1k (at 0 0) (layer F.SilkS) hide
+    (fp_text value 820 (at 0 0) (layer F.SilkS) hide
       (effects (font (size 1.397 1.27) (thickness 0.2032)))
     )
@@
       (effects (font (size 1.397 1.27) (thickness 0.2032)))
     )
-    (fp_text value 22k (at 0 0) (layer F.SilkS) hide
+    (fp_text value 15k (at 0 0) (layer F.SilkS) hide
       (effects (font (size 1.397 1.27) (thickness 0.2032)))
     )
@@
       (effects (font (size 1.397 1.27) (thickness 0.2032)))
     )
-    (fp_text value 1k (at 0 0) (layer F.SilkS) hide
+    (fp_text value 820 (at 0 0) (layer F.SilkS) hide
       (effects (font (size 1.397 1.27) (thickness 0.2032)))
     )
@@
       (effects (font (size 1.397 1.27) (thickness 0.2032)))
     )
-    (fp_text value 22k (at 0 0) (layer F.SilkS) hide
+    (fp_text value 15k (at 0 0) (layer F.SilkS) hide
       (effects (font (size 1.397 1.27) (thickness 0.2032)))
     )
@@
       (effects (font (size 1.397 1.27) (thickness 0.2032)))
     )
-    (fp_text value 1k (at 0 0) (layer F.SilkS) hide
+    (fp_text value 820 (at 0 0) (layer F.SilkS) hide
       (effects (font (size 1.397 1.27) (thickness 0.2032)))
     )
@@
       (effects (font (size 1.397 1.27) (thickness 0.2032)))
     )
-    (fp_text value 1k (at 0 0) (layer F.SilkS) hide
+    (fp_text value 820 (at 0 0) (layer F.SilkS) hide
       (effects (font (size 1.397 1.27) (thickness 0.2032)))
     )
@@
       (effects (font (size 1.397 1.27) (thickness 0.2032)))
     )
-    (fp_text value 1k (at 0 0) (layer F.SilkS) hide
+    (fp_text value 820 (at 0 0) (layer F.SilkS) hide
       (effects (font (size 1.397 1.27) (thickness 0.2032)))
     )
@@
       (effects (font (size 1.397 1.27) (thickness 0.2032)))
     )
-    (fp_text value 1k (at 0 0) (layer F.SilkS) hide
+    (fp_text value 820 (at 0 0) (layer F.SilkS) hide
       (effects (font (size 1.397 1.27) (thickness 0.2032)))
     )
@@
       (effects (font (size 1.397 1.27) (thickness 0.2032)))
     )
-    (fp_text value 22k (at 0 0) (layer F.SilkS) hide
+    (fp_text value 15k (at 0 0) (layer F.SilkS) hide
       (effects (font (size 1.397 1.27) (thickness 0.2032)))
     )
@@
       (effects (font (size 1.397 1.27) (thickness 0.2032)))
     )
-    (fp_text value 22k (at 0 0) (layer F.SilkS) hide
+    (fp_text value 15k (at 0 0) (layer F.SilkS) hide
       (effects (font (size 1.397 1.27) (thickness 0.2032)))
     )
@@
       (effects (font (size 1.397 1.27) (thickness 0.2032)))
     )
-    (fp_text value 1k (at 0 0) (layer F.SilkS) hide
+    (fp_text value 820 (at 0 0) (layer F.SilkS) hide
       (effects (font (size 1.397 1.27) (thickness 0.2032)))
     )
