File: hardware/voice2.kicad_sch (KiCad schematic)
At the start: 29 parts, among them IC1 LM13700, U12 MCP4922-E/P, U13 SSM2044

Commit message: hardware: OverCycler3 schematics WIP
Parts:
- removed RV3: 1k, ~, symbol overcycler2-rescue:POT
- added R131, R137: 470, ~, symbol overcycler2-rescue:R
Connections:
- net GND: now also R131.1, R137.2
- net at IC1.3 (+), R61.2: now also R131.2
- net at IC1.4 (-): now also R137.1
Other:
- note removed: "Adjust RV2 to reduce DC offset at IC1.5 or IC1.12 between VCA fully open and fully closed (set OscA,OscB,Noise volume to zero)"

Commit message: hardware: OverCycler3 schematics WIP2
Changed lines of the file:
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@@
   )
   (global_label "SPI_MOSI" (shape input) (at 35.56 90.17 180)
-    (effects (font (size 0.9906 0.9906)) (justify right))
+    (effects (font (size 1.27 1.27)) (justify right))
     (property "Intersheetrefs" "${INTERSHEET_REFS}" (at 35.56 90.17 0)
       (effects (font (size 1.27 1.27)) hide)
@@
   )
   (global_label "NOISE" (shape input) (at 78.74 83.82 180)
-    (effects (font (size 0.9906 0.9906)) (justify right))
+    (effects (font (size 1.27 1.27)) (justify right))
     (property "Intersheetrefs" "${INTERSHEET_REFS}" (at 78.74 83.82 0)
       (effects (font (size 1.27 1.27)) hide)
@@
   )
   (global_label "SPI_SCK" (shape input) (at 35.56 92.71 180)
-    (effects (font (size 0.9906 0.9906)) (justify right))
+    (effects (font (size 1.27 1.27)) (justify right))
     (property "Intersheetrefs" "${INTERSHEET_REFS}" (at 35.56 92.71 0)
       (effects (font (size 1.27 1.27)) hide)
@@
   )
   (global_label "DAC_RES" (shape input) (at 107.95 78.74 180)
-    (effects (font (size 0.9906 0.9906)) (justify right))
+    (effects (font (size 1.27 1.27)) (justify right))
     (property "Intersheetrefs" "${INTERSHEET_REFS}" (at 107.95 78.74 0)
       (effects (font (size 1.27 1.27)) hide)
@@
   )
   (global_label "DAC_MIXA" (shape input) (at 50.8 83.82 90)
-    (effects (font (size 0.9906 0.9906)) (justify left))
+    (effects (font (size 1.27 1.27)) (justify left))
     (property "Intersheetrefs" "${INTERSHEET_REFS}" (at 50.8 83.82 0)
       (effects (font (size 1.27 1.27)) hide)
@@
   )
   (global_label "DAC_MIXB" (shape input) (at 50.8 106.68 270)
-    (effects (font (size 0.9906 0.9906)) (justify right))
+    (effects (font (size 1.27 1.27)) (justify right))
     (property "Intersheetrefs" "${INTERSHEET_REFS}" (at 50.8 106.68 0)
       (effects (font (size 1.27 1.27)) hide)
@@
   )
   (hierarchical_label "OUT" (shape output) (at 259.08 88.9 0) (fields_autoplaced)
-    (effects (font (size 0.9906 0.9906)) (justify left))
+    (effects (font (size 1.27 1.27)) (justify left))
   )
   (hierarchical_label "DAC_FC" (shape input) (at 149.86 115.57 180) (fields_autoplaced)
-    (effects (font (size 0.9906 0.9906)) (justify right))
+    (effects (font (size 1.27 1.27)) (justify right))
   )
   (hierarchical_label "DAC_VCA" (shape input) (at 207.01 115.57 180) (fields_autoplaced)
-    (effects (font (size 0.9906 0.9906)) (justify right))
+    (effects (font (size 1.27 1.27)) (justify right))
   )
   (hierarchical_label "SPI_CS" (shape input) (at 35.56 95.25 180) (fields_autoplaced)
-    (effects (font (size 0.9906 0.9906)) (justify right))
+    (effects (font (size 1.27 1.27)) (justify right))
   )
   (symbol (lib_id "overcycler2-rescue:SSM2044") (at 133.35 95.25 0) (unit 1)

Commit message: hardware: OverCycler3 schematics Rev1 OK
Parts:
- renumbered C43 to C71, C44 to C72, C45 to C73, C46 to C74, C47 to C75, C48 to C76, C90 to C77, C49 to C78, C50 to C79, C51 to C80, R55 to R87, R56 to R88, R58 to R89, R57 to R90, R59 to R91, R60 to R92, R61 to R93, R137 to R94, R131 to R95, R62 to R96, R63 to R97, R64 to R98, R65 to R99
Other:
- note added: "Use film capacitors for C53..C56, preferably within 1% of theoretical value."
- note removed: "Use film capacitors for C36..C39, preferably within 1% of theoretical value."
- title: Voice for OverCycler 2 -> Voice for OverCycler 3

Commit message: hardware: SSM2044 -> SSI2144
Parts:
- removed U13: SSM2044, MODULE, symbol overcycler2-rescue:SSM2044
- added U9: SSI2144, Package_SO:SSOP-16_3.9x4.9mm_P0.635mm, symbol Audio:SSI2144
Connections:
- net +5V: now also U9.16 (V+)
- net -5V: now also U9.8 (V-)
- net GND: now also U9.9 (GND)
- net at R.2, R.2, R.2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: now also U9.1 (SIG_IN+)
- net at C76.1: now also U9.12 (C1B)
- net at C76.2: now also U9.13 (C1A)
- net at C75.1: now also U9.10 (C2B)
- net at C77.2, R88.2, R89.1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: now also U9.15 (FREQ_CTRL)
- net at C75.2: now also U9.11 (C2A)
- net at R90.2: now also U9.2 (SIG_IN-)
- net at R87.2: now also U9.14 (Q_CTRL)
- net at C78.1, R91.1: now also U9.3 (OUT)
- net at C73.1: now also U9.4 (C4A)
- net at C73.2: now also U9.5 (C4B)
- net at C74.1: now also U9.6 (C3A)
- net at C74.2: now also U9.7 (C3B)
Other:
- moved on the sheet: C73, C74, C75, C76, C77, C78, C79, C80, IC1B, R87, R88, R89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
