File: hardware/overcycler2.kicad_sch (KiCad schematic)
At the start: 104 parts, among them P1 LPC_P1, P2 LPC_P2, P3 FT232, P4 PANEL, P5 SDCARD, P6 MIDI_IN, P7 FOOT_IN, P8 AC_IN, P9 AUDIO_OUT, Q1 BC547, SW1 RESET, U1 TLV1543, U2 74HC138, U3 LTC1660, U4 LTC1660, U5 TL074, U6 TL074, U7 LM1084IT-5.0/NOPB, U8 LM2990-5.0/NOPB, U9 LM1084IT-ADJ/NOPB

Commit message: hardware: OverCycler3 schematics WIP
Parts:
- removed C1: 10u, ~, symbol overcycler2-rescue:CP1
- removed C2, C26, C27, C30: 100n, ~, symbol overcycler2-rescue:C
- removed C25: 10000u 16v, ~, symbol overcycler2-rescue:CP1
- removed D1, D6, D7: 1N5819, ~, symbol overcycler2-rescue:DIODESCH
- removed P6: MIDI_IN, symbol overcycler2-rescue:CONN_2
- removed P7: FOOT_IN, symbol overcycler2-rescue:CONN_2
- removed P8: AC_IN, symbol overcycler2-rescue:CONN_2
- removed P9: AUDIO_OUT, symbol overcycler2-rescue:CONN_8
- removed R126: 220, ~, symbol overcycler2-rescue:R
- removed R127: 120, ~, symbol overcycler2-rescue:R
- removed R4: 1k, ~, symbol overcycler2-rescue:R
- removed U3, U4: LTC1660, MODULE, symbol overcycler2-rescue:LTC1660
- removed U7: LM1084IT-5.0/NOPB, TO-220, symbol overcycler2-rescue:LM1084IT-5.0/NOPB
- removed U8: LM2990-5.0/NOPB, TO-220, symbol overcycler2-rescue:LM7905CT
- removed U9: LM1084IT-ADJ/NOPB, TO-220, symbol overcycler2-rescue:LM1084IT-ADJ/NOPB
- added D1: 1N4148, ~, symbol overcycler2-rescue:DIODE
- added J1: USB_B, symbol Connector:USB_B
- added J2, J3, J4: AudioJack2, symbol Connector_Audio:AudioJack2
- added J5: DIN-5_180degree, symbol Connector:DIN-5_180degree
- added PS1: IA0505S-2W, Converter_DCDC:Converter_DCDC_XP_POWER-IAxxxxS_THT, symbol Converter_DCDC:IA0505S
- added PS2: IB0503LSY-1WR1, Converter_DCDC:Converter_DCDC_XP_POWER-IAxxxxS_THT, symbol Converter_DCDC:IA0503S
- added R141, R142: 1k, ~, symbol overcycler2-rescue:R
- added R143, R144: 2k2, ~, symbol overcycler2-rescue:R
- added RV2: 47k, symbol Device:R_Potentiometer_Dual
- added U7: AD5674R, MODULE, symbol AD5674R:AD5674R
- C24: value 10000u 16v -> 470u
- R34, R35: value 1k -> 47
Connections:
- net +3.3V: now also PS2.6 (+Vout), U7.18 (VLOGIC), U7.20 (/RESET), U7.6 (GAIN)
- net +5V: now also PS1.7 (+Vout), R142.1, U7.2 (VDD)
- net -5V: now also PS1.9 (-Vout)
- net DAC_FC0: now also U7.25 (VOUT8)
- net DAC_FC1: now also U7.24 (VOUT9)
- net DAC_FC2: now also U7.23 (VOUT10)
- net DAC_FC3: now also U7.22 (VOUT11)
- net DAC_FC4: now also U7.14 (VOUT12)
- net DAC_FC5: now also U7.13 (VOUT13)
- net DAC_MIXA: now also U7.12 (VOUT14)
- net DAC_MIXB: now also U7.11 (VOUT15)
- net DAC_MIXN: now also U7.8 (VOUT6)
- net DAC_RES: now also U7.7 (VOUT7)
- net DAC_VCA0: now also U7.1 (VOUT0)
- net DAC_VCA1: now also U7.28 (VOUT1)
- net DAC_VCA2: now also U7.27 (VOUT2)
- net DAC_VCA3: now also U7.26 (VOUT3)
- net DAC_VCA4: now also U7.10 (VOUT4)
- net DAC_VCA5: now also U7.9 (VOUT5)
- net GND: now also J2.S, J3.S, J4.S, PS1.10 (0V), PS2.4 (-Vout), R141.1, RV2.1, RV2.4, U7.15 (GND), U7.16 (GND), U7.17 (/LDAC); no longer C24.2, U1.12 (A10)
- net at R3.1: now also J5.4
- net at OC1.3 (C): now also D1.1 (A), J5.5
- net at OC1.2 (A), R3.2: now also D1.2 (K)
- net at R5.2, R7.1: now also J4.T
- net at R34.1: now also J3.T
- net at R35.1: now also J2.T
- net at R30.1, U6.1: now also R143.1, RV2.3
- net at U6.5 (+): now also RV2.2
- net at R31.1, U6.14: now also R144.1, RV2.6
- net at U6.10 (+): now also RV2.5
- net SPI_CS6: no longer names the net of U2.9 (O6)
- net SPI_CS7: no longer names the net of U2.7 (O7)
- net UNR+: no longer names the net of C24.1
- net UNR+: now also J1.1 (VBUS), PS1.1 (+Vin), PS2.1 (+Vin)
- new net: C24.2, J1.4 (GND), PS1.2 (-Vin), PS2.2 (-Vin)
- new net ADC_MIX: R141.2, R142.2, R143.2, R144.2, U1.12 (A10)
- new net CV_SPI_MOSI: U7.5 (SDI)
- new net CV_SPI_SCK: U7.4 (SCLK)
- new net CV_SPI_SSEL: U7.3 (/SYNC)
- new net USB_DM: J1.2 (D-)
- new net USB_DP: J1.3 (D+)
Other:
- note added: "All capacitors should be minimum 16V unless specified All polarized capacitors are tantalum All unpolarised capacitors are ceramic All resistors are 5% 1/4w Data entry potentiometers are 4.7k linear taper"
- note removed: "1: left master volume to pot 2: left master volume from pot 3: master volume ground 4: right master volume to pot 5: right master volume from pot 6: master jacks ground 7: left master jack 8: right master jack"
- note removed: "All capacitors should be minimum 16V unless specified All polarized capacitors are electrolytic All unpolarised capacitors are film All resistors are 5% 1/4w Data entry potentiometers are 4.7k linear taper Master volume potentiometer is 47k dual audio taper"
- note removed: "Pin 1 is DIN socket pin 4 Pin 2 is DIN socket pin 5"
- note removed: "Use mininum 7.5VAC 1A power supply Higher voltage may overheat the regulators"
- moved on the sheet: C10, C11, C12, C13, C14, C15, C16, C17, C18, C19, C20, C21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

Commit message: hardware: OverCycler3 schematics WIP2
Parts:
- removed C88: 2u2, ~, symbol overcycler2-rescue:CP1
- removed P1: LPC_P1, ~, symbol overcycler2-rescue:CONN_33
- removed P2: LPC_P2, symbol overcycler2-rescue:CONN_33
- removed P3: FT232, symbol overcycler2-rescue:CONN_6
- removed P5: SDCARD, symbol overcycler2-rescue:CONN_7
- removed RV1: 10k, ~, symbol overcycler2-rescue:POT
- removed SW1: RESET, ~, symbol overcycler2-rescue:SW_PUSH
- added C1, C25: 22p, ~, symbol overcycler2-rescue:C
- added C100, C101, C102, C103, C104, C105, C106, C107, C108, C109, C110, C2, C26, C27, C30, C88, C96, C97, C98, C99: 100n, ~, symbol overcycler2-rescue:C
- added D6: BZV55B3V3, Diode_SMD:D_MiniMELF, symbol Diode:BZV55B3V3
- added P6: FT232, symbol overcycler2-rescue:CONN_6
- added R145: 10k, ~, symbol overcycler2-rescue:R
- added R146, R147, R4: 1k, ~, symbol overcycler2-rescue:R
- added R148: 33, ~, symbol overcycler2-rescue:R
- added R149: 1k5, ~, symbol overcycler2-rescue:R
- added R150: 330, ~, symbol overcycler2-rescue:R
- added SW2: RESET, ~, symbol overcycler2-rescue:SW_PUSH
- added U3: LPC1778FBD144, MODULE, symbol LPC1778FBD144:LPC1778FBD144
- added U4: XT26G02ELGIGA, MODULE, symbol XT26G02ELGIGA:XT26G02ELGIGA
- added Y1: 12MHz, symbol Device:Crystal
- R128: value 10k -> 33
Connections:
- net +3.3V: now also C19.1, C100.1, C26.1, C27.1, C30.1, C88.1, C96.1, C97.1, C98.1, C99.1, P6.1, R147.1, R4.1, U3.102 (VDD(3V3)), U3.114 (VDD(3V3)), U3.121 (VDD(REG)(3V3)), U3.138 (VDD(3V3)), U3.14 (VDDA), U3.17 (VREFP), U3.18 (VDD(REG)(3V3)), U3.41 (VDD(3V3)), U3.60 (VDD(REG)(3V3)), U3.62 (VDD(3V3)), U3.77 (VDD(3V3)), U4.3 (/WP), U4.7 (/HOLD), U4.8 (VCC); no longer R128.1
- net +5V: no longer C19.1
- net ADC_ADDR: now also U3.10 (P0[25])
- net ADC_CLK: now also U3.35 (P0[27])
- net ADC_CS: now also U3.13 (P0[23])
- net ADC_EOC: now also U3.34 (P0[28])
- net ADC_OUT: now also U3.11 (P0[24])
- net CV_SPI_MOSI: now also U3.135 (P1[1])
- net CV_SPI_SCK: now also U3.136 (P1[0])
- net CV_SPI_SSEL: now also U3.132 (P1[8])
- net FOOT_IN: now also U3.38 (P3[26])
- net GND: now also C1.2, C100.2, C101.2, C102.2, C103.2, C104.2, C105.2, C106.2, C107.2, C108.2, C109.2, C110.2, C2.2, C25.2, C26.2, C27.2, C30.2, C88.2, C96.2, C97.2, C98.2, C99.2, P6.4, SW2.1, U3.103 (VSS), U3.117 (VSS), U3.119 (VSSREG), U3.139 (VSS), U3.15 (VSSA), U3.22 (VSSREG), U3.44 (VSS), U3.59 (VSSREG), U3.65 (VSS), U3.79 (VSS), U4.4 (VSS)
- net KP_1_R1: now also U3.80 (P0[22])
- net KP_2_R2: now also U3.82 (P0[21])
- net KP_3_R3: now also U3.83 (P0[20])
- net KP_4_R4: now also U3.85 (P0[19])
- net KP_5_C1: now also U3.69 (P0[10])
- net KP_6_C2: now also U3.122 (P4[29])
- net KP_7_C3: now also U3.118 (P4[28])
- net KP_8_C4: now also U3.71 (P2[13])
- net LCD_DB4: now also U3.106 (P2[1])
- net LCD_DB5: now also U3.107 (P2[0])
- net LCD_DB6: now also U3.105 (P2[2])
- net LCD_DB7: now also U3.100 (P2[3])
- net LCD_E1: now also U3.96 (P2[6])
- net LCD_E2: now also U3.95 (P2[7])
- net LCD_RS: now also U3.99 (P2[4])
- net LCD_RW: now also U3.97 (P2[5])
- net MIDI_IN: now also U3.70 (P0[11])
- net P_0: now also C106.1
- net P_1: now also C107.1
- net P_2: now also C108.1
- net P_3: now also C109.1
- net P_4: now also C110.1
- net P_5: now also C105.1
- net P_6: now also C104.1
- net P_7: now also C103.1
- net P_8: now also C102.1
- net P_9: now also C101.1
- net SPI_MOSI: now also U3.54 (P1[24])
- net SPI_MUX_A: now also U3.89 (P0[15])
- net SPI_MUX_B: now also U3.90 (P0[16])
- net SPI_MUX_C: now also U3.115 (P0[5])
- net SPI_SCK: now also U3.49 (P1[20])
- net SPI_SSEL: now also U3.50 (P1[21])
- net USB_DM: now also R128.1, U3.43 (P0[30]); no longer J1.2 (D-)
- net USB_DP: now also R148.1, U3.42 (P0[29]); no longer J1.3 (D+)
- net at R128.2: now also J1.2 (D-)
- net at P4.12 (P12): now also R146.1
- net at C24.1, J1.1 (VBUS), PS1.1 (+Vin)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: now also R150.1
- net at C24.2, J1.4 (GND), PS1.2 (-Vin)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: now also D6.2 (A)
- net CV_SPI_MISO: now reaches U7.19 (SDO)
- net CV_SPI_MISO: now also U3.133 (P1[4])
- new net: J1.3 (D+), R148.2, R149.1
- new net: D6.1 (K), R149.2, R150.2
- new net: R145.2, R4.2, SW2.2
- new net FLASH_SPI_MISO: U3.111 (P0[8]), U4.2 (DO)
- new net FLASH_SPI_MOSI: U3.109 (P0[9]), U4.5 (DI)
- new net FLASH_SPI_SCK: U3.112 (P0[7]), U4.6 (CLK)
- new net FLASH_SPI_SSEL: U3.113 (P0[6]), U4.1 (/CS)
- new net LCD_CTRST: R146.2, U3.8 (P0[26])
- new net PROG_BOOT: P6.6, R147.2, U3.76 (P2[10])
- new net PROG_RXD: P6.3, U3.142 (P0[3])
- new net PROG_TXD: P6.2, U3.141 (P0[2])
- new net RESET: C2.1, R145.1, U3.24 (RESET)
- new net XTAL1: C1.1, U3.31 (XTAL1), Y1.1
- new net XTAL2: C25.1, U3.33 (XTAL2), Y1.2
Other:
- note removed: "Solder a microSD to SD adapter using a pin strip Pins are per SD specifications"
- moved on the sheet: C10, C11, C12, C13, C14, C15, C16, C17, C18, C20, C21, C22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

Commit message: hardware: OverCycler3 schematics Rev1 OK
Parts:
- added SW2: POWER, symbol Switch:SW_SPST
- renumbered C12 to C10, C13 to C11, C14 to C12, C15 to C13, C16 to C14, C17 to C15, C24 to C16, C18 to C17, C20 to C18, C21 to C19, C6 to C2, C22 to C20, C19 to C21, C26 to C22, C28 to C23, C29 to C24, C27 to C25, C30 to C26, C88 to C27, C96 to C28, C97 to C29, C7 to C3, C98 to C30, C99 to C31, C33 to C32, C95 to C33, C100 to C34, C4 to C35, C5 to C36, C3 to C37, C101 to C38, C102 to C39, C8 to C4, C103 to C40, C104 to C41, C105 to C42, C106 to C43, C107 to C44, C108 to C45, C109 to C46, C110 to C47, C23 to C48, C31 to C49, C9 to C5, C32 to C50, C10 to C6, C11 to C7, C2 to C8, C25 to C9, D6 to D1, D1 to D6, J4 to J2, J5 to J3, J2 to J4, J3 to J5, P6 to P1, P4 to P2, R4 to R1, R8 to R10, R9 to R11, R10 to R12, R11 to R13, R12 to R14, R5 to R15, R13 to R16, R7 to R17, R14 to R18, R15 to R19, R128 to R2, R16 to R20, R17 to R21, R1 to R22, R2 to R23, R18 to R24, R19 to R25, R146 to R26, R3 to R27, R20 to R28, R21 to R29, R145 to R3, R22 to R30, R23 to R31, R24 to R32, R25 to R33, R26 to R34, R27 to R35, R28 to R36, R29 to R37, R142 to R38, R143 to R39, R148 to R4, R144 to R40, R141 to R41, R130 to R42, R30 to R43, R31 to R44, R32 to R45, R33 to R46, R34 to R47, R35 to R48, R149 to R5, R150 to R6, R147 to R7, R129 to R8, R6 to R9, RV2 to RV1, SW2 to SW1, U4 to U1, U5 to U2, U1 to U4, U2 to U5
Connections:
- net at C16.1, PS1.1 (+Vin), PS2.1 (+Vin)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: now also SW2.2 (B); no longer J1.1 (VBUS)
- new net: J1.1 (VBUS), SW2.1 (A)
Other:
- note added: "LCD Display is NHD‐0440WH Keypad is 16 keys 4*4 matrix Data entry potentiometers are 4.7k linear taper"
- note added: "Select Q1 for 0.3Vpp..0.4Vpp of noise at U5.1 R9 value can be adjusted if need be"
- note removed: "All capacitors should be minimum 16V unless specified All polarized capacitors are tantalum All unpolarised capacitors are ceramic All resistors are 5% 1/4w Data entry potentiometers are 4.7k linear taper"
- note removed: "Select Q1 for 0.3Vpp..0.4Vpp of noise at U5.1 R6 value can be adjusted if need be"
- title: OverCycler 2 full board -> OverCycler 3 full board
- moved on the sheet: C16, C23, C24, C32, D1, PS1, PS2, R5, R6

Commit message: hardware: noise transistor change -- minor fixes
Parts:
- removed Q1: BC547, TO92, symbol overcycler2-rescue:BC547
- added Q1: 2SC945, Package_TO_SOT_THT_AKL:TO-92_Inline_Wide_ECB, symbol PCM_Transistor_BJT_AKL:2SC945
Connections:
- net at C33.2, R8.1: now also Q1.3 (B)
- net at C35.1, R9.1: now also Q1.1 (E)
Other:
- note added: "Select Q1 for 0.3Vpp..0.4Vpp of noise at U2.1 R9 value can be adjusted if need be"
- note removed: "Select Q1 for 0.3Vpp..0.4Vpp of noise at U5.1 R9 value can be adjusted if need be"
Changed lines of the file:
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@@
     (stroke (width 0) (type default))
   )
-  (text "Select Q1 for\n0.3Vpp..0.4Vpp\nof noise at U5.1\nR9 value can be \nadjusted if need be"
+  (text "Select Q1 for\n0.3Vpp..0.4Vpp\nof noise at U2.1\nR9 value can be \nadjusted if need be"
     (at 142.24 83.82 0)
     (effects (font (size 1.524 1.524)) (justify left bottom))
@@
     )
   )
-  (symbol (lib_id "overcycler2-rescue:BC547") (at 146.05 59.69 0) (mirror x) (unit 1)
-    (in_bom yes) (on_board yes) (dnp no)
-    (property "Reference" "Q1" (at 146.05 55.9054 0)
-      (effects (font (size 1.016 1.016)) (justify right))
-    )
-    (property "Value" "BC547" (at 146.05 63.5 0)
-      (effects (font (size 1.016 1.016)) (justify right))
-    )
-    (property "Footprint" "TO92" (at 143.51 62.2808 0)
-      (effects (font (size 0.7366 0.7366)))
-    )
-    (property "Datasheet" "~" (at 146.05 59.69 0)
-      (effects (font (size 1.524 1.524)))
-    )
-    (pin "1")
-    (pin "2")
-    (pin "3")
-    (instances
-      (project "overcycler2"
-        (path "/f3616c1d-a98e-4f9d-ac17-0c5545b71bc4"
-          (reference "Q1") (unit 1)
-        )
-      )
-    )
-  )
   (symbol (lib_id "overcycler2-rescue:R") (at 148.59 45.72 180) (unit 1)
     (in_bom yes) (on_board yes) (dnp no)
@@
       (effects (font (size 1.27 1.27)) (justify left))
     )
-    (property "Value" "100u" (at 138.43 67.31 0)
+    (property "Value" "100u" (at 132.08 67.31 0)
       (effects (font (size 1.27 1.27)) (justify left))
     )
@@
         )
       )
+    )
+  )
+  (symbol (lib_id "PCM_Transistor_BJT_AKL:2SC945") (at 146.05 59.69 0) (mirror x) (unit 1)
+    (in_bom yes) (on_board yes) (dnp no) (fields_autoplaced)
+    (property "Reference" "Q1" (at 151.13 58.42 0)
+      (effects (font (size 1.27 1.27)) (justify left))
+    )
+    (property "Value" "2SC945" (at 151.13 60.96 0)
+      (effects (font (size 1.27 1.27)) (justify left))
+    )
+    (property "Footprint" "Package_TO_SOT_THT_AKL:TO-92_Inline_Wide_ECB" (at 151.13 62.23 0)
+      (effects (font (size 1.27 1.27)) hide)
+    )
+    (property "Datasheet" "http://www.unisonic.com.tw/datasheet/2SC945.pdf" (at 146.05 59.69 0)
+      (effects (font (size 1.27 1.27)) hide)
+    )
+    (pin "1")
+    (pin "2")
+    (pin "3")
+    (instances
+      (project "overcycler2"
+        (path "/f3616c1d-a98e-4f9d-ac17-0c5545b71bc4"
+          (reference "Q1") (unit 1)
+        )
+      )

Commit message: hardware: USB GND should be tied to GND -- minor fixes
Parts:
- removed D1: BZV55B3V3, Diode_SMD:D_MiniMELF, symbol Diode:BZV55B3V3
- removed R6: 330, ~, symbol overcycler2-rescue:R
- added C49: 100n, ~, symbol overcycler2-rescue:C
- added FB1: FerriteBead, symbol Device:FerriteBead
- added R42: 4k7, ~, symbol overcycler2-rescue:R
- renumbered C16 to C13, C13 to C14, C14 to C15, C15 to C16, C23 to C21, C24 to C22, C21 to C23, C22 to C24, C32 to C31, C31 to C32, C49 to C50, C50 to C51, D2 to D1, D3 to D2, D4 to D3, D5 to D4, D6 to D5, R11 to R10, R12 to R11, R13 to R12, R14 to R13, R15 to R14, R16 to R15, R17 to R16, R18 to R17, R19 to R18, R20 to R19, R21 to R20, R22 to R21, R23 to R22, R24 to R23, R25 to R24, R26 to R25, R27 to R26, R28 to R27, R29 to R28, R30 to R29, R31 to R30, R32 to R31, R33 to R32, R34 to R33, R35 to R34, R36 to R35, R37 to R36, R38 to R37, R39 to R38, R40 to R39, R41 to R40, R42 to R41, R7 to R6, R8 to R7, R9 to R8, R10 to R9
Connections:
- net +3.3V: now also R5.1, R42.1; no longer U4.14 (REF+)
- net GND: now also C49.2, FB1.1
- net at J1.3 (D+), R4.2: now also R5.2; no longer R5.1
- net at C13.2, J1.4 (GND), PS1.2 (-Vin)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: now also FB1.2
- new net: C49.1, R42.2, U4.14 (REF+)
Other:
- note added: "Select Q1 for 0.3Vpp..0.4Vpp of noise at U2.1 R8 value can be adjusted if need be"
- note removed: "Select Q1 for 0.3Vpp..0.4Vpp of noise at U2.1 R9 value can be adjusted if need be"
- moved on the sheet: C13, C21, C22, C31, PS1, PS2, R41, R5, U4, U5

Commit message: hardware: adjusted mixer levels
Parts:
- R29, R34: value 150k -> 120k
- R31, R32: value 68k -> 82k
Changed lines of the file:
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@@
       (effects (font (size 1.016 1.016)))
     )
-    (property "Value" "150k" (at 302.2854 53.1622 90)
+    (property "Value" "120k" (at 302.2854 53.1622 90)
       (effects (font (size 1.016 1.016)))
     )
@@
       (effects (font (size 1.016 1.016)))
     )
-    (property "Value" "68k" (at 302.2854 43.0022 90)
+    (property "Value" "82k" (at 302.2854 43.0022 90)
       (effects (font (size 1.016 1.016)))
     )
@@
       (effects (font (size 1.016 1.016)))
     )
-    (property "Value" "68k" (at 302.2854 36.6522 90)
+    (property "Value" "82k" (at 302.2854 36.6522 90)
       (effects (font (size 1.016 1.016)))
     )
@@
       (effects (font (size 1.016 1.016)))
     )
-    (property "Value" "150k" (at 302.2854 26.4922 90)
+    (property "Value" "120k" (at 302.2854 26.4922 90)
       (effects (font (size 1.016 1.016)))
     )

Commit message: hardware: sch small changes -- footprints assigned
Parts:
- C1, C10, C11, C12, C14, C15, C16, C17, C18, C19, C2, C20, C23, C24, C25, C26, C27, C28, C29, C3, C30, C32, C34, C35, C37, C38, C39, C4, C40, C41, C42, C43, C44, C45, C46, C47, C49, C5, C50, C51, C6, C7, C8, C9: footprint ~ -> Capacitor_SMD:C_0805_2012Metric
- C13: footprint ~ -> Capacitor_Tantalum_SMD:CP_EIA-7343-43_Kemet-X
- C21, C22, C31: footprint ~ -> Capacitor_Tantalum_SMD:CP_EIA-3216-18_Kemet-A
- C33, C36, C48: footprint ~ -> Capacitor_Tantalum_SMD:CP_EIA-3528-21_Kemet-B
- D1, D2, D3, D4, D5: footprint ~ -> Diode_SMD:D_SOD-123
- FB1: footprint (none) -> Inductor_SMD:L_0805_2012Metric
- J1: footprint (none) -> Connector_USB:USB_B_Lumberg_2411_02_Horizontal
- J2, J4, J5: value AudioJack2 -> AudioJack3_Switch; footprint (none) -> Connector_Audio:Jack_6.35mm_Neutrik_NMJ6HFD2_Horizontal; symbol Connector_Audio:AudioJack2 -> Connector_Audio:AudioJack3_Switch
- J3: footprint (none) -> DIN-5-180:DIN-5-180
- OC1: footprint optocoupler-DIL08 -> Package_DIP:DIP-8_W7.62mm
- P1: footprint (none) -> Connector_PinSocket_2.54mm:PinSocket_1x06_P2.54mm_Vertical
- P2: footprint (none) -> Connector_IDC:IDC-Header_2x20_P2.54mm_Vertical
- PS1: footprint Converter_DCDC:Converter_DCDC_XP_POWER-IAxxxxS_THT -> JETEKPS:IA0505S-2W
- PS2: footprint Converter_DCDC:Converter_DCDC_XP_POWER-IAxxxxS_THT -> JETEKPS:IB0503LSY
- Q1: footprint Package_TO_SOT_THT_AKL:TO-92_Inline_Wide_ECB -> Package_TO_SOT_SMD:SOT-23
- R1, R10, R11, R12, R13, R14, R15, R16, R17, R18, R19, R2, R20, R21, R22, R23, R24, R25, R26, R27, R28, R29, R3, R30, R31, R32, R33, R34, R35, R36, R37, R38, R39, R4, R40, R41, R42, R43, R44, R45, R46, R5, R6, R7, R8, R9: footprint ~ -> Resistor_SMD:R_0805_2012Metric
- R47, R48: value 47 -> 330; footprint ~ -> Resistor_SMD:R_0805_2012Metric
- RV1: footprint (none) -> Potentiometer_THT:Potentiometer_Alps_RK163_Dual_Horizontal
- SW1: footprint ~ -> Button_Switch_THT:SW_Tactile_SPST_Angled_PTS645Vx83-2LFS
- SW2: footprint (none) -> SPUN192600:SPUN192600; symbol Switch:SW_SPST -> Switch:SW_Push_DPDT
- U1: footprint MODULE -> Package_LGA:LGA-8_8x6mm_P1.27mm
- U2, U6: footprint (none) -> Package_SO:SO-14_3.9x8.65mm_P1.27mm
- U3: footprint MODULE -> Package_QFP:LQFP-144_20x20mm_P0.5mm
- U4: footprint MODULE -> Package_SO:SOIC-20W_7.5x12.8mm_P1.27mm
- U5: footprint ~ -> Package_SO:SO-16_3.9x9.9mm_P1.27mm
- U7: footprint MODULE -> Package_DFN_QFN:QFN-28-1EP_4x4mm_P0.4mm_EP2.6x2.6mm
- Y1: footprint (none) -> Crystal:Crystal_SMD_HC49-SD
Connections:
- net GND: now also J2.SN, J4.SN, J5.SN, U7.29 (PAD)
- net at J2.T, R14.2, R16.1: now also J2.TN
- net at C50.2, R45.2, U6.7: now also R47.1; no longer R48.2
- net at C51.2, R46.2, U6.8: now also R48.1; no longer R47.2
- net at J5.T: now also R48.2; no longer R47.1
- net at J4.T: now also R47.2; no longer R48.1
- net at C35.1, R8.1: now also Q1.2 (E); no longer Q1.1 (E)
- net at C33.2, R7.1: now also Q1.1 (B); no longer Q1.3 (B)
- net at C13.1, PS1.1 (+Vin), PS2.1 (+Vin): now also SW2.1 (A), SW2.4 (A); no longer SW2.2 (B)
- net at J1.1 (VBUS): now also SW2.2 (B), SW2.5 (B); no longer SW2.1 (A)
- new net: J4.TN, J5.R
- new net: J4.R, J5.TN
Other:
- moved on the sheet: C37, C50, C51, R14, R27, R28, R29, R30, R31, R32, R33, R34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
