File: hardware/overcycler3.kicad_pcb (KiCad board)
At the start: 2 copper layers, 200.7 x 99.1 mm, 308 parts, among them IC1 LM13700, IC2 LM13700, IC3 LM13700, J1 USB_B, J2 AudioJack3_Switch, J3 DIN-5_180degree, J4 AudioJack3_Switch, J5 AudioJack3_Switch, P1 FT232, P2 PANEL, Q1 2SC945, SW1 RESET, SW2 POWER, U1 XT26G02ELGIGA, U10 MCP4922-ESL, U11 SSI2144, U12 MCP4922-ESL, U13 SSI2144, U14 MCP4922-ESL, U15 SSI2144, U16 MCP4922-ESL, U17 SSI2144, U18 MCP4922-ESL, U19 SSI2144, U2 TL074, U20 AD5328B, U3 LPC1778FBD144, U4 TLV2556, U5 74HC138, U6 TL074, U7 AD5328B, U8 MCP4922-ESL, U9 SSI2144, Y1 12MHz

Commit message: hardware: chnaged some capacitor values and footprints
Parts:
- C102, C103, C52, C53, C62, C63, C72, C73, C82, C83, C92, C93: footprint Capacitor_Tantalum_SMD:CP_EIA-3216-18_Kemet-A -> Capacitor_SMD:C_0805_2012Metric
- C109, C59, C69, C79, C89, C99: value 33u -> 47u; footprint Capacitor_Tantalum_SMD:CP_EIA-3216-18_Kemet-A -> Capacitor_SMD:C_1206_3216Metric
- moved C30 31.0 mm to (78.7, 106.5), turned to -90 degrees
- moved C34 5.69 mm to (85.9, 70.2), turned to 90 degrees
- moved C17 5.57 mm to (85.9, 93.2), turned to 90 degrees
- moved R21 2.29 mm to (65.1, 79.0)
- moved C72 1.59 mm to (123.2, 122.7), turned to 90 degrees
- moved C82 1.59 mm to (180.3, 122.7), turned to 90 degrees
- moved C102 1.55 mm to (199.1, 122.7), turned to 90 degrees
- moved C52 1.55 mm to (104.1, 122.7), turned to 90 degrees
- moved C92 1.48 mm to (142.2, 122.7), turned to 90 degrees
- moved C62 1.48 mm to (161.3, 122.7), turned to 90 degrees
- moved C18 1.46 mm to (78.7, 110.3)
- moved C53 0.45 mm to (107.6, 121.9)
- moved C63 0.45 mm to (164.8, 121.9)
- moved C83 0.45 mm to (183.7, 121.9)
- moved C93 0.45 mm to (145.7, 121.9)
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Routing:
- net GND: track 1285.8 -> 60.6 mm, vias 12 -> 0
- net +5V: track 655.5 -> 8.94 mm, vias 14 -> 0
- net -5V: track 539.0 -> 0.00 mm, vias 11 -> 0
- net +3.3V: track 419.4 -> 38.9 mm, vias 5 -> 0
- net SPI_SCK: track 221.2 -> 0.00 mm, vias 3 -> 0
- net SPI_MOSI: track 219.6 -> 0.00 mm, vias 3 -> 0
- net /ADC_MIX: track 172.9 -> 0.00 mm, vias 2 -> 0
- net DAC_MIXA: track 164.1 -> 0.00 mm, vias 6 -> 0
- net DAC_MIXB: track 161.9 -> 0.00 mm, vias 6 -> 0
- net Net-(U6D--): track 155.8 -> 0.00 mm, vias 2 -> 0
- net DAC_RES: track 147.8 -> 0.00 mm, vias 7 -> 0
- net /SPI_CS5: track 134.6 -> 0.00 mm
- net /DAC_VCA5: track 121.5 -> 0.00 mm, vias 2 -> 0
- net /DAC_MIXN: track 114.5 -> 0.00 mm, vias 2 -> 0
- net /DAC_FC5: track 110.2 -> 0.00 mm, vias 2 -> 0
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
Commit message: hardware: improved routing
Routing:
- net GND: track 60.6 -> 1263.1 mm
- net +5V: track 8.94 -> 662.3 mm, vias 0 -> 18
- net -5V: track 0.00 -> 557.5 mm, vias 0 -> 12
- net +3.3V: track 38.9 -> 433.4 mm, vias 0 -> 7
- net SPI_MOSI: track 0.00 -> 235.7 mm, vias 0 -> 6
- net SPI_SCK: track 0.00 -> 215.5 mm, vias 0 -> 4
- net DAC_MIXB: track 0.00 -> 185.5 mm, vias 0 -> 6
- net DAC_MIXA: track 0.00 -> 161.2 mm, vias 0 -> 6
- net Net-(U6D--): track 0.00 -> 147.9 mm, vias 0 -> 3
- net DAC_RES: track 0.00 -> 147.6 mm, vias 0 -> 7
- net /ADC_MIX: track 0.00 -> 144.2 mm, vias 0 -> 2
- net /SPI_CS5: track 0.00 -> 133.9 mm
- net /DAC_VCA5: track 0.00 -> 122.6 mm, vias 0 -> 2
- net /DAC_MIXN: track 0.00 -> 113.4 mm, vias 0 -> 2
- net /DAC_FC5: track 0.00 -> 108.0 mm, vias 0 -> 2
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
Commit message: Manual PCB routing by Guimli WIP
Parts:
- removed the C34 at (85.9, 70.2)
- added C34: 100n, Capacitor_SMD:C_0805_2012Metric, F.Cu at (110.7, 96.0)
- added C34: 100n, Capacitor_SMD:C_0805_2012Metric, F.Cu at (244.0, 108.7)
- moved U7 163.6 mm to (249.1, 108.7), turned to -90 degrees
- moved P1 79.4 mm to (113.3, 114.4), turned to 180 degrees
- moved R6 77.7 mm to (117.1, 108.0), turned to 90 degrees
- moved C21 73.2 mm to (97.3, 80.3), turned to 0 degrees
- moved R1 67.1 mm to (50.1, 102.3)
- moved C22 65.6 mm to (89.7, 80.3)
- moved R22 65.5 mm to (118.3, 92.0)
- moved R5 64.3 mm to (68.3, 99.1)
- moved R3 62.4 mm to (50.1, 99.3)
- moved D1 61.0 mm to (257.6, 123.6), turned to 90 degrees
- moved U1 59.1 mm to (114.1, 125.3), turned to -90 degrees
- moved C8 57.7 mm to (50.1, 96.3)
- moved C23 55.6 mm to (99.8, 134.8), turned to 0 degrees
- moved D2 55.4 mm to (257.6, 117.3), turned to 90 degrees
- moved C54 54.2 mm to (152.2, 116.3)
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Connections:
- U1 pad 9: unconnected-(U1-NC-Pad9) -> GND
- U10 pad 3: /SPI_CS3 -> /SPI_CS4
- U12 pad 3: /SPI_CS1 -> /SPI_CS2
- U14 pad 3: /SPI_CS4 -> /SPI_CS5
- U16 pad 3: /SPI_CS2 -> /SPI_CS3
- U18 pad 3: /SPI_CS5 -> /SPI_CS6
- U20 pad 10: /DAC_FC4 -> /DAC_FC2
- U20 pad 11: /DAC_FC5 -> /DAC_VCA0
- U20 pad 12: DAC_MIXA -> /DAC_VCA1
- U20 pad 13: DAC_MIXB -> /DAC_VCA2
- U20 pad 2: /SPI_CS7 -> /SPI_CS0
- U20 pad 4: /DAC_FC0 -> DAC_MIXB
- U20 pad 5: /DAC_FC1 -> DAC_MIXA
- U20 pad 6: /DAC_FC2 -> /DAC_FC0
- U20 pad 7: /DAC_FC3 -> /DAC_FC1
- U7 pad 10: /DAC_VCA4 -> DAC_RES
- U7 pad 11: /DAC_VCA5 -> /DAC_FC3
- U7 pad 12: /DAC_MIXN -> /DAC_FC4
- U7 pad 13: DAC_RES -> /DAC_FC5
- U7 pad 2: /SPI_CS6 -> /SPI_CS7
- U7 pad 4: /DAC_VCA0 -> /DAC_MIXN
- U7 pad 5: /DAC_VCA1 -> /DAC_VCA3
- U7 pad 6: /DAC_VCA2 -> /DAC_VCA4
- U7 pad 7: /DAC_VCA3 -> /DAC_VCA5
- U8 pad 3: /SPI_CS0 -> /SPI_CS1
Routing:
- net GND: track 1263.1 -> 208.8 mm, vias 0 -> 177
- net +3.3V: track 433.4 -> 51.3 mm, vias 7 -> 2
- net /SPI_CS7: track 25.6 -> 159.7 mm, vias 2 -> 0
- net +5V: track 662.3 -> 529.8 mm, vias 18 -> 6
- net /DAC_VCA5: track 122.6 -> 17.2 mm, vias 2 -> 0
- net /DAC_MIXN: track 113.4 -> 13.7 mm, vias 2 -> 0
- net /DAC_FC5: track 108.0 -> 18.6 mm
- net -5V: track 557.5 -> 468.9 mm, vias 12 -> 11
- net /PROG_TXD: track 68.5 -> 3.05 mm, vias 2 -> 0
- net /PROG_RXD: track 69.8 -> 4.63 mm, vias 2 -> 0
- net NOISE: track 106.3 -> 167.3 mm, vias 6 -> 2
- net /FOOT_IN: track 57.2 -> 0.00 mm, vias 2 -> 0
- net /SPI_CS6: track 51.7 -> 105.0 mm, vias 2 -> 0
- net /RESET: track 55.6 -> 3.03 mm, vias 2 -> 0
- net /DAC_VCA4: track 99.1 -> 46.5 mm
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- added copper zone on B.Cu, net GND
- added copper zone on F.Cu, net GND
Other:
- board size 200.7 x 99.1 mm -> 217 x 97 mm

Commit message: Manual PCB routing by Guimli WIP2
Parts:
- removed C28: 100n, Capacitor_SMD:C_0805_2012Metric
- moved C30 40.4 mm to (119.7, 125.3), turned to 90 degrees
- moved R1 11.2 mm to (59.5, 96.2), turned to 180 degrees
- moved C8 11.2 mm to (59.5, 102.3), turned to 180 degrees
- moved SW1 11.1 mm to (50.3, 102.5), turned to 90 degrees
- moved R6 10.9 mm to (109.0, 100.8), turned to -90 degrees
- moved C31 9.87 mm to (52.6, 80.5)
- moved R3 9.45 mm to (59.5, 99.2), turned to 180 degrees
- moved C21 8.73 mm to (88.6, 80.5), turned to 180 degrees
- moved C22 6.67 mm to (96.4, 80.5), turned to 180 degrees
- moved R16 6.20 mm to (99.8, 73.6)
- moved C37 6.18 mm to (99.8, 67.2)
- moved R5 6.14 mm to (74.1, 101.1)
- moved R2 5.36 mm to (69.0, 101.1)
- moved R4 5.36 mm to (71.6, 101.1)
- moved FB1 3.42 mm to (60.2, 73.8), turned to 0 degrees
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Connections:
- net /USB_DM renamed /USB_D-
- net /USB_DP renamed /USB_D+
- net Net-(J1-D+) renamed /D+
- net Net-(J1-D-) renamed /D-
- U1 pad 9: GND -> unconnected-(U1-NC-Pad9)
Routing:
- net +3.3V: track 51.3 -> 457.4 mm, vias 2 -> 1
- net +5V: track 529.8 -> 593.1 mm, vias 6 -> 14
- net /FOOT_IN: track 0.00 -> 61.2 mm, vias 0 -> 2
- net /USB_GND: track 0.00 -> 56.2 mm
- net /D+: track 0.00 -> 43.6 mm, vias 0 -> 1
- net /D-: track 0.00 -> 39.7 mm, vias 0 -> 1
- net /RESET: track 3.03 -> 38.9 mm, vias 0 -> 2
- net /USB_D-: track 0.00 -> 21.1 mm
- net /USB_D+: track 0.00 -> 20.4 mm
- net /USB_5V: track 22.6 -> 38.7 mm
- net Net-(R1-Pad2): track 3.02 -> 14.4 mm
- net Net-(J2-PadT): track 16.2 -> 24.8 mm
- net SPI_SCK: track 247.0 -> 240.8 mm
- net /PROG_TXD: track 3.05 -> 9.24 mm
- net SPI_MOSI: track 243.4 -> 237.4 mm
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
Commit message: Manual PCB routing by Guimli WIP3
Parts:
- moved R6 16.5 mm to (118.4, 114.4), turned to 180 degrees
- moved P1 12.7 mm to (113.3, 101.7), turned to 0 degrees
- moved R25 0.95 mm to (92.2, 135.1)
- moved R26 0.53 mm to (116.4, 82.2)
Connections:
- U1 pad 9: unconnected-(U1-NC-Pad9) -> GND
Routing:
- net +3.3V: track 457.4 -> 468.1 mm, vias 1 -> 2
- net +5V: track 593.1 -> 585.5 mm
- net /PROG_TXD: track 9.24 -> 15.6 mm
- net SPI_SCK: track 240.8 -> 246.7 mm
- net /SPI_MUX_C: track 36.8 -> 42.6 mm
- net /FOOT_IN: track 61.2 -> 57.8 mm
- net Net-(D5-A): track 56.6 -> 54.0 mm
- net /ADC_MIX: track 142.4 -> 139.9 mm
- net /PROG_BOOT: track 44.1 -> 45.9 mm, vias 2 -> 1
- net /ADC_SPI_MOSI: track 49.4 -> 47.9 mm
- net /SPI_MUX_B: track 40.6 -> 42.1 mm
- net /ADC_SPI_SCK: track 51.1 -> 49.8 mm
- net /LCD_CTRST: track 29.1 -> 27.9 mm
- net /ADC_SPI_SSEL: track 46.0 -> 47.1 mm
- net /SPI_CS0: track 33.6 -> 32.7 mm
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