File: hardware/overcycler3.kicad_pcb (KiCad board)
At the start: 2 copper layers, 601 x 380.4 mm, 347 parts, among them IC1 LM13700, IC2 LM13700, IC3 LM13700, J1 USB_B, J10 Control_Down, J2 AudioJack3_Switch, J3 DIN-5_180degree, J4 AudioJack3_Switch, J5 AudioJack3_Switch, J6 Control_Up, J7 Keyboard, J8 Display, J9 FT232, Q1 2SC945, SW1 RESET, SW2 POWER, U1 XT26G02CWSIGA, U10 MCP4922-ESL, U11 SSI2144, U12 MCP4922-ESL, U13 SSI2144, U14 MCP4922-ESL, U15 SSI2144, U16 MCP4922-ESL, U17 SSI2144, U18 MCP4922-ESL, U19 SSI2144, U2 TL064, U20 AD5328B, U3 LPC1778FBD144, U4 TLV2556, U5 74HC138, U6 TL064, U7 AD5328B, U8 MCP4922-ESL, U9 SSI2144, Y1 12MHz

Commit message: hardware: sch/pcb updates by Guimli
Parts:
- removed U20: AD5328B, Package_SO:TSSOP-16_4.4x5mm_P0.65mm
- C20, C29: value 100n -> 10u; footprint Capacitor_SMD:C_0805_2012Metric -> Capacitor_Tantalum_SMD:CP_EIA-3216-18_Kemet-A
- U1: value XT26G02CWSIGA -> W25Q512JVFIQ; footprint Package_SON:WSON-8-1EP_8x6mm_P1.27mm_EP3.4x4.3mm -> Package_SO:SOIC-16W_7.5x10.3mm_P1.27mm
- U7: value AD5328B -> AD5674R; footprint Package_SO:TSSOP-16_4.4x5mm_P0.65mm -> Additional:LFCSP-28-1EP_4x4mm_P0.4mm_EP2.6x2.6mm_ThermalVias
- moved C112 663.2 mm to (324.6, 187.2)
- moved C2 625.6 mm to (315.6, 133.8), turned to 0 degrees
- moved C17 622.8 mm to (293.1, 133.8), turned to 0 degrees
- moved C116 611.3 mm to (297.2, 122.7)
- moved C114 591.6 mm to (264.5, 145.9), turned to 180 degrees
- moved R12 584.1 mm to (317.6, 189.4), turned to 180 degrees
- moved C35 583.4 mm to (317.6, 179.9), turned to 180 degrees
- moved Q1 582.5 mm to (319.5, 174.5), turned to -90 degrees
- moved R9 582.1 mm to (317.6, 183.0), turned to 180 degrees
- moved R7 581.7 mm to (321.4, 179.2), turned to -90 degrees
- moved R10 580.1 mm to (317.6, 186.2), turned to 0 degrees
- moved R11 577.7 mm to (314.4, 173.5), turned to 0 degrees
- moved R15 577.7 mm to (314.4, 176.7), turned to 180 degrees
- moved R13 575.4 mm to (313.1, 191.3), turned to 180 degrees
- moved R8 574.8 mm to (317.2, 170.3), turned to 180 degrees
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- renumbered C7 to C115, C3 to C116, C7 to C117, C5 to C7
Connections:
- C112 pad 1: DAC_MIXB -> /DAC_MIXN
- C113 pad 1: /DAC_MIXN -> DAC_MIXB
- C18 pad 1: +3.3V -> +5V
- C19 pad 1: +3.3V -> +3V3
- C20 pad 1: +3.3V -> +5V
- C23 pad 1: +3.3V -> +3V3
- C24 pad 1: +3.3V -> +3V3
- C25 pad 1: +3.3V -> +3V3
- C26 pad 1: +3.3V -> +3V3
- C27 pad 1: +3.3V -> +3V3
- C28 pad 1: +3.3V -> +3V3
- C29 pad 1: +3.3V -> +3V3
- C30 pad 1: +3.3V -> +3V3
- C32 pad 1: +3.3V -> +3V3
- C34 pad 1: +5V -> +3V3
- C35 pad 2: Net-(U2A-+) -> Net-(U2D-+)
- J10 pad 2: /P_5 -> GND
- J10 pad 3: /P_6 -> /P_5
- J10 pad 4: /P_7 -> /P_6
- J10 pad 5: /P_8 -> /P_7
- J10 pad 6: /P_9 -> /P_8
- J10 pad 7: GND -> /P_9
- J6 pad 2: /P_0 -> GND
- J6 pad 3: /P_1 -> /P_0
- J6 pad 4: /P_2 -> /P_1
- J6 pad 5: /P_3 -> /P_2
- J6 pad 6: /P_4 -> /P_3
- J6 pad 7: GND -> /P_4
- R10 pad 1: Net-(U2B-+) -> Net-(U2C-+)
- R11 pad 2: Net-(U2A--) -> Net-(U2D--)
- R12 pad 2: Net-(U2B-+) -> Net-(U2C-+)
- R13 pad 1: Net-(U2B--) -> Net-(U2C--)
- R13 pad 2: Net-(U2C--) -> Net-(U2B--)
- R15 pad 1: Net-(U2A--) -> Net-(U2D--)
- R151 pad 2: Net-(U20-VOUTB) -> Net-(U7-VOUT6)
- R152 pad 1: /USB_GND -> /Power_Supply/USB_GND
- R152 pad 2: /D+ -> /Power_Supply/D+
- R17 pad 2: Net-(U2C--) -> Net-(U2B--)
- R18 pad 2: Net-(U2B--) -> Net-(U2C--)
- R2 pad 1: /USB_D- -> USB_D-
- R2 pad 2: /D- -> /Power_Supply/D-
- R23 pad 2: Net-(U2D--) -> Net-(U2A--)
- R24 pad 1: Net-(U2D--) -> Net-(U2A--)
- R4 pad 1: /USB_D+ -> USB_D+
- R4 pad 2: /D+ -> /Power_Supply/D+
- R41 pad 2: Net-(U7-VOUTA) -> Net-(U7-VOUT10)
- R42 pad 2: Net-(U20-VOUTA) -> Net-(U7-VOUT7)
- R5 pad 1: /D+ -> /Power_Supply/D+
- R5 pad 2: /USB_5V -> /Power_Supply/USB_5V
- R9 pad 2: Net-(U2A-+) -> Net-(U2D-+)
- U1 pad 1: /FLASH_SPI_SSEL -> +3V3
- U1 pad 2: /FLASH_SPI_MISO -> +3V3
- U1 pad 4: GND -> unconnected-(U1-NC-Pad4)
- U1 pad 5: /FLASH_SPI_MOSI -> unconnected-(U1-NC-Pad5)
- U1 pad 6: /FLASH_SPI_SCK -> unconnected-(U1-NC-Pad6)
- U1 pad 7: +3V3 -> /FLASH_SPI_SSEL
- U1 pad 8: +3V3 -> /FLASH_SPI_MISO
- U1 pad 9: GND -> +3V3
- U2 pad 1: Net-(R15-Pad2) -> Net-(C48-Pad1)
- U2 pad 10: GND -> Net-(U2C-+)
- U2 pad 12: Net-(D2-K) -> Net-(U2D-+)
- U2 pad 14: Net-(C48-Pad1) -> Net-(R15-Pad2)
- U2 pad 3: Net-(U2A-+) -> Net-(D2-K)
- U2 pad 5: Net-(U2B-+) -> GND
- U2 pad 7: Net-(U2B--) -> Net-(R17-Pad1)
- U2 pad 8: Net-(R17-Pad1) -> Net-(U2C--)
- U5 pad 7: /SPI_CS7 -> unconnected-(U5-~{Y7}-Pad7)
- U7 pad 1: +5V -> /DAC_VCA0
- U7 pad 10: DAC_RES -> /DAC_FC0
- U7 pad 11: /DAC_FC3 -> /DAC_FC1
- U7 pad 12: /DAC_FC4 -> /DAC_FC2
- U7 pad 13: /DAC_FC5 -> /DAC_FC3
- U7 pad 14: GND -> /DAC_FC4
- U7 pad 15: SPI_MOSI -> GND
- U7 pad 16: SPI_SCK -> GND
- U7 pad 2: /SPI_CS7 -> +5V
- U7 pad 3: +5V -> /SPI_CS0
- U7 pad 4: Net-(U7-VOUTA) -> SPI_SCK
- U7 pad 5: /DAC_VCA3 -> SPI_MOSI
- U7 pad 6: /DAC_VCA4 -> +3V3
- U7 pad 7: /DAC_VCA5 -> Net-(U7-VOUT7)
- U7 pad 8: +5V -> Net-(U7-VOUT6)
- U7 pad 9: +5V -> DAC_RES
Routing:
- net +3.3V: track 455.9 -> 0.00 mm
- net -5V: track 491.0 -> 246.9 mm, vias 11 -> 8
- net Net-(U7-VOUT10): track 0.00 -> 211.5 mm
- net /SPI_CS7: track 159.7 -> 0.00 mm
- net +5V: track 604.4 -> 457.0 mm, vias 14 -> 15
- net /DAC_VCA5: track 17.2 -> 144.6 mm
- net GND: track 193.9 -> 77.7 mm, vias 285 -> 148
- net /DAC_FC5: track 18.6 -> 130.1 mm, vias 2 -> 0
- net /ADC_MIX: track 114.3 -> 8.97 mm, vias 2 -> 1
- net SPI_SCK: track 246.7 -> 146.5 mm, vias 9 -> 7
- net SPI_MOSI: track 236.8 -> 142.3 mm, vias 9 -> 7
- net +3V3: track 0.00 -> 86.2 mm, vias 0 -> 2
- net /DAC_VCA4: track 46.5 -> 120.3 mm, vias 2 -> 0
- net /DAC_FC4: track 35.8 -> 103.1 mm, vias 2 -> 0
- net DAC_RES: track 199.5 -> 135.1 mm, vias 10 -> 0
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- removed copper zone on B.Cu, net GND
- removed copper zone on F.Cu, net GND
Other:
- board size 601 x 380.4 mm -> 233.7 x 168.2 mm

Commit message: hardware: sch/pcb updates by Guimli
Parts:
- removed the C10 at (-74.5, 126.4)
- removed the C11 at (236.3, 150.0)
- removed the C12 at (-70.0, 111.4)
- removed the C12 at (258.8, 150.0)
- removed the C14 at (281.4, 150.0)
- removed the C15 at (303.9, 150.0)
- removed the C16 at (326.5, 150.0)
- removed the C17 at (-70.0, 123.4)
- removed the C18 at (-70.0, 126.4)
- removed the C19 at (-65.6, 108.4)
- removed the C2 at (270.5, 133.8)
- removed the C20 at (142.2, 89.9)
- removed the C23 at (164.7, 155.2)
- removed the C24 at (-65.6, 117.4)
- removed the C25 at (-65.6, 120.4)
- removed the C26 at (-65.6, 123.4)
- removed the C27 at (-65.6, 126.4)
- removed the C28 at (-46.5, 101.8)
- removed the C28 at (-61.1, 108.4)
- removed the C29 at (119.5, 111.4)
- removed the C30 at (-61.1, 111.4)
- removed the C30 at (-26.7, 206.5)
- removed the C32 at (-94.4, 198.1)
- removed the C34 at (-61.1, 120.4)
- removed the C4 at (202.3, 133.8)
- removed the C6 at (292.4, 81.2)
- removed the R152 at (-71.3, 149.3)
- removed the R2 at (-55.7, 90.3)
- removed the R4 at (-55.7, 93.2)
- removed the R5 at (-55.7, 96.2)
- added C118: 100nF, Capacitor_SMD:C_0805_2012Metric, F.Cu at (207.0, 122.7)
- added C119: 100nF, Capacitor_SMD:C_0805_2012Metric, F.Cu at (229.6, 122.7)
- added C12: 100nF, Capacitor_SMD:C_0805_2012Metric, F.Cu at (236.3, 150.0)
- added C120: 100nF, Capacitor_SMD:C_0805_2012Metric, F.Cu at (252.1, 122.7)
- added C121: 100nF, Capacitor_SMD:C_0805_2012Metric, F.Cu at (247.3, 133.8)
- added C122: 100nF, Capacitor_SMD:C_0805_2012Metric, F.Cu at (202.3, 133.8)
- added C123: 100nF, Capacitor_SMD:C_0805_2012Metric, F.Cu at (269.9, 133.8)
- added C124: 100nF, Capacitor_SMD:C_0805_2012Metric, F.Cu at (315.0, 133.8)
- added C125: 100nF, Capacitor_SMD:C_0805_2012Metric, F.Cu at (326.5, 150.0)
- added C28: 100nF, Capacitor_SMD:C_0805_2012Metric, F.Cu at (133.7, 152.9)
- added C30: 100nF, Capacitor_SMD:C_0805_2012Metric, F.Cu at (164.7, 155.3)
- C10, C11, C14, C15, C16, C17, C18, C19, C22, C23, C24, C25, C26, C27, C31, C32, C34: value 100n -> 100nF
- C115, C116, C117: value 10n -> 100nF
- C13: value 470u -> 470uF
- C2, C3, C4, C5, C6, C7: value 10n -> 10nF
- C20, C21, C29: value 10u -> 10uF
- J10, J6: footprint Connector_JST:JST_XH_B7B-XH-A_1x07_P2.50mm_Vertical -> Connector_JST:JST_PH_B7B-PH-K_1x07_P2.00mm_Vertical
- moved C16 375.1 mm to (303.9, 150.0), turned to 90 degrees
- moved C15 352.9 mm to (281.4, 150.0), turned to 90 degrees
- moved C11 331.5 mm to (258.8, 150.0), turned to 90 degrees
- moved C4 296.1 mm to (263.5, 98.6), turned to 180 degrees
- moved C31 258.9 mm to (195.3, 150.3), turned to 180 degrees
- moved C32 250.3 mm to (185.7, 159.4), turned to -90 degrees
- moved R5 241.7 mm to (161.4, 76.0)
- moved C49 227.1 mm to (138.5, 170.6)
- moved L1 224.2 mm to (139.5, 165.2), turned to 90 degrees
- moved R2 222.5 mm to (139.0, 130.3)
- moved R4 222.2 mm to (141.2, 130.3)
- moved R25 221.2 mm to (163.4, 176.4), turned to 0 degrees
- moved R6 214.6 mm to (178.8, 138.5)
- moved R152 213.9 mm to (156.9, 76.0)
- moved J9 212.5 mm to (178.8, 119.5)
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Connections:
- U3 pad 132: /ADC_SPI_SSEL -> /SPI_SSEL
- U3 pad 133: /ADC_SPI_MISO -> unconnected-(U3-P1[4]-Pad133)
- U3 pad 135: /ADC_SPI_MOSI -> SPI_MOSI
- U3 pad 136: /ADC_SPI_SCK -> SPI_SCK
- U3 pad 26: (no net) -> unconnected-(U3-RTC_ALARM-Pad26)
- U3 pad 49: SPI_SCK -> /ADC_SPI_SCK
- U3 pad 50: /SPI_SSEL -> /ADC_SPI_SSEL
- U3 pad 53: unconnected-(U3-P1[23]-Pad53) -> /ADC_SPI_MISO
- U3 pad 54: SPI_MOSI -> /ADC_SPI_MOSI
Routing:
- net -5V: track 246.9 -> 581.1 mm, vias 8 -> 21
- net +5V: track 457.0 -> 714.2 mm, vias 15 -> 22
- net /KP_8_C4: track 6.76 -> 212.0 mm
- net /KP_5_C1: track 10.1 -> 200.2 mm
- net /KP_1_R1: track 1.98 -> 186.4 mm
- net /KP_3_R3: track 5.17 -> 183.4 mm
- net /KP_2_R2: track 5.87 -> 182.5 mm
- net /KP_4_R4: track 8.17 -> 184.6 mm
- net /KP_6_C2: track 0.00 -> 155.3 mm, vias 0 -> 1
- net /KP_7_C3: track 4.41 -> 158.6 mm, vias 0 -> 1
- net /Power_Supply/D+: track 0.00 -> 81.6 mm
- net /Power_Supply/D-: track 0.00 -> 80.2 mm
- net +3V3: track 86.2 -> 163.1 mm
- net /Power_Supply/USB_GND: track 0.00 -> 68.7 mm
- net /P_9: track 0.00 -> 58.2 mm
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