File: hardware/voice3.kicad_sch (KiCad schematic)
At the start: 30 parts, among them IC1 LM13700, U12 MCP4922-ESL, U9 SSI2144

Commit message: hardware: CV DAC change -- misc changes -- draft routing
Parts:
- C75, C76, C77: footprint Capacitor_SMD:C_1206_3216Metric -> Capacitor_SMD:C_0603_1608Metric
Changed lines of the file:
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@@
       (effects (font (size 1.016 1.016)) (justify left))
     )
-    (property "Footprint" "Capacitor_SMD:C_1206_3216Metric" (at 107.95 88.5952 0)
+    (property "Footprint" "Capacitor_SMD:C_0603_1608Metric" (at 107.95 88.5952 0)
       (effects (font (size 0.762 0.762)) hide)
     )
@@
       (effects (font (size 1.016 1.016)) (justify left))
     )
-    (property "Footprint" "Capacitor_SMD:C_1206_3216Metric" (at 107.95 96.2152 0)
+    (property "Footprint" "Capacitor_SMD:C_0603_1608Metric" (at 107.95 96.2152 0)
       (effects (font (size 0.762 0.762)) hide)
     )
@@
       (effects (font (size 1.016 1.016)) (justify left))
     )
-    (property "Footprint" "Capacitor_SMD:C_1206_3216Metric" (at 115.57 101.9048 0)
+    (property "Footprint" "Capacitor_SMD:C_0603_1608Metric" (at 115.57 101.9048 0)
       (effects (font (size 0.762 0.762)) hide)
     )

Commit message: hardware: chnaged some capacitor values and footprints
Parts:
- C72, C73: footprint Capacitor_Tantalum_SMD:CP_EIA-3216-18_Kemet-A -> Capacitor_SMD:C_0805_2012Metric
- C79: value 33u -> 47u; footprint Capacitor_Tantalum_SMD:CP_EIA-3216-18_Kemet-A -> Capacitor_SMD:C_1206_3216Metric
Changed lines of the file:
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@@
       (effects (font (size 1.27 1.27)) (justify left))
     )
-    (property "Value" "33u" (at 168.91 96.52 0)
-      (effects (font (size 1.27 1.27)) (justify left))
-    )
-    (property "Footprint" "Capacitor_Tantalum_SMD:CP_EIA-3216-18_Kemet-A" (at 166.37 97.79 0)
+    (property "Value" "47u" (at 168.91 96.52 0)
+      (effects (font (size 1.27 1.27)) (justify left))
+    )
+    (property "Footprint" "Capacitor_SMD:C_1206_3216Metric" (at 166.37 97.79 0)
       (effects (font (size 1.524 1.524)) hide)
     )
@@
       (effects (font (size 1.27 1.27)) (justify left))
     )
-    (property "Footprint" "Capacitor_Tantalum_SMD:CP_EIA-3216-18_Kemet-A" (at 71.12 91.44 0)
+    (property "Footprint" "Capacitor_SMD:C_0805_2012Metric" (at 71.12 91.44 0)
       (effects (font (size 1.524 1.524)) hide)
     )
@@
       (effects (font (size 1.27 1.27)) (justify left))
     )
-    (property "Footprint" "Capacitor_Tantalum_SMD:CP_EIA-3216-18_Kemet-A" (at 71.12 99.06 0)
-      (effects (font (size 1.524 1.524)) hide)
-    )
+    (property "Footprint" "Capacitor_SMD:C_0805_2012Metric" (at 71.12 99.06 0)
+      (effects (font (size 1.524 1.524)) hide)
+    )

Commit message: Manual PCB routing by Guimli Done!
Parts:
- U9: footprint Package_SO:SSOP-16_3.9x4.9mm_P0.635mm -> Additional:SSOP-16_3.9x4.9mm_P0.635mm
Changed lines of the file:
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@@
       (effects (font (size 1.27 1.27)))
     )
-    (property "Footprint" "Package_SO:SSOP-16_3.9x4.9mm_P0.635mm" (at 157.48 100.33 0)
+    (property "Footprint" "Additional:SSOP-16_3.9x4.9mm_P0.635mm" (at 157.48 100.33 0)
       (effects (font (size 1.27 1.27)) hide)
     )

Commit message: hardware: Adding LCSC references
Parts:
- C72, C73: LCSC (none) -> C45783
- C74, C80: LCSC (none) -> C13967
- C75, C76, C77: LCSC (none) -> C5299898
- C78: LCSC (none) -> C519567
- C79: LCSC (none) -> C96123
- C81: LCSC (none) -> C16133
- IC1: LCSC (none) -> C5160094
- R, R87, R91: LCSC (none) -> C17475
- R, R98: LCSC (none) -> C17560
- R, R90, R97: LCSC (none) -> C17837
- R86: LCSC (none) -> C17772
- R89: LCSC (none) -> C17655
- R92, R96, R99: LCSC (none) -> C17673
- R93: LCSC (none) -> C17414
- R94, R95: LCSC (none) -> C17710
- U12: LCSC (none) -> C39851
- U9: LCSC (none) -> C9900070109
Changed lines of the file:
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@@
       (effects (font (size 1.524 1.524)))
+    )
+    (property "LCSC" "C5299898" (at 114.3 87.63 0)
+      (effects (font (size 1.27 1.27)) hide)
     )
     (pin "1")
@@
       (effects (font (size 1.524 1.524)))
     )
+    (property "LCSC" "C5299898" (at 114.3 95.25 0)
+      (effects (font (size 1.27 1.27)) hide)
+    )
     (pin "1")
     (pin "2")
@@
       (effects (font (size 1.524 1.524)))
     )
+    (property "LCSC" "C5299898" (at 109.22 102.87 0)
+      (effects (font (size 1.27 1.27)) hide)
+    )
     (pin "1")
     (pin "2")
@@
       (effects (font (size 1.524 1.524)))
     )
+    (property "LCSC" "C519567" (at 109.22 110.49 0)
+      (effects (font (size 1.27 1.27)) hide)
+    )
     (pin "1")
     (pin "2")
@@
       (effects (font (size 0.762 0.762)))
     )
+    (property "LCSC" "C17837" (at 97.028 107.95 0)
+      (effects (font (size 1.27 1.27)) hide)
+    )
     (pin "1")
     (pin "2")
@@
       (effects (font (size 0.762 0.762)))
     )
+    (property "LCSC" "C17655" (at 96.012 129.54 0)
+      (effects (font (size 1.27 1.27)) hide)
+    )
     (pin "1")
     (pin "2")
@@
       (effects (font (size 0.762 0.762)))
     )
+    (property "LCSC" "C17475" (at 85.09 145.542 0)
+      (effects (font (size 1.27 1.27)) hide)
+    )
     (pin "1")
     (pin "2")
@@
       (effects (font (size 0.762 0.762)))
     )
+    (property "LCSC" "C17772" (at 85.09 119.888 0)
+      (effects (font (size 1.27 1.27)) hide)
+    )
     (pin "1")
     (pin "2")
@@
     (property "Datasheet" "~" (at 109.22 129.54 0)
       (effects (font (size 0.762 0.762)))
+    )
+    (property "LCSC" "C17475" (at 111.252 129.54 0)
+      (effects (font (size 1.27 1.27)) hide)
     )
     (pin "1")
@@
       (effects (font (size 1.524 1.524)))
     )
+    (property "LCSC" "C96123" (at 163.83 96.52 0)
+      (effects (font (size 1.27 1.27)) hide)
+    )
     (pin "1")
     (pin "2")
@@
     (property "Datasheet" "~" (at 158.75 106.68 0)
       (effects (font (size 0.762 0.762)))
+    )
+    (property "LCSC" "C17673" (at 160.782 106.68 0)
+      (effects (font (size 1.27 1.27)) hide)
     )
     (pin "1")
@@
     )
     (property "Datasheet" "http://ww1.microchip.com/downloads/en/devicedoc/21897a.pdf" (at 45.72 95.25 0)
+      (effects (font (size 1.27 1.27)) hide)
+    )
+    (property "LCSC" "C39851" (at 49.53 83.82 0)
       (effects (font (size 1.27 1.27)) hide)
     )
@@
       (effects (font (size 0.762 0.762)))
     )
+    (property "LCSC" "C17475" (at 85.09 89.408 0)
+      (effects (font (size 1.27 1.27)) hide)
+    )
     (pin "1")
     (pin "2")
@@
       (effects (font (size 1.524 1.524)))
     )
+    (property "LCSC" "C45783" (at 68.58 90.17 0)
+      (effects (font (size 1.27 1.27)) hide)
+    )
     (pin "1")
     (pin "2")
@@
       (effects (font (size 1.524 1.524)))
     )
+    (property "LCSC" "C45783" (at 68.58 97.79 0)
+      (effects (font (size 1.27 1.27)) hide)
+    )
     (pin "1")
     (pin "2")
@@
       (effects (font (size 0.762 0.762)))
     )
+    (property "LCSC" "C17475" (at 85.09 97.028 0)
+      (effects (font (size 1.27 1.27)) hide)
+    )
     (pin "1")
     (pin "2")
@@
       (effects (font (size 0.762 0.762)))
     )
+    (property "LCSC" "C17560" (at 85.09 81.788 0)
+      (effects (font (size 1.27 1.27)) hide)
+    )
     (pin "1")
     (pin "2")
@@
       (effects (font (size 0.762 0.762)))
     )
+    (property "LCSC" "C17837" (at 91.948 107.95 0)
+      (effects (font (size 1.27 1.27)) hide)
+    )
     (pin "1")
     (pin "2")
@@
     (property "Datasheet" "" (at 208.28 91.44 0)
       (effects (font (size 1.524 1.524)))
+    )
+    (property "LCSC" "C5160094" (at 204.47 99.06 0)
+      (effects (font (size 1.27 1.27)) hide)
     )
     (pin "10")
@@
       (effects (font (size 0.762 0.762)))
     )
+    (property "LCSC" "C17673" (at 207.01 119.888 0)
+      (effects (font (size 1.27 1.27)) hide)
+    )
     (pin "1")
     (pin "2")
@@
     (property "Datasheet" "~" (at 215.9 129.54 0)
       (effects (font (size 0.762 0.762)))
+    )
+    (property "LCSC" "C17837" (at 213.868 129.54 0)
+      (effects (font (size 1.27 1.27)) hide)
     )
     (pin "1")
@@
       (effects (font (size 1.524 1.524)))
     )
+    (property "LCSC" "C13967" (at 223.52 130.81 0)
+      (effects (font (size 1.27 1.27)) hide)
+    )
     (pin "1")
     (pin "2")
@@
       (effects (font (size 0.762 0.762)))
     )
+    (property "LCSC" "C17560" (at 228.092 99.06 0)
+      (effects (font (size 1.27 1.27)) hide)
+    )
     (pin "1")
     (pin "2")
@@
     (property "Datasheet" "~" (at 241.3 99.06 0)
       (effects (font (size 0.762 0.762)))
+    )
+    (property "LCSC" "C17673" (at 243.332 99.06 0)
+      (effects (font (size 1.27 1.27)) hide)
     )
     (pin "1")
@@
       (effects (font (size 1.524 1.524)))
     )
+    (property "LCSC" "C16133" (at 250.19 90.17 0)
+      (effects (font (size 1.27 1.27)) hide)
+    )
     (pin "1")
     (pin "2")
@@
     (property "Datasheet" "~" (at 180.34 97.79 0)
       (effects (font (size 0.762 0.762)))
+    )
+    (property "LCSC" "C17414" (at 180.34 95.758 0)
+      (effects (font (size 1.27 1.27)) hide)
     )
     (pin "1")
@@
       (effects (font (size 1.524 1.524)))
     )
+    (property "LCSC" "C13967" (at 101.6 130.81 0)
+      (effects (font (size 1.27 1.27)) hide)
+    )
     (pin "1")
     (pin "2")
@@
       (effects (font (size 0.762 0.762)))
     )
+    (property "LCSC" "C17710" (at 193.802 90.17 0)
+      (effects (font (size 1.27 1.27)) hide)
+    )
     (pin "1")
     (pin "2")
@@
     )
     (property "Datasheet" "http://www.soundsemiconductor.com/downloads/ssi2144datasheet.pdf" (at 152.4 104.14 0)
+      (effects (font (size 1.27 1.27)) hide)
+    )
+    (property "LCSC" "C9900070109" (at 152.4 94.1421 0)
       (effects (font (size 1.27 1.27)) hide)
     )
@@
       (effects (font (size 0.762 0.762)))
     )
-    (pin "1")
+    (property "LCSC" "C17710" (at 193.802 74.93 0)
+      (effects (font (size 1.27 1.27)) hide)
+    )
+    (pin "1")
