File: hardware/voice3.kicad_sch (KiCad schematic)
At the start: 30 parts, among them IC1 LM13700, U12 MCP4922-ESL, U9 SSI2144

Commit message: hardware: sch/pcb updates by Guimli
Parts:
- renumbered C73 to C100, C80 to C21, C74 to C35, C76 to C48, C77 to C49, C79 to C59, C75 to C67, C78 to C68, C81 to C8, C72 to C89, R90 to R100, R87 to R106, R83 to R114, R84 to R122, R88 to R123, R85 to R124, R98 to R24, R99 to R31, R97 to R32, R94 to R43, R95 to R50, R96 to R51, R89 to R69, R86 to R70, R91 to R71, R93 to R72, R92 to R93, U12 to U11, U9 to U3

Commit message: hardware: LCSC review, production files ok
Parts:
- R114: LCSC C17560 -> C17475
- R123: LCSC C17837 -> C17475
Changed lines of the file:
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@@
 			)
 		)
-		(property "LCSC" "C17560"
+		(property "LCSC" "C17475"
 			(at 100.33 74.168 0)
 			(effects
@@
 			)
 		)
-		(property "LCSC" "C17837"
+		(property "LCSC" "C17475"
 			(at 105.918 104.14 0)
 			(effects

Commit message: hardware: sch/pcb changes by Guimli (adding USB isolator, misc fixes)
Parts:
- C7: renamed from C8; footprint Capacitor_Tantalum_SMD:CP_EIA-3528-21_Kemet-B -> Additional:CP_EIA-3528-21_Kemet-B
- R113: renamed from R114; LCSC C17475 -> C17560
- R120: renamed from R123; LCSC C17475 -> C17837
- renumbered C21 to C20, C35 to C33, C48 to C46, C49 to C47, C59 to C58, C67 to C65, C68 to C66, C89 to C87, C100 to C88, R106 to R105, R122 to R119, R124 to R121, R24 to R23, R32 to R29, R31 to R30, R43 to R42, R51 to R48, R50 to R49, R69 to R65, R70 to R66, R71 to R67, R72 to R68, R93 to R92, R100 to R99, U11 to U10
Connections:
- net at C20.2, R29.2, R48.2: now also IC1.16; no longer IC1.1
- net at R49.2, R68.2: now also IC1.14 (+); no longer IC1.3 (+)
- net at R42.1: now also IC1.13 (-); no longer IC1.4 (-)
- net at IC1.10, R23.1: now also IC1.12; no longer IC1.5

Commit message: hardware: voice mixer -> 820 ohms
Parts:
- R120: value 15k -> 820
Changed lines of the file:
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@@
 			)
 		)
-		(property "Value" "15k"
+		(property "Value" "820"
 			(at 107.95 104.14 90)
 			(effects
