File: hardware/overcycler3.kicad_sch (KiCad schematic)
At the start: 127 parts, among them J1 USB_B, J2 AudioJack3_Switch, J3 DIN-5_180degree, J4 AudioJack3_Switch, J5 AudioJack3_Switch, P1 FT232, P2 PANEL, Q1 2SC945, SW1 RESET, SW2 POWER, U1 XT26G02ELGIGA, U2 TL074, U3 LPC1778FBD144, U4 TLV1543, U5 74HC138, U6 TL074, U7 AD5674R, Y1 12MHz

Commit message: hardware: beginning of overcycler 3 PCB
Parts:
- SW1: footprint Button_Switch_THT:SW_Tactile_SPST_Angled_PTS645Vx83-2LFS -> Button_Switch_THT:SW_PUSH_6mm

Commit message: hardware: CV DAC change -- misc changes -- draft routing
Parts:
- removed U7: AD5674R, Package_DFN_QFN:QFN-28-1EP_4x4mm_P0.4mm_EP2.6x2.6mm, symbol AD5674R:AD5674R
- added U20, U7: AD5328B, Package_SO:TSSOP-16_4.4x5mm_P0.65mm, symbol AD5328B:AD5328B
- Y1: footprint Crystal:Crystal_SMD_HC49-SD -> Crystal:Crystal_SMD_ECS_CSM3X-2Pin_7.6x4.1mm
Connections:
- net +3.3V: no longer C34.1
- net +5V: now also C34.1, U20.3 (VDD), U20.8 (VREFABCD), U20.9 (VREFEFGH), U7.3 (VDD), U7.8 (VREFABCD), U7.9 (VREFEFGH)
- net DAC_FC0: now also U20.4 (VOUTA)
- net DAC_FC1: now also U20.5 (VOUTB)
- net DAC_FC2: now also U20.6 (VOUTC)
- net DAC_FC3: now also U20.7 (VOUTD)
- net DAC_FC4: now also U20.10 (VOUTE)
- net DAC_FC5: now also U20.11 (VOUTF)
- net DAC_MIXA: now also U20.12 (VOUTG)
- net DAC_MIXB: now also U20.13 (VOUTH)
- net DAC_MIXN: now also U7.12 (VOUTG)
- net DAC_RES: now also U7.13 (VOUTH)
- net DAC_VCA0: now also U7.4 (VOUTA)
- net DAC_VCA1: now also U7.5 (VOUTB)
- net DAC_VCA2: now also U7.6 (VOUTC)
- net DAC_VCA3: now also U7.7 (VOUTD)
- net DAC_VCA4: now also U7.10 (VOUTE)
- net DAC_VCA5: now also U7.11 (VOUTF)
- net GND: now also U20.1 (/LDAC), U20.14 (GND), U7.1 (/LDAC), U7.14 (GND)
- net SPI_MOSI: now also U20.15 (DIN), U7.15 (DIN)
- net SPI_SCK: now also U20.16 (SCLK), U7.16 (SCLK)
- net SPI_CS7: now reaches U5.7 (O7)
- net SPI_CS7: now also U20.2 (/SYNC)
- net SPI_CS6: now reaches U5.9 (O6)
- net SPI_CS6: now also U7.2 (/SYNC)
- net USB_5V: now reaches C13.1, PS1.1 (+Vin), PS2.1 (+Vin)
- net USB_5V: now also SW2.3 (C), SW2.6 (C); no longer SW2.1 (A), SW2.4 (A)
- net USB_GND: now reaches C13.2, FB1.2, J1.4 (GND), PS1.2 (-Vin), PS2.2 (-Vin)
- net USB_VBUS: now reaches J1.1 (VBUS), SW2.2 (B), SW2.5 (B)
- net CV_SPI_MISO: no longer names the net of U3.133 (P1[4])
- net CV_SPI_MOSI: no longer names the net of U3.135 (P1[1])
- net CV_SPI_SCK: no longer names the net of U3.136 (P1[0])
- net CV_SPI_SSEL: no longer names the net of U3.132 (P1[8])
Other:
- moved on the sheet: C18, C19, C20, C23, C24, C25, C26, C27, C28, C29, C30, C32

Commit message: hardware: TLV2556 ADC in SPI -- improved draft routing
Parts:
- removed R41: 1k, Resistor_SMD:R_0805_2012Metric, symbol overcycler2-rescue:R
- U4: value TLV1543 -> TLV2556
Connections:
- net ADC_SPI_SSEL: now reaches U3.132 (P1[8])
- net ADC_SPI_SSEL: now also U4.15 (/CS)
- net ADC_SPI_MISO: now reaches U3.133 (P1[4])
- net ADC_SPI_MISO: now also U4.16 (DATA_OUT)
- net ADC_SPI_MOSI: now reaches U3.135 (P1[1])
- net ADC_SPI_MOSI: now also U4.17 (DATA_IN)
- net ADC_SPI_SCK: now reaches U3.136 (P1[0])
- net ADC_SPI_SCK: now also U4.18 (I/O_CLOCK)
- net ADC_ADDR: no longer names the net of U3.10 (P0[25])
- net ADC_ADDR: no longer U4.17 (ADDRESS)
- net ADC_CLK: no longer names the net of U3.35 (P0[27])
- net ADC_CLK: no longer U4.18 (I/O_CLOCK)
- net ADC_CS: no longer names the net of U3.13 (P0[23])
- net ADC_CS: no longer U4.15 (/CS)
- net ADC_EOC: no longer names the net of U4.19 (EOC)
- net ADC_EOC: no longer U3.34 (P0[28])
- net ADC_OUT: no longer names the net of U3.11 (P0[24])
- net ADC_OUT: no longer U4.16 (DATA_OUT)
Other:
- moved on the sheet: C49, R42

Commit message: Manual PCB routing by Guimli WIP
Connections:
- net DAC_FC0: now also U20.6 (VOUTC); no longer U20.4 (VOUTA)
- net DAC_FC1: now also U20.7 (VOUTD); no longer U20.5 (VOUTB)
- net DAC_FC2: now also U20.10 (VOUTE); no longer U20.6 (VOUTC)
- net DAC_FC3: now also U7.11 (VOUTF); no longer U20.7 (VOUTD)
- net DAC_FC4: now also U7.12 (VOUTG); no longer U20.10 (VOUTE)
- net DAC_FC5: now also U7.13 (VOUTH); no longer U20.11 (VOUTF)
- net DAC_MIXA: now also U20.5 (VOUTB); no longer U20.12 (VOUTG)
- net DAC_MIXB: now also U20.4 (VOUTA); no longer U20.13 (VOUTH)
- net DAC_MIXN: now also U7.4 (VOUTA); no longer U7.12 (VOUTG)
- net DAC_RES: now also U7.10 (VOUTE); no longer U7.13 (VOUTH)
- net DAC_VCA0: now also U20.11 (VOUTF); no longer U7.4 (VOUTA)
- net DAC_VCA1: now also U20.12 (VOUTG); no longer U7.5 (VOUTB)
- net DAC_VCA2: now also U20.13 (VOUTH); no longer U7.6 (VOUTC)
- net DAC_VCA3: now also U7.5 (VOUTB); no longer U7.7 (VOUTD)
- net DAC_VCA4: now also U7.6 (VOUTC); no longer U7.10 (VOUTE)
- net DAC_VCA5: now also U7.7 (VOUTD); no longer U7.11 (VOUTF)
- net SPI_CS0: now also U20.2 (/SYNC)
- net SPI_CS6: no longer U7.2 (/SYNC)
- net SPI_CS7: now also U7.2 (/SYNC); no longer U20.2 (/SYNC)

Commit message: Manual PCB routing by Guimli WIP2
Connections:
- net D+: now reaches J1.3 (D+), R4.2, R5.2
- net D-: now reaches J1.2 (D-), R2.2
- net USB_DM renamed USB_D-
- net USB_DP renamed USB_D+
Changed lines of the file:
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@@
     (effects (font (size 1.524 1.524)) (justify left bottom))
   )
-  (label "USB_DM" (at 140.97 217.17 90) (fields_autoplaced)
+  (label "USB_D-" (at 140.97 217.17 90) (fields_autoplaced)
     (effects (font (size 1.27 1.27)) (justify left bottom))
   )
@@
     (effects (font (size 1.524 1.524)) (justify left bottom))
   )
-  (label "USB_DP" (at 138.43 217.17 90) (fields_autoplaced)
+  (label "USB_D+" (at 138.43 217.17 90) (fields_autoplaced)
     (effects (font (size 1.27 1.27)) (justify left bottom))
   )
@@
     (effects (font (size 1.27 1.27)) (justify left bottom))
   )
-  (label "USB_DP" (at 34.29 53.34 270) (fields_autoplaced)
+  (label "USB_D+" (at 34.29 53.34 270) (fields_autoplaced)
     (effects (font (size 1.27 1.27)) (justify right bottom))
   )
@@
     (effects (font (size 1.27 1.27)) (justify left bottom))
   )
+  (label "D+" (at 26.67 35.56 0) (fields_autoplaced)
+    (effects (font (size 1.27 1.27)) (justify left bottom))
+  )
   (label "RESET" (at 29.21 198.12 0) (fields_autoplaced)
     (effects (font (size 1.27 1.27)) (justify left bottom))
@@
     (effects (font (size 1.27 1.27)) (justify right bottom))
   )
+  (label "D-" (at 26.67 38.1 0) (fields_autoplaced)
+    (effects (font (size 1.27 1.27)) (justify left bottom))
+  )
   (label "KP_8_C4" (at 238.76 149.86 0) (fields_autoplaced)
     (effects (font (size 1.27 1.27)) (justify left bottom))
@@
     (effects (font (size 1.27 1.27)) (justify right bottom))
   )
-  (label "USB_DM" (at 29.21 53.34 270) (fields_autoplaced)
-    (effects (font (size 1.27 1.27)) (justify right bottom))
-  )
+  (label "USB_D-" (at 29.21 53.34 270) (fields_autoplaced)
+    (effects (font (size 1.27 1.27)) (justify right bottom))
+  )

Commit message: Manual PCB routing by Guimli Done!
Parts:
- U3: Manufacturer (none) -> NXP Semicon; Part (none) -> Extended Part; Supplier (none) -> C37701
Changed lines of the file:
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@@
       (effects (font (size 1.27 1.27)) hide)
     )
-    (property "Datasheet" "DOCUMENTATION" (at 215.9 236.22 0)
+    (property "Datasheet" "https://www.nxp.com/docs/en/data-sheet/LPC178X_7X.pdf" (at 215.9 236.22 0)
       (effects (font (size 1.27 1.27)) hide)
     )
+    (property "Part" "Extended Part" (at 215.9 236.22 90)
+      (effects (font (size 1.27 1.27)) hide)
+    )
+    (property "Manufacturer" "NXP Semicon" (at 215.9 236.22 90)
+      (effects (font (size 1.27 1.27)) hide)
+    )
+    (property "Supplier" "C37701" (at 215.9 236.22 90)
+      (effects (font (size 1.27 1.27)) hide)
+    )

Commit message: hardware: Adding LCSC references
Parts:
- C1, C9: LCSC (none) -> C1804
- C10, C11, C12, C14, C15, C16, C17, C18, C19, C20, C23, C24, C25, C26, C27, C29, C30, C32, C34, C35, C37, C38, C39, C40, C41, C42, C43, C44, C45, C46, C47, C49, C8: LCSC (none) -> C28233
- C13: LCSC (none) -> C561869
- C2, C3, C4, C5, C6, C7: LCSC (none) -> C1710
- C21, C22, C31: LCSC (none) -> C7171
- C33, C36, C48: LCSC (none) -> C16133
- C50, C51: LCSC (none) -> C1790
- D1, D2, D3, D4, D5: LCSC (none) -> C81598
- FB1: LCSC (none) -> C1017
- J1: LCSC (none) -> C720549
- J2, J4, J5: LCSC (none) -> C309275
- J3: LCSC (none) -> C2939344
- OC1: LCSC (none) -> C2904409
- P1: LCSC (none) -> C40877
- P2: LCSC (none) -> C3013500
- PS1: LCSC (none) -> C5198614
- PS2: LCSC (none) -> C5198623
- Q1: LCSC (none) -> C2991935
- R1, R11, R25, R37, R40, R6: LCSC (none) -> C17513
- R10: LCSC (none) -> C17593
- R12, R13, R14, R17, R3, R7: LCSC (none) -> C17414
- R15, R24: LCSC (none) -> C149504
- R16, R22, R23, R42: LCSC (none) -> C17673
- R18, R20: LCSC (none) -> C17710
- R19: LCSC (none) -> C34154
- R2, R4: LCSC (none) -> C17634
- R21: LCSC (none) -> C17590
- R26: LCSC (none) -> C17557
- R27, R36: LCSC (none) -> C17633
- R28, R35, R45, R46: LCSC (none) -> C17713
- R29, R34: LCSC (none) -> C17436
- R30, R33: LCSC (none) -> C17756
- R31, R32: LCSC (none) -> C17840
- R38, R39: LCSC (none) -> C17520
- R43, R44: LCSC (none) -> C17475
- R47, R48: LCSC (none) -> C17630
- R5: LCSC (none) -> C4310
- R8: LCSC (none) -> C17709
- R9: LCSC (none) -> C17514
- SW1: LCSC (none) -> C428628
- SW2: LCSC (none) -> C390926
- U1: LCSC (none) -> C2759961
- U2, U6: LCSC (none) -> C6964
- U20, U7: LCSC (none) -> C29162
- U3: LCSC (none) -> C37701
- U4: LCSC (none) -> C527513
- U5: LCSC (none) -> C5602
- Y1: LCSC (none) -> C2975358

Commit message: hardware: improved LCSC references
Parts:
- OC1: LCSC C2904409 -> C4071
- Q1: LCSC C2991935 -> C181154
- U1: LCSC C2759961 -> C5362272
Changed lines of the file:
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@@
       (effects (font (size 1.524 1.524)))
     )
-    (property "LCSC" "C2904409" (at 253.365 259.715 0)
+    (property "LCSC" "C4071" (at 253.365 259.715 0)
       (effects (font (size 1.27 1.27)) hide)
     )
@@
       (effects (font (size 1.27 1.27)) hide)
     )
-    (property "LCSC" "C2759961" (at 115.57 251.46 0)
+    (property "LCSC" "C5362272" (at 115.57 251.46 0)
       (effects (font (size 1.27 1.27)) hide)
     )
@@
       (effects (font (size 1.27 1.27)) hide)
     )
-    (property "LCSC" "C2991935" (at 151.13 58.42 0)
+    (property "LCSC" "C181154" (at 151.13 58.42 0)
       (effects (font (size 1.27 1.27)) hide)
     )
