File: hardware/overcycler3.kicad_sch (KiCad schematic)
At the start: 97 parts, among them J10 Control_Down, J2 AudioJack3_Switch, J3 DIN-5_180degree, J4 AudioJack3_Switch, J5 AudioJack3_Switch, J6 Control_Up, J7 Keyboard, J8 Display, J9 FT232, Q1 2SC945, SW1 RESET, U1 XT26G02CWSIGA, U2 TL064, U3 LPC1778FBD144, U4 TLV2556, U5 74HC138, U6 TL064, Y1 12MHz

Commit message: sch: NAND -> 512Mb NOR FLASH
Parts:
- removed U1: XT26G02CWSIGA, Package_SON:WSON-8-1EP_8x6mm_P1.27mm_EP3.4x4.3mm, symbol Additional:XT26G02ELGIGA
- added U?: W25Q512JVFIQ, Package_SO:SOIC-16W_7.5x10.3mm_P1.27mm, symbol W25Q512JVFIQ:W25Q512JVFIQ
Connections:
- net +3V3: now also U?.1 (/HOLD), U?.2 (VCC), U?.3 (/RESET), U?.9 (/WP)
- net FLASH_SPI_MISO: now also U?.8 (DO)
- net FLASH_SPI_MOSI: now also U?.15 (DI)
- net FLASH_SPI_SCK: now also U?.16 (CLK)
- net FLASH_SPI_SSEL: now also U?.7 (/CS)
- net GND: now also U?.10 (GND)
- no-connect marks 99 -> 106
Other:
- moved on the sheet: C8, R1, R3, SW1

Commit message: hardware: sch/pcb updates by Guimli
Parts:
- removed C? (x3): 100n, Capacitor_SMD:C_0805_2012Metric, symbol Additional:C
- removed R? (x3): 10k, Resistor_SMD:R_0805_2012Metric, symbol Additional:R
- removed U?: AD5674R, MODULE, symbol AD5674R:AD5674R
- removed U?: W25Q512JVFIQ, Package_SO:SOIC-16W_7.5x10.3mm_P1.27mm, symbol W25Q512JVFIQ:W25Q512JVFIQ
- added C112, C113, C114: 100n, Capacitor_SMD:C_0805_2012Metric, symbol Additional:C
- added R151, R41, R42: 10k, Resistor_SMD:R_0805_2012Metric, symbol Additional:R
- added U1: W25Q512JVFIQ, Package_SO:SOIC-16W_7.5x10.3mm_P1.27mm, symbol Additional:W25Q512JVFIQ
- added U7: AD5674R, Additional:LFCSP-28-1EP_4x4mm_P0.4mm_EP2.6x2.6mm_ThermalVias, symbol Additional:AD5674R
Connections:
- net +3V3: now also U1.1 (HOLD(IO3)), U1.2 (VCC), U1.3 (~{RESET}), U1.9 (~{WP}(IO2)), U7.18 (VLOGIC), U7.20 (~{RESET}), U7.6 (GAIN)
- net +5V: now also U7.2 (VDD)
- net DAC_FC0: now also U7.10 (VOUT4)
- net DAC_FC1: now also U7.11 (VOUT15)
- net DAC_FC2: now also U7.12 (VOUT14)
- net DAC_FC3: now also U7.13 (VOUT13)
- net DAC_FC4: now also U7.14 (VOUT12)
- net DAC_FC5: now also U7.22 (VOUT11)
- net DAC_MIXA: now also C114.1, R151.1
- net DAC_MIXB: now also C113.1, R42.1
- net DAC_MIXN: now also C112.1, R41.1
- net DAC_RES: now also U7.9 (VOUT5)
- net DAC_VCA0: now also U7.1 (VOUT0)
- net DAC_VCA1: now also U7.28 (VOUT1)
- net DAC_VCA2: now also U7.27 (VOUT2)
- net DAC_VCA3: now also U7.26 (VOUT3)
- net DAC_VCA4: now also U7.25 (VOUT8)
- net DAC_VCA5: now also U7.24 (VOUT9)
- net FLASH_SPI_MISO: now also U1.8 (DO(IO1))
- net FLASH_SPI_MOSI: now also U1.15 (DI(IO0))
- net FLASH_SPI_SCK: now also U1.16 (CLK)
- net FLASH_SPI_SSEL: now also U1.7 (~{CS})
- net GND: now also J10.2 (Pin_2), J6.2 (Pin_2), U2.5 (+), C112.2, C113.2, C114.2, U1.10 (GND), U7.15 (GND), U7.16 (GND), U7.17 (~{LDAC}), U7.29 (GND); no longer J10.7 (Pin_7), J6.7 (Pin_7), U2.10 (+)
- net P_0: now also J6.3 (Pin_3); no longer J6.2 (Pin_2)
- net P_1: now also J6.4 (Pin_4); no longer J6.3 (Pin_3)
- net P_2: now also J6.5 (Pin_5); no longer J6.4 (Pin_4)
- net P_3: now also J6.6 (Pin_6); no longer J6.5 (Pin_5)
- net P_4: now also J6.7 (Pin_7); no longer J6.6 (Pin_6)
- net P_5: now also J10.3 (Pin_3); no longer J10.2 (Pin_2)
- net P_6: now also J10.4 (Pin_4); no longer J10.3 (Pin_3)
- net P_7: now also J10.5 (Pin_5); no longer J10.4 (Pin_4)
- net P_8: now also J10.6 (Pin_6); no longer J10.5 (Pin_5)
- net P_9: now also J10.7 (Pin_7); no longer J10.6 (Pin_6)
- net SPI_CS0: now also U7.3 (~{SYNC})
- net SPI_MOSI: now also U7.5 (SDI)
- net SPI_SCK: now also U7.4 (SCLK)
- net at R10.1, R12.2: now also U2.10 (+); no longer U2.5 (+)
- net at R13.1, R18.2: now also U2.8, U2.9 (-); no longer U2.6 (-), U2.7
- net at R15.2, R19.2: now also U2.14; no longer U2.1
- net at R11.2, R15.1: now also U2.13 (-); no longer U2.2 (-)
- net at C35.2, R9.2: now also U2.12 (+); no longer U2.3 (+)
- net at R17.1, R20.2: now also U2.7; no longer U2.8
- net at R13.2, R17.2: now also U2.6 (-); no longer U2.9 (-)
- net at D2.2 (K), D3.1 (A), R19.1: now also U2.3 (+); no longer U2.12 (+)
- net at R23.2, R24.1: now also U2.2 (-); no longer U2.13 (-)
- net at C48.1, R24.2: now also U2.1; no longer U2.14
- new net: R41.2, U7.23 (VOUT10)
- new net: R42.2, U7.7 (VOUT7)
- new net: R151.2, U7.8 (VOUT6)
- no-connect marks 106 -> 99
Other:
- moved on the sheet: C8, R1, R3, SW1

Commit message: hardware: sch/pcb updates by Guimli
Parts:
- J10, J6: footprint Connector_JST:JST_XH_B7B-XH-A_1x07_P2.50mm_Vertical -> Connector_JST:JST_PH_B7B-PH-K_1x07_P2.00mm_Vertical
Connections:
- net ADC_SPI_MISO: now also U3.53 (P1[23]); no longer U3.133 (P1[4])
- net ADC_SPI_MOSI: now also U3.54 (P1[24]); no longer U3.135 (P1[1])
- net ADC_SPI_SCK: now also U3.49 (P1[20]); no longer U3.136 (P1[0])
- net ADC_SPI_SSEL: now also U3.50 (P1[21]); no longer U3.132 (P1[8])
- net SPI_MOSI: now also U3.135 (P1[1]); no longer U3.54 (P1[24])
- net SPI_SCK: now also U3.136 (P1[0]); no longer U3.49 (P1[20])
- net SPI_SSEL: now also U3.132 (P1[8]); no longer U3.50 (P1[21])
- no-connect marks 99 -> 100
Other:
- moved on the sheet: U1

Commit message: hardware: sch/pcb updates by Guimli
Parts:
- J2, J4, J5: footprint Connector_Audio:Jack_6.35mm_Neutrik_NMJ6HFD2_Horizontal -> Additional:Jack_6.35mm_OFFHOOYA_PJ-609AE_Horizontal
Connections:
- net +3V3: now also J10.2 (Pin_2), J6.2 (Pin_2), U5.6 (E2); no longer J10.1 (Pin_1), J6.1 (Pin_1), U1.1 (~{HOLD}(IO3)), U1.9 (~{WP}(IO2)), U5.4 (~{E0})
- net GND: now also J10.1 (Pin_1), J6.1 (Pin_1); no longer J10.2 (Pin_2), J6.2 (Pin_2)
- net KP_1_R1: now also U3.90 (P0[16]); no longer U3.80 (P0[22])
- net KP_2_R2: now also U3.87 (P0[17]); no longer U3.82 (P0[21])
- net KP_3_R3: now also U3.86 (P0[18]); no longer U3.83 (P0[20])
- net KP_5_C1: now also U3.83 (P0[20]); no longer U3.69 (P0[10])
- net KP_6_C2: now also U3.82 (P0[21]); no longer U3.122 (P4[29])
- net KP_7_C3: now also U3.80 (P0[22]); no longer U3.118 (P4[28])
- net KP_8_C4: now also U3.13 (P0[23]); no longer U3.71 (P2[13])
- net LCD_DB4: now also U3.100 (P2[3]); no longer U3.106 (P2[1])
- net LCD_DB5: now also U3.105 (P2[2]); no longer U3.107 (P2[0])
- net LCD_DB6: now also U3.106 (P2[1]); no longer U3.105 (P2[2])
- net LCD_DB7: now also U3.107 (P2[0]); no longer U3.100 (P2[3])
- net LCD_E1: now also U3.99 (P2[4]); no longer U3.96 (P2[6])
- net LCD_RS: now also U3.96 (P2[6]); no longer U3.99 (P2[4])
- net SPI_MUX_A: now also U3.128 (P1[14]); no longer U3.89 (P0[15])
- net SPI_MUX_B: now also U3.126 (P1[15]); no longer U3.90 (P0[16])
- net SPI_MUX_C: now also U3.125 (P1[16]); no longer U3.115 (P0[5])
- net SPI_SSEL: now also U5.4 (~{E0}); no longer U5.6 (E2)
- net at R10.1, R12.2: now also U2.3 (+); no longer U2.10 (+)
- net at R13.1, R18.2: now also U2.1, U2.2 (-); no longer U2.8, U2.9 (-)
- net at C48.1, R24.2: now also U2.8; no longer U2.1
- net at R23.2, R24.1: now also U2.9 (-); no longer U2.2 (-)
- net at D2.2 (K), D3.1 (A), R19.1: now also U2.10 (+); no longer U2.3 (+)
- net FLASH_~{WP}: now reaches U3.116 (P0[4])
- net FLASH_~{WP}: now also U1.9 (~{WP}(IO2))
- new net FLASH_~{HOLD}: U1.1 (~{HOLD}(IO3)), U3.115 (P0[5])
- no-connect marks 100 -> 97
Other:
- moved on the sheet: C50, C51, J4, J7, J8, J9, R37, R40, R47, R6, U1

Commit message: hardware: sch/pcb updates by Guimli
Parts:
- J1: renamed from J3; footprint DIN-5-180:DIN-5-180 -> Additional:HOOYA DIN-504-M10
- J2: footprint Additional:Jack_6.35mm_OFFHOOYA_PJ-609AE_Horizontal -> Additional:Jack_6.35mm_HOOYA_PJ-609AE_Horizontal
- J3: renamed from J4; footprint Additional:Jack_6.35mm_OFFHOOYA_PJ-609AE_Horizontal -> Additional:Jack_6.35mm_HOOYA_PJ-609AE_Horizontal
- J4: renamed from J5; footprint Additional:Jack_6.35mm_OFFHOOYA_PJ-609AE_Horizontal -> Additional:Jack_6.35mm_HOOYA_PJ-609AE_Horizontal
- Q1: symbol PCM_Transistor_BJT_AKL:2SC945 -> Additional:2SC945
- renumbered C51 to C1, C43 to C107, C44 to C110, C45 to C113, C46 to C115, C47 to C116, C112 to C117, C49 to C118, C33 to C119, C48 to C120, C36 to C121, C35 to C122, C42 to C124, C41 to C125, C40 to C127, C39 to C128, C38 to C129, C37 to C27, C9 to C31, C1 to C32, C50 to C5, C8 to C64, C113 to C92, C114 to C93, D5 to D1, D1 to D2, D4 to D3, D2 to D4, D3 to D5, J9 to J6, J6 to J7, J7 to J9, R47 to R10, R43 to R11, R42 to R111, R6 to R112, R45 to R12, R30 to R13, R41 to R137, R8 to R138, R7 to R139, R32 to R14, R25 to R140, R9 to R141, R23 to R142, R11 to R143, R24 to R144, R15 to R145, R10 to R146, R19 to R147, R12 to R148, R18 to R149, R28 to R15, R13 to R150, R17 to R151, R20 to R152, R34 to R16, R27 to R17, R31 to R18, R33 to R19, R29 to R20, R35 to R21, R36 to R22, R44 to R3, R46 to R4, R26 to R41, R40 to R5, R39 to R6, R14 to R60, R16 to R61, R22 to R62, R21 to R63, R1 to R64, R48 to R7, R37 to R8, R3 to R89, R38 to R9, R151 to R98, SW1 to SW2, U6 to U1, U1 to U16, U5 to U17, U4 to U18, U2 to U19, U7 to U2, U3 to U9
Connections:
- no-connect marks 97 -> 98

Commit message: hardware: LCSC review, production files ok
Parts:
- J10, J7: LCSC (none) -> C157981
- J6: LCSC C40877 -> C40877
- J9: LCSC C7465591 -> C157972
- U16: LCSC C2962011 -> C2962011
Changed lines of the file:
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@@
 			)
 		)
+		(property "LCSC" "C157981"
+			(at 90.17 242.5699 0)
+			(effects
+				(font
+					(size 1.27 1.27)
+				)
+				(hide yes)
+			)
+		)
 		(pin "4"
 		)
@@
 			)
 		)
-		(property "LCSC" "C7465591"
+		(property "LCSC" "C157972"
 			(at 124.46 256.54 0)
 			(effects
@@
 			)
 		)
+		(property "LCSC" "C157981"
+			(at 90.17 220.9799 0)
+			(effects
+				(font
+					(size 1.27 1.27)
+				)
+				(hide yes)
+			)
+		)
 		(pin "4"
 		)
@@
 			)
 		)
-		(property "LCSC" "     C40877"
+		(property "LCSC" "C40877"
 			(at 152.4 218.44 0)
 			(effects
@@
 			)
 		)
-		(property "LCSC" "  C2962011"
+		(property "LCSC" "C2962011"
 			(at 231.14 261.62 0)
 			(effects

Commit message: hardware: sch/pcb changes by Guimli (adding USB isolator, misc fixes)
Parts:
- C118: footprint Capacitor_Tantalum_SMD:CP_EIA-3216-18_Kemet-A -> Additional:CP_EIA-3216-18_Kemet-A
- C119, C120, C121: footprint Capacitor_Tantalum_SMD:CP_EIA-3528-21_Kemet-B -> Additional:CP_EIA-3528-21_Kemet-B
- D1, D2, D3, D4, D5: footprint Diode_SMD:D_SOD-123 -> Additional:D_SOD-123
- J10, J7: LCSC C157981 -> (none)
- J6: LCSC C40877 -> C40877
- J8: footprint Connector_IDC:IDC-Header_2x08_P2.54mm_Vertical -> Additional:IDC-Header_2x08_P2.54mm_Vertical_Mirrored
- J9: LCSC C157972 -> C7465591
- U16: LCSC C2962011 -> C2962011
Connections:
- net LCD_DB4: now also U9.105 (P2[2]); no longer U9.100 (P2[3])
- net LCD_DB5: now also U9.100 (P2[3]); no longer U9.105 (P2[2])
- net LCD_DB6: now also U9.107 (P2[0]); no longer U9.106 (P2[1])
- net LCD_DB7: now also U9.106 (P2[1]); no longer U9.107 (P2[0])
- net LCD_E1: now also U9.97 (P2[5]); no longer U9.99 (P2[4])
- net LCD_RW: now also U9.99 (P2[4]); no longer U9.97 (P2[5])
- net KP_1_R1 renamed KP_1_C1
- net KP_2_R2 renamed KP_2_C2
- net KP_3_R3 renamed KP_3_C3
- net KP_4_R4 renamed KP_4_C4
- net KP_5_C1 renamed KP_5_R1
- net KP_6_C2 renamed KP_6_R2
- net KP_7_C3 renamed KP_7_R3
- net KP_8_C4 renamed KP_8_R4
Other:
- moved on the sheet: R112
