File: hardware/Power_Supply.kicad_sch (KiCad schematic)
At the start: 47 parts, among them IC1 LM13700, IC2 LM13700, IC3 LM13700, J1 USB_B, SW2 POWER, U2 TL064, U6 TL064

Commit message: hardware: sch/pcb updates by Guimli
Parts:
- added C115, C116, C117: 10n, Capacitor_SMD:C_0805_2012Metric, symbol Additional:C
Connections:
- net -5V: now also C115.2, C116.2, C117.2
- net GND: now also C115.1, C116.1, C117.1

Commit message: hardware: sch/pcb updates by Guimli
Parts:
- added C118, C119, C120, C121, C122, C123, C124, C125: 100nF, Capacitor_SMD:C_0805_2012Metric, symbol Additional:C
- C10, C11, C12, C14, C15, C16, C17, C18, C19, C22, C23, C24, C25, C26, C27, C28, C30, C31, C32, C34: value 100n -> 100nF
- C115, C116, C117: value 10n -> 100nF; LCSC C1710 -> C28233
- C13: value 470u -> 470uF
- C2, C3, C4, C5, C6, C7: value 10n -> 10nF
- C20, C21, C29: value 10u -> 10uF
Connections:
- net +5V: now also C121.1, C122.1, C123.1, C124.1, C125.1
- net -5V: now also C118.2, C119.2, C120.2
- net GND: now also C118.1, C119.1, C120.1, C121.2, C122.2, C123.2, C124.2, C125.2
Other:
- moved on the sheet: C10, C11, C115, C116, C117, C12, C13, C14, C15, C16, C17, C18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

Commit message: hardware: sch/pcb updates by Guimli
Parts:
- added C126, C127, C128, C129: 100nF, Capacitor_SMD:C_0805_2012Metric, symbol Additional:C
Connections:
- net +5V: now also C128.1, C129.1
- net -5V: now also C126.2, C127.2
- net GND: now also C126.1, C127.1, C128.2, C129.2
Other:
- moved on the sheet: C10, C11, C115, C116, C117, C118, C119, C12, C120, C121, C122, C123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

Commit message: hardware: sch/pcb updates by Guimli
Parts:
- IC2, IC3: LCSC (none) -> C5160094
- PS1: symbol Converter_DCDC:IA0505S -> Additional:IA0505S-2W
- PS2: symbol Converter_DCDC:IA0503S -> Additional:IB0503LSY-1WR1
- U1: renamed from U6; LCSC (none) -> C6959
- U19: renamed from U2; LCSC (none) -> C6959
- renumbered C10 to C101, C12 to C102, C11 to C103, C15 to C104, C16 to C105, C125 to C106, C31 to C108, C28 to C109, C24 to C111, C30 to C112, C32 to C114, C127 to C123, C129 to C126, C20 to C13, C2 to C14, C3 to C15, C4 to C16, C5 to C17, C6 to C18, C7 to C19, C126 to C2, C29 to C26, C22 to C28, C18 to C29, C128 to C3, C34 to C30, C118 to C34, C119 to C36, C120 to C38, C13 to C4, C115 to C40, C116 to C42, C117 to C44, C25 to C45, C21 to C6, C26 to C77, C122 to C78, C14 to C79, C121 to C80, C123 to C81, C17 to C82, C124 to C83, C19 to C84, C27 to C85, C23 to C86, J1 to J5, R152 to R1, R5 to R2, R2 to R90, R4 to R91, SW2 to SW1

Commit message: hardware: LCSC review, production files ok
Parts:
- PS1: LCSC C5198614 -> C512062
Changed lines of the file:
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@@
 			)
 		)
-		(property "LCSC" "C5198614"
+		(property "LCSC" "C512062"
 			(at 82.55 76.2 0)
 			(effects

Commit message: hardware: sch/pcb changes by Guimli (adding USB isolator, misc fixes)
Parts:
- added C130, C131, C132: 100nF, Capacitor_SMD:C_0805_2012Metric, symbol Additional:C
- added U20: ADUM3160, Package_SO:SOIC-16W_7.5x10.3mm_P1.27mm, symbol Interface_USB:ADUM3160
- C13, C26, C6: footprint Capacitor_Tantalum_SMD:CP_EIA-3216-18_Kemet-A -> Additional:CP_EIA-3216-18_Kemet-A
- C4: footprint Capacitor_Tantalum_SMD:CP_EIA-7343-43_Kemet-X -> Additional:CP_EIA-7343-43_Kemet-X
- PS1: LCSC C512062 -> C5198614
Connections:
- net +3V3: now also C131.1, U20.12 (PIN), U20.13 (SPD), U20.14 (VDD2), U20.16 (VBUS2)
- net D+: now also U20.10 (DD+); no longer J5.3 (D+), R1.2, R2.1
- net D-: now also U20.11 (DD-); no longer J5.2 (D-)
- net GND: now also C131.2, U20.15 (GND2), U20.9 (GND2); no longer H1.1
- net USB_5V: now also C132.1, U20.1 (VBUS1)
- net USB_GND: now also J5.5 (Shield), C130.2, C132.2, U20.2 (GND1), U20.8 (GND1)
- net USB_VBUS: no longer names the net of J5.1 (VBUS), SW1.2 (B), SW1.5 (B)
- new net: C130.1, U20.3 (VDD1), U20.4 (PDEN), U20.5 (SPU)
- new net UD+: J5.3 (D+), R1.2, R2.1, U20.7 (UD+)
- new net UD-: J5.2 (D-), U20.6 (UD-)
Other:
- moved on the sheet: C101, C102, C103, C104, C105, C106, C108, C109, C111, C112, C114, C123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

Commit message: hwarware: IA0505S-2W, JETEKPS -> RLT
Parts:
- PS1: LCSC C5198614 -> C512062; Manufacturer JETEKPS -> RLT
Changed lines of the file:
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@@
 			)
 		)
-		(property "Datasheet" "https://www.lcsc.com/datasheet/lcsc_datasheet_2210141730_JETEKPS-IA0505S-2W_C5198614.pdf"
+		(property "Datasheet" "https://wmsc.lcsc.com/wmsc/upload/file/pdf/v2/lcsc/2004151709_rlt-IA0505S-2W_C512062.pdf"
 			(at 173.99 58.42 0)
 			(effects
@@
 			)
 		)
-		(property "Manufacturer" "JETEKPS"
+		(property "Manufacturer" "RLT"
 			(at 184.15 60.96 0)
 			(effects
@@
 			)
 		)
-		(property "LCSC" "C5198614"
+		(property "LCSC" "C512062"
 			(at 184.15 63.5 0)
 			(effects
