File: hardware/Power_Supply.kicad_sch (KiCad schematic)
At the start: 66 parts, among them IC1 LM13700, IC2 LM13700, IC3 LM13700, J5 USB_B, SW1 POWER, U1 TL064, U19 TL064, U20 ADUM3160

Commit message: hardware: don't add pullup on D+, ADUM3160 handles it
Parts:
- removed R1: 2k7, Resistor_SMD:R_0805_2012Metric, symbol Additional:R
- removed R2: 1k5, Resistor_SMD:R_0805_2012Metric, symbol Additional:R
Changed lines of the file:
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@@
 	)
 	(junction
-		(at 154.94 119.38)
+		(at 93.98 43.18)
 		(diameter 0)
 		(color 0 0 0 0)
 	)
 	(junction
-		(at 100.33 125.73)
+		(at 154.94 119.38)
 		(diameter 0)
 		(color 0 0 0 0)
 	)
 	(junction
-		(at 173.99 132.08)
+		(at 100.33 125.73)
 		(diameter 0)
 		(color 0 0 0 0)
 	)
 	(junction
-		(at 74.93 113.03)
+		(at 173.99 132.08)
 		(diameter 0)
 		(color 0 0 0 0)
 	)
 	(junction
-		(at 86.36 33.02)
+		(at 74.93 113.03)
 		(diameter 0)
 		(color 0 0 0 0)
@@
 	)
 	(junction
-		(at 86.36 55.88)
-		(diameter 0)
-		(color 0 0 0 0)
-	)
-	(junction
 		(at 66.04 50.8)
 		(diameter 0)
@@
 	)
 	(junction
-		(at 86.36 86.36)
-		(diameter 0)
-		(color 0 0 0 0)
-	)
-	(junction
 		(at 180.34 132.08)
 		(diameter 0)
@@
 	)
 	(junction
-		(at 93.98 33.02)
-		(diameter 0)
-		(color 0 0 0 0)
-	)
-	(junction
 		(at 166.37 33.02)
 		(diameter 0)
@@
 	(wire
 		(pts
-			(xy 86.36 50.8) (xy 86.36 55.88)
-		)
-		(stroke
-			(width 0)
-			(type default)
-		)
-	)
-	(wire
-		(pts
 			(xy 49.53 113.03) (xy 55.88 113.03)
 		)
@@
 	(wire
 		(pts
-			(xy 86.36 76.2) (xy 86.36 86.36)
-		)
-		(stroke
-			(width 0)
-			(type default)
-		)
-	)
-	(wire
-		(pts
 			(xy 237.49 119.38) (xy 243.84 119.38)
 		)
@@
 	(wire
 		(pts
-			(xy 86.36 33.02) (xy 93.98 33.02)
-		)
-		(stroke
-			(width 0)
-			(type default)
-		)
-	)
-	(wire
-		(pts
 			(xy 148.59 106.68) (xy 154.94 106.68)
 		)
@@
 	(wire
 		(pts
-			(xy 86.36 86.36) (xy 93.98 86.36)
-		)
-		(stroke
-			(width 0)
-			(type default)
-		)
-	)
-	(wire
-		(pts
 			(xy 193.04 106.68) (xy 193.04 107.95)
 		)
@@
 	(wire
 		(pts
-			(xy 63.5 55.88) (xy 86.36 55.88)
+			(xy 63.5 55.88) (xy 104.14 55.88)
 		)
 		(stroke
@@
 	(wire
 		(pts
-			(xy 93.98 33.02) (xy 93.98 64.77)
+			(xy 93.98 33.02) (xy 93.98 43.18)
 		)
 		(stroke
@@
 	(wire
 		(pts
-			(xy 55.88 86.36) (xy 86.36 86.36)
+			(xy 55.88 86.36) (xy 93.98 86.36)
 		)
 		(stroke
@@
 	(wire
 		(pts
-			(xy 86.36 33.02) (xy 86.36 38.1)
-		)
-		(stroke
-			(width 0)
-			(type default)
-		)
-	)
-	(wire
-		(pts
 			(xy 154.94 106.68) (xy 161.29 106.68)
 		)
@@
 	(wire
 		(pts
-			(xy 86.36 55.88) (xy 86.36 63.5)
-		)
-		(stroke
-			(width 0)
-			(type default)
-		)
-	)
-	(wire
-		(pts
 			(xy 193.04 119.38) (xy 199.39 119.38)
 		)
@@
 	(wire
 		(pts
-			(xy 43.18 124.46) (xy 43.18 125.73)
+			(xy 93.98 43.18) (xy 93.98 64.77)
 		)
 		(stroke
@@
 	(wire
 		(pts
-			(xy 93.98 74.93) (xy 93.98 86.36)
+			(xy 43.18 124.46) (xy 43.18 125.73)
 		)
 		(stroke
@@
 	(wire
 		(pts
-			(xy 113.03 113.03) (xy 113.03 114.3)
+			(xy 93.98 74.93) (xy 93.98 86.36)
 		)
 		(stroke
@@
 	(wire
 		(pts
-			(xy 180.34 119.38) (xy 180.34 120.65)
+			(xy 113.03 113.03) (xy 113.03 114.3)
 		)
 		(stroke
@@
 	(wire
 		(pts
-			(xy 212.09 130.81) (xy 212.09 132.08)
+			(xy 180.34 119.38) (xy 180.34 120.65)
 		)
 		(stroke
@@
 	(wire
 		(pts
-			(xy 186.69 130.81) (xy 186.69 132.08)
+			(xy 212.09 130.81) (xy 212.09 132.08)
 		)
 		(stroke
@@
 	(wire
 		(pts
-			(xy 86.36 55.88) (xy 104.14 55.88)
+			(xy 186.69 130.81) (xy 186.69 132.08)
 		)
 		(stroke
@@
 	(wire
 		(pts
-			(xy 81.28 33.02) (xy 86.36 33.02)
-		)
-		(stroke
-			(width 0)
-			(type default)
-		)
-	)
-	(wire
-		(pts
 			(xy 180.34 132.08) (xy 186.69 132.08)
 		)
@@
 	(wire
 		(pts
-			(xy 81.28 43.18) (xy 81.28 33.02)
-		)
-		(stroke
-			(width 0)
-			(type default)
-		)
-	)
-	(wire
-		(pts
 			(xy 106.68 113.03) (xy 113.03 113.03)
 		)
@@
 	(wire
 		(pts
+			(xy 81.28 43.18) (xy 93.98 43.18)
+		)
+		(stroke
+			(width 0)
+			(type default)
+		)
+	)
+	(wire
+		(pts
 			(xy 148.59 118.11) (xy 148.59 119.38)
 		)
@@
 	)
 	(symbol
-		(lib_id "Additional:R")
-		(at 86.36 69.85 180)
-		(unit 1)
-		(exclude_from_sim no)
-		(in_bom yes)
-		(on_board yes)
-		(dnp no)
-		(property "Reference" "R1"
-			(at 88.9 69.85 0)
-			(effects
-				(font
-					(size 1.016 1.016)
-				)
-			)
-		)
-		(property "Value" "2k7"
-			(at 86.36 69.85 90)
-			(effects
-				(font
-					(size 1.016 1.016)
-				)
-			)
-		)
-		(property "Footprint" "Resistor_SMD:R_0805_2012Metric"
-			(at 88.138 69.85 90)
-			(effects
-				(font
-					(size 0.762 0.762)
-				)
-				(hide yes)
-			)
-		)
-		(property "Datasheet" "~"
-			(at 86.36 69.85 0)
-			(effects
-				(font
-					(size 0.762 0.762)
-				)
-			)
-		)
-		(property "Description" ""
-			(at 86.36 69.85 0)
-			(effects
-				(font
-					(size 1.27 1.27)
-				)
-				(hide yes)
-			)
-		)
-		(property "LCSC" "C114520"
-			(at 84.328 69.85 0)
-			(effects
-				(font
-					(size 1.27 1.27)
-				)
-				(hide yes)
-			)
-		)
-		(pin "1"
-		)
-		(pin "2"
-		)
-		(instances
-			(project "overcycler3"
-				(path "/f3616c1d-a98e-4f9d-ac17-0c5545b71bc4/347aba77-50ac-4a87-997c-5d48101c82e0"
-					(reference "R1")
-					(unit 1)
-				)
-			)
-		)
-	)
-	(symbol
 		(lib_id "Additional:C")
 		(at 199.39 113.03 0)
@@
 					(unit 1)
 				)
-			)
-		)
-	)
-	(symbol
-		(lib_id "Additional:R")
-		(at 86.36 44.45 180)
-		(unit 1)
-		(exclude_from_sim no)
-		(in_bom yes)
-		(on_board yes)
-		(dnp no)
-		(property "Reference" "R2"
-			(at 88.9 44.45 0)
-			(effects
-				(font
-					(size 1.016 1.016)
-				)
-			)
-		)
-		(property "Value" "1k5"
-			(at 86.36 44.45 90)
-			(effects
-				(font
-					(size 1.016 1.016)
-				)
-			)
-		)
-		(property "Footprint" "Resistor_SMD:R_0805_2012Metric"
-			(at 88.138 44.45 90)
-			(effects
-				(font
-					(size 0.762 0.762)
-				)
-				(hide yes)
-			)
-		)
-		(property "Datasheet" "~"
-			(at 86.36 44.45 0)
-			(effects
-				(font
-					(size 0.762 0.762)
-				)
-			)
-		)
-		(property "Description" ""
-			(at 86.36 44.45 0)
-			(effects
-				(font
-					(size 1.27 1.27)
-				)
-				(hide yes)
-			)
-		)
-		(property "LCSC" "C4310"
-			(at 84.328 44.45 0)
-			(effects
-				(font
-					(size 1.27 1.27)
-				)
-				(hide yes)
-			)
-		)
-		(pin "1"
-		)
-		(pin "2"
-		)
-		(instances
-			(project "overcycler3"
-				(path "/f3616c1d-a98e-4f9d-ac17-0c5545b71bc4/347aba77-50ac-4a87-997c-5d48101c82e0"
-					(reference "R2")
-					(unit 1)
-				)

Commit message: Add ADuM3160 and correct enclosure rear
- ADuM3160 added for USB isolation
- Correction of USB traces to respect 90Ω in two-layer PCBs
- Integration of Noise circuit modifications
Parts:
- added R1, R2: 24, Resistor_SMD:R_0603_1608Metric, symbol Additional:R
- R90, R91: footprint Resistor_SMD:R_0805_2012Metric -> Resistor_SMD:R_0603_1608Metric; LCSC C17634 -> C23140
Connections:
- net D+: now also J5.3 (D+), R1.2; no longer R91.2, U20.10 (DD+)
- net D-: now also J5.2 (D-), R2.2; no longer R90.2, U20.11 (DD-)
- net UD+: now also R1.1; no longer J5.3 (D+)
- net UD-: now also R2.1; no longer J5.2 (D-)
- new net DD+: R91.2, U20.10 (DD+)
- new net DD-: R90.2, U20.11 (DD-)
Changed lines of the file:
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@@
 	(wire
 		(pts
-			(xy 63.5 55.88) (xy 104.14 55.88)
+			(xy 63.5 55.88) (xy 80.01 55.88)
 		)
 		(stroke
@@
 	(wire
 		(pts
+			(xy 92.71 58.42) (xy 104.14 58.42)
+		)
+		(stroke
+			(width 0)
+			(type default)
+		)
+	)
+	(wire
+		(pts
 			(xy 148.59 119.38) (xy 148.59 120.65)
 		)
@@
 	(wire
 		(pts
+			(xy 92.71 55.88) (xy 104.14 55.88)
+		)
+		(stroke
+			(width 0)
+			(type default)
+		)
+	)
+	(wire
+		(pts
 			(xy 148.59 132.08) (xy 148.59 133.35)
 		)
@@
 	(wire
 		(pts
-			(xy 63.5 58.42) (xy 104.14 58.42)
+			(xy 63.5 58.42) (xy 80.01 58.42)
 		)
 		(stroke
@@
 		)
 	)
+	(label "UD-"
+		(at 95.25 58.42 0)
+		(fields_autoplaced yes)
+		(effects
+			(font
+				(size 1.27 1.27)
+			)
+			(justify left bottom)
+		)
+	)
 	(label "USB_5V"
 		(at 166.37 33.02 0)
@@
 		)
 	)
-	(label "UD+"
-		(at 64.77 55.88 0)
+	(label "D+"
+		(at 66.04 55.88 0)
 		(fields_autoplaced yes)
 		(effects
@@
 		)
 	)
-	(label "D-"
+	(label "DD-"
 		(at 135.89 58.42 0)
 		(fields_autoplaced yes)
@@
 		)
 	)
-	(label "UD-"
-		(at 64.77 58.42 0)
+	(label "D-"
+		(at 66.04 58.42 0)
 		(fields_autoplaced yes)
 		(effects
@@
 		)
 	)
-	(label "D+"
+	(label "DD+"
 		(at 135.89 55.88 0)
 		(fields_autoplaced yes)
@@
 		)
 	)
+	(label "UD+"
+		(at 95.25 55.88 0)
+		(fields_autoplaced yes)
+		(effects
+			(font
+				(size 1.27 1.27)
+			)
+			(justify left bottom)
+		)
+	)
 	(global_label "USB_D+"
 		(shape output)
@@
 	)
 	(symbol
+		(lib_id "Additional:R")
+		(at 86.36 55.88 270)
+		(unit 1)
+		(exclude_from_sim no)
+		(in_bom yes)
+		(on_board yes)
+		(dnp no)
+		(property "Reference" "R1"
+			(at 86.36 53.848 90)
+			(effects
+				(font
+					(size 1.016 1.016)
+				)
+			)
+		)
+		(property "Value" "24"
+			(at 86.36 55.88 90)
+			(effects
+				(font
+					(size 1.016 1.016)
+				)
+			)
+		)
+		(property "Footprint" "Resistor_SMD:R_0603_1608Metric"
+			(at 86.36 54.102 90)
+			(effects
+				(font
+					(size 0.762 0.762)
+				)
+				(hide yes)
+			)
+		)
+		(property "Datasheet" "~"
+			(at 86.36 55.88 0)
+			(effects
+				(font
+					(size 0.762 0.762)
+				)
+			)
+		)
+		(property "Description" ""
+			(at 86.36 55.88 0)
+			(effects
+				(font
+					(size 1.27 1.27)
+				)
+				(hide yes)
+			)
+		)
+		(property "LCSC" " C25804"
+			(at 86.36 57.912 0)
+			(effects
+				(font
+					(size 1.27 1.27)
+				)
+				(hide yes)
+			)
+		)
+		(pin "1"
+		)
+		(pin "2"
+		)
+		(instances
+			(project "overcycler3"
+				(path "/f3616c1d-a98e-4f9d-ac17-0c5545b71bc4/347aba77-50ac-4a87-997c-5d48101c82e0"
+					(reference "R1")
+					(unit 1)
+				)
+			)
+		)
+	)
+	(symbol
 		(lib_id "Additional:CP")
 		(at 236.22 55.88 0)
@@
 	)
 	(symbol
+		(lib_id "Additional:R")
+		(at 86.36 58.42 270)
+		(unit 1)
+		(exclude_from_sim no)
+		(in_bom yes)
+		(on_board yes)
+		(dnp no)
+		(property "Reference" "R2"
+			(at 86.36 60.452 90)
+			(effects
+				(font
+					(size 1.016 1.016)
+				)
+			)
+		)
+		(property "Value" "24"
+			(at 86.36 58.42 90)
+			(effects
+				(font
+					(size 1.016 1.016)
+				)
+			)
+		)
+		(property "Footprint" "Resistor_SMD:R_0603_1608Metric"
+			(at 86.36 56.642 90)
+			(effects
+				(font
+					(size 0.762 0.762)
+				)
+				(hide yes)
+			)
+		)
+		(property "Datasheet" "~"
+			(at 86.36 58.42 0)
+			(effects
+				(font
+					(size 0.762 0.762)
+				)
+			)
+		)
+		(property "Description" ""
+			(at 86.36 58.42 0)
+			(effects
+				(font
+					(size 1.27 1.27)
+				)
+				(hide yes)
+			)
+		)
+		(property "LCSC" " C25804"
+			(at 86.36 60.452 0)
+			(effects
+				(font
+					(size 1.27 1.27)
+				)
+				(hide yes)
+			)
+		)
+		(pin "1"
+		)
+		(pin "2"
+		)
+		(instances
+			(project "overcycler3"
+				(path "/f3616c1d-a98e-4f9d-ac17-0c5545b71bc4/347aba77-50ac-4a87-997c-5d48101c82e0"
+					(reference "R2")
+					(unit 1)
+				)
+			)
+		)
+	)
+	(symbol
 		(lib_id "power:GND")
 		(at 151.13 166.37 0)
@@
 			)
 		)
-		(property "Footprint" "Resistor_SMD:R_0805_2012Metric"
+		(property "Footprint" "Resistor_SMD:R_0603_1608Metric"
 			(at 144.78 56.642 90)
 			(effects
@@
 			)
 		)
-		(property "LCSC" "C17634"
+		(property "LCSC" "C23140"
 			(at 144.78 60.452 0)
 			(effects
@@
 			)
 		)
-		(property "Footprint" "Resistor_SMD:R_0805_2012Metric"
+		(property "Footprint" "Resistor_SMD:R_0603_1608Metric"
 			(at 144.78 54.102 90)
 			(effects
@@
 			)
 		)
-		(property "LCSC" "C17634"
+		(property "LCSC" "C23140"
 			(at 144.78 57.912 0)
 			(effects

Commit message: Replace "Main Output" by "Output"
- Replace "Main Output" by "Output" on Panel Rear
- Manually add Teardown
- Replace 24Ω by 33Ω on USB Isolator
Parts:
- R1, R2: value 24 -> 33; LCSC C25804 -> C23140
Changed lines of the file:
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@@
 			)
 		)
-		(property "Value" "24"
+		(property "Value" "33"
 			(at 86.36 55.88 90)
 			(effects
@@
 			)
 		)
-		(property "LCSC" " C25804"
+		(property "LCSC" "C23140"
 			(at 86.36 57.912 0)
 			(effects
@@
 			)
 		)
-		(property "Value" "24"
+		(property "Value" "33"
 			(at 86.36 58.42 90)
 			(effects
@@
 			)
 		)
-		(property "LCSC" " C25804"
+		(property "LCSC" "C23140"
 			(at 86.36 60.452 0)
 			(effects

Commit message: hardware: add missing D+ pullup resistor (MCU side)
Parts:
- added R144: 1k5, Resistor_SMD:R_0603_1608Metric, symbol Additional:R
Connections:
- net +3V3: now also R144.1
- net USB_D+: now also R144.2
Other:
- moved on the sheet: C13, C26, C4, C6, PS1, PS2

Commit message: Add USB pullup resistor
- Add USB pullup resistor
Connections:
- net DD+: now also R144.2
- net USB_D+: no longer R144.2
Other:
- moved on the sheet: R144, R90, R91
Changed lines of the file:
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@@
 	)
 	(junction
+		(at 137.16 55.88)
+		(diameter 0)
+		(color 0 0 0 0)
+	)
+	(junction
 		(at 106.68 125.73)
 		(diameter 0)
@@
 	)
 	(junction
-		(at 152.4 55.88)
-		(diameter 0)
-		(color 0 0 0 0)
-	)
-	(junction
 		(at 180.34 119.38)
 		(diameter 0)
@@
 	(wire
 		(pts
+			(xy 137.16 55.88) (xy 143.51 55.88)
+		)
+		(stroke
+			(width 0)
+			(type default)
+		)
+	)
+	(wire
+		(pts
 			(xy 186.69 106.68) (xy 186.69 107.95)
 		)
@@
 	(wire
 		(pts
-			(xy 152.4 55.88) (xy 151.13 55.88)
-		)
-		(stroke
-			(width 0)
-			(type default)
-		)
-	)
-	(wire
-		(pts
 			(xy 212.09 119.38) (xy 218.44 119.38)
 		)
@@
 	(wire
 		(pts
-			(xy 157.48 58.42) (xy 151.13 58.42)
+			(xy 157.48 58.42) (xy 156.21 58.42)
 		)
 		(stroke
@@
 	(wire
 		(pts
-			(xy 157.48 55.88) (xy 152.4 55.88)
+			(xy 157.48 55.88) (xy 156.21 55.88)
 		)
 		(stroke
@@
 	(wire
 		(pts
+			(xy 137.16 54.61) (xy 137.16 55.88)
+		)
+		(stroke
+			(width 0)
+			(type default)
+		)
+	)
+	(wire
+		(pts
 			(xy 132.08 40.64) (xy 132.08 48.26)
 		)
@@
 	(wire
 		(pts
-			(xy 152.4 40.64) (xy 152.4 41.91)
+			(xy 137.16 40.64) (xy 137.16 41.91)
 		)
 		(stroke
@@
 	(wire
 		(pts
-			(xy 129.54 55.88) (xy 138.43 55.88)
+			(xy 129.54 55.88) (xy 137.16 55.88)
 		)
 		(stroke
@@
 	(wire
 		(pts
-			(xy 132.08 40.64) (xy 152.4 40.64)
+			(xy 132.08 40.64) (xy 137.16 40.64)
 		)
 		(stroke
@@
 	(wire
 		(pts
-			(xy 152.4 54.61) (xy 152.4 55.88)
-		)
-		(stroke
-			(width 0)
-			(type default)
-		)
-	)
-	(wire
-		(pts
 			(xy 101.6 48.26) (xy 101.6 60.96)
 		)
@@
 	(wire
 		(pts
-			(xy 129.54 58.42) (xy 138.43 58.42)
+			(xy 129.54 58.42) (xy 143.51 58.42)
 		)
 		(stroke
@@
 	)
 	(label "DD-"
-		(at 135.89 58.42 0)
+		(at 139.7 58.42 0)
 		(fields_autoplaced yes)
 		(effects
@@
 	)
 	(label "DD+"
-		(at 135.89 55.88 0)
+		(at 139.7 55.88 0)
 		(fields_autoplaced yes)
 		(effects
@@
 	(symbol
 		(lib_id "Additional:R")
-		(at 144.78 58.42 270)
+		(at 149.86 58.42 270)
 		(unit 1)
 		(exclude_from_sim no)
@@
 		(dnp no)
 		(property "Reference" "R90"
-			(at 144.78 60.452 90)
+			(at 149.86 60.452 90)
 			(effects
 				(font
@@
 		)
 		(property "Value" "33"
-			(at 144.78 58.42 90)
+			(at 149.86 58.42 90)
 			(effects
 				(font
@@
 		)
 		(property "Footprint" "Resistor_SMD:R_0603_1608Metric"
-			(at 144.78 56.642 90)
+			(at 149.86 56.642 90)
 			(effects
 				(font
@@
 		)
 		(property "Datasheet" "~"
-			(at 144.78 58.42 0)
+			(at 149.86 58.42 0)
 			(effects
 				(font
@@
 		)
 		(property "Description" ""
-			(at 144.78 58.42 0)
+			(at 149.86 58.42 0)
 			(effects
 				(font
@@
 		)
 		(property "LCSC" "C23140"
-			(at 144.78 60.452 0)
+			(at 149.86 60.452 0)
 			(effects
 				(font
@@
 	(symbol
 		(lib_id "Additional:R")
-		(at 152.4 48.26 0)
+		(at 137.16 48.26 0)
 		(unit 1)
 		(exclude_from_sim no)
@@
 		(dnp no)
 		(property "Reference" "R144"
-			(at 150.368 48.26 90)
+			(at 135.128 48.26 90)
 			(effects
 				(font
@@
 		)
 		(property "Value" "1k5"
-			(at 152.4 48.26 90)
+			(at 137.16 48.26 90)
 			(effects
 				(font
@@
 		)
 		(property "Footprint" "Resistor_SMD:R_0603_1608Metric"
-			(at 150.622 48.26 90)
+			(at 135.382 48.26 90)
 			(effects
 				(font
@@
 		)
 		(property "Datasheet" "~"
-			(at 152.4 48.26 0)
+			(at 137.16 48.26 0)
 			(effects
 				(font
@@
 		)
 		(property "Description" ""
-			(at 152.4 48.26 0)
+			(at 137.16 48.26 0)
 			(effects
 				(font
@@
 		)
 		(property "LCSC" "C22843"
-			(at 154.432 48.26 0)
+			(at 139.192 48.26 0)
 			(effects
 				(font
@@
 	(symbol
 		(lib_id "Additional:R")
-		(at 144.78 55.88 270)
+		(at 149.86 55.88 270)
 		(unit 1)
 		(exclude_from_sim no)
@@
 		(dnp no)
 		(property "Reference" "R91"
-			(at 144.78 53.848 90)
+			(at 149.86 53.848 90)
 			(effects
 				(font
@@
 		)
 		(property "Value" "33"
-			(at 144.78 55.88 90)
+			(at 149.86 55.88 90)
 			(effects
 				(font
@@
 		)
 		(property "Footprint" "Resistor_SMD:R_0603_1608Metric"
-			(at 144.78 54.102 90)
+			(at 149.86 54.102 90)
 			(effects
 				(font
@@
 		)
 		(property "Datasheet" "~"
-			(at 144.78 55.88 0)
+			(at 149.86 55.88 0)
 			(effects
 				(font
@@
 		)
 		(property "Description" ""
-			(at 144.78 55.88 0)
+			(at 149.86 55.88 0)
 			(effects
 				(font
@@
 		)
 		(property "LCSC" "C23140"
-			(at 144.78 57.912 0)
+			(at 149.86 57.912 0)
 			(effects
 				(font

Commit message: hardware: updated some LCSC references
Parts:
- U20: LCSC C284149 -> C284149
Changed lines of the file:
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@@
 			)
 		)
-		(property "LCSC" " C284149"
+		(property "LCSC" "C284149"
 			(at 116.84 58.42 0)
 			(effects

Commit message: hardware: 47uF reservoir for 3V3 (properer than prev commit)
Parts:
- C26: value 10uF -> 47u; footprint Additional:CP_EIA-3216-18_Kemet-A -> Capacitor_SMD:C_1206_3216Metric; LCSC C7171 -> C96123
Changed lines of the file:
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@@
-	)
-	(symbol
-		(lib_id "Additional:CP")
-		(at 242.57 55.88 0)
-		(unit 1)
-		(exclude_from_sim no)
-		(in_bom yes)
-		(on_board yes)
-		(dnp no)
-		(property "Reference" "C26"
-			(at 243.84 53.34 0)
-			(effects
-				(font
-					(size 1.27 1.27)
-				)
-				(justify left)
-			)
-		)
-		(property "Value" "10uF"
-			(at 243.84 58.42 0)
-			(effects
-				(font
-					(size 1.27 1.27)
-				)
-				(justify left)
-			)
-		)
-		(property "Footprint" "Additional:CP_EIA-3216-18_Kemet-A"
-			(at 242.57 55.88 0)
-			(effects
-				(font
-					(size 1.524 1.524)
-				)
-				(hide yes)
-			)
-		)
-		(property "Datasheet" "~"
-			(at 242.57 55.88 0)
-			(effects
-				(font
-					(size 1.524 1.524)
-				)
-			)
-		)
-		(property "Description" ""
-			(at 242.57 55.88 0)
-			(effects
-				(font
-					(size 1.27 1.27)
-				)
-				(hide yes)
-			)
-		)
-		(property "LCSC" "C7171"
-			(at 243.84 53.34 0)
-			(effects
-				(font
-					(size 1.27 1.27)
-				)
-				(hide yes)
-			)
-		)
-		(pin "1"
-		)
-		(pin "2"
-		)
-		(instances
-			(project "overcycler3"
-				(path "/f3616c1d-a98e-4f9d-ac17-0c5545b71bc4/347aba77-50ac-4a87-997c-5d48101c82e0"
-					(reference "C26")
-					(unit 1)
-				)
-			)
-		)
 	)
 	(symbol
@@
 					(unit 1)
 				)
+			)
+		)
+	)
+	(symbol
+		(lib_id "Additional:CP")
+		(at 242.57 55.88 0)
+		(unit 1)
+		(exclude_from_sim no)
+		(in_bom yes)
+		(on_board yes)
+		(dnp no)
+		(property "Reference" "C26"
+			(at 243.84 53.34 0)
+			(effects
+				(font
+					(size 1.27 1.27)
+				)
+				(justify left)
+			)
+		)
+		(property "Value" "47u"
+			(at 243.84 58.42 0)
+			(effects
+				(font
+					(size 1.27 1.27)
+				)
+				(justify left)
+			)
+		)
+		(property "Footprint" "Capacitor_SMD:C_1206_3216Metric"
+			(at 242.57 55.88 0)
+			(effects
+				(font
+					(size 1.524 1.524)
+				)
+				(hide yes)
+			)
+		)
+		(property "Datasheet" "~"
+			(at 242.57 55.88 0)
+			(effects
+				(font
+					(size 1.524 1.524)
+				)
+			)
+		)
+		(property "Description" ""
+			(at 242.57 55.88 0)
+			(effects
+				(font
+					(size 1.27 1.27)
+				)
+				(hide yes)
+			)
+		)
+		(property "LCSC" "C96123"
+			(at 243.84 53.34 0)
+			(effects
+				(font
+					(size 1.27 1.27)
+				)
+				(hide yes)
+			)
+		)
+		(pin "1"
+		)
+		(pin "2"
+		)
+		(instances
+			(project "overcycler3"
+				(path "/f3616c1d-a98e-4f9d-ac17-0c5545b71bc4/347aba77-50ac-4a87-997c-5d48101c82e0"
+					(reference "C26")
+					(unit 1)
+				)
