File: hardware/Power_Supply.kicad_sch (KiCad schematic)
At the start: 67 parts, among them IC1 LM13700, IC2 LM13700, IC3 LM13700, J5 USB_B, SW1 POWER, U1 TL064, U19 TL064, U20 ADUM3160

Commit message: harware: changed some LCSC refs to accomodate for stock
Parts:
- PS1: LCSC C512062 -> C7465214
- PS2: LCSC C5198623 -> C5369606
Changed lines of the file:
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@@
 			)
 		)
-		(property "LCSC" "C5198623"
+		(property "LCSC" "C5369606"
 			(at 226.06 60.96 0)
 			(effects
@@
 			)
 		)
-		(property "LCSC" "C512062"
+		(property "LCSC" "C7465214"
 			(at 190.5 63.5 0)
 			(effects
