File: enclosure/PT-10 Rear/PT-10 Rear.kicad_pcb (KiCad board)
At the start: 2 copper layers, 217.9 x 52.6 mm, 0 parts

Commit message: enclosure: fixed Rear
Other:
- board text added: "MAIN OUTPUT"
- board text removed: "MAIN"
- board text removed: "OUTPUT"

Commit message: Add ADuM3160 and correct enclosure rear
- ADuM3160 added for USB isolation
- Correction of USB traces to respect 90Ω in two-layer PCBs
- Integration of Noise circuit modifications
Other:
- outline, holes or cut-outs redrawn
- board text added: "OUTPUT MAIN"
- board text removed: "MAIN OUTPUT"

Commit message: Replace "Main Output" by "Output"
- Replace "Main Output" by "Output" on Panel Rear
- Manually add Teardown
- Replace 24Ω by 33Ω on USB Isolator
Other:
- board text added: "OUTPUT"
- board text removed: "OUTPUT MAIN"
Changed lines of the file:
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@@
 		)
 	)
-	(gr_text "OUTPUT MAIN"
+	(gr_text "OUTPUT"
 		(at 75.595 92.7525 0)
 		(layer "F.SilkS")
@@
 			(justify bottom)
 		)
-		(render_cache "OUTPUT MAIN" 0
+		(render_cache "OUTPUT" 0
 			(polygon
 				(pts
-					(xy 58.810632 92.0725) (xy 55.309167 92.0725) (xy 55.309167 91.372011) (xy 56.009655 91.372011)
-					(xy 58.110143 91.372011) (xy 58.110143 89.271523) (xy 56.009655 89.271523) (xy 56.009655 91.372011)
-					(xy 55.309167 91.372011) (xy 55.309167 88.571034) (xy 58.810632 88.571034)
+					(xy 66.505258 92.0725) (xy 63.003793 92.0725) (xy 63.003793 91.372011) (xy 63.704281 91.372011)
+					(xy 65.804769 91.372011) (xy 65.804769 89.271523) (xy 63.704281 89.271523) (xy 63.704281 91.372011)
+					(xy 63.003793 91.372011) (xy 63.003793 88.571034) (xy 66.505258 88.571034)
 				)
 			)
 			(polygon
 				(pts
-					(xy 59.506236 92.0725) (xy 59.506236 88.571034) (xy 60.206724 88.571034) (xy 60.206724 91.372011)
-					(xy 62.307213 91.372011) (xy 62.307213 88.571034) (xy 63.007701 88.571034) (xy 63.007701 92.0725)
+					(xy 67.200862 92.0725) (xy 67.200862 88.571034) (xy 67.90135 88.571034) (xy 67.90135 91.372011)
+					(xy 70.001839 91.372011) (xy 70.001839 88.571034) (xy 70.702327 88.571034) (xy 70.702327 92.0725)
 				)
 			)
 			(polygon
 				(pts
-					(xy 65.07888 92.0725) (xy 65.07888 89.271523) (xy 63.703305 89.271523) (xy 63.703305 88.571034)
-					(xy 67.20477 88.571034) (xy 67.20477 89.271523) (xy 65.779369 89.271523) (xy 65.779369 92.0725)
+					(xy 72.773506 92.0725) (xy 72.773506 89.271523) (xy 71.397931 89.271523) (xy 71.397931 88.571034)
+					(xy 74.899396 88.571034) (xy 74.899396 89.271523) (xy 73.473995 89.271523) (xy 73.473995 92.0725)
 				)
 			)
 			(polygon
 				(pts
-					(xy 71.401839 90.696924) (xy 68.600862 90.696924) (xy 68.600862 92.0725) (xy 67.900374 92.0725)
-					(xy 67.900374 89.996435) (xy 68.600862 89.996435) (xy 70.701351 89.996435) (xy 70.701351 89.271523)
-					(xy 68.600862 89.271523) (xy 68.600862 89.996435) (xy 67.900374 89.996435) (xy 67.900374 88.571034)
-					(xy 71.401839 88.571034)
+					(xy 79.096465 90.696924) (xy 76.295488 90.696924) (xy 76.295488 92.0725) (xy 75.595 92.0725) (xy 75.595 89.996435)
+					(xy 76.295488 89.996435) (xy 78.395977 89.996435) (xy 78.395977 89.271523) (xy 76.295488 89.271523)
+					(xy 76.295488 89.996435) (xy 75.595 89.996435) (xy 75.595 88.571034) (xy 79.096465 88.571034)
 				)
 			)
 			(polygon
 				(pts
-					(xy 72.097443 92.0725) (xy 72.097443 88.571034) (xy 72.797931 88.571034) (xy 72.797931 91.372011)
-					(xy 74.89842 91.372011) (xy 74.89842 88.571034) (xy 75.598908 88.571034) (xy 75.598908 92.0725)
+					(xy 79.792069 92.0725) (xy 79.792069 88.571034) (xy 80.492557 88.571034) (xy 80.492557 91.372011)
+					(xy 82.593046 91.372011) (xy 82.593046 88.571034) (xy 83.293534 88.571034) (xy 83.293534 92.0725)
 				)
 			)
 			(polygon
 				(pts
-					(xy 77.670088 92.0725) (xy 77.670088 89.271523) (xy 76.294512 89.271523) (xy 76.294512 88.571034)
-					(xy 79.795977 88.571034) (xy 79.795977 89.271523) (xy 78.370576 89.271523) (xy 78.370576 92.0725)
+					(xy 85.364714 92.0725) (xy 85.364714 89.271523) (xy 83.989138 89.271523) (xy 83.989138 88.571034)
+					(xy 87.490603 88.571034) (xy 87.490603 89.271523) (xy 86.065202 89.271523) (xy 86.065202 92.0725)
 				)
 			)
-			(polygon
-				(pts
-					(xy 81.890604 92.0725) (xy 81.890604 88.571034) (xy 85.342244 88.571034) (xy 85.342244 92.0725)
-					(xy 84.641755 92.0725) (xy 84.641755 89.271523) (xy 83.966668 89.271523) (xy 83.966668 92.0725)
-					(xy 83.26618 92.0725) (xy 83.26618 89.271523) (xy 82.591093 89.271523) (xy 82.591093 92.0725)
-				)
-			)
-			(polygon
-				(pts
-					(xy 89.589139 92.0725) (xy 88.88865 92.0725) (xy 88.88865 90.696924) (xy 86.788162 90.696924) (xy 86.788162 92.0725)
-					(xy 86.087673 92.0725) (xy 86.087673 89.996435) (xy 86.788162 89.996435) (xy 88.88865 89.996435)
-					(xy 88.88865 89.271523) (xy 86.788162 89.271523) (xy 86.788162 89.996435) (xy 86.087673 89.996435)
-					(xy 86.087673 88.571034) (xy 89.589139 88.571034)
-				)
-			)
-			(polygon
-				(pts
-					(xy 90.284742 92.0725) (xy 90.284742 88.571034) (xy 90.985231 88.571034) (xy 90.985231 92.0725)
-				)
-			)
-			(polygon
-				(pts
-					(xy 91.683765 92.0725) (xy 91.683765 88.571034) (xy 95.185231 88.571034) (xy 95.185231 92.0725)
-					(xy 94.484742 92.0725) (xy 94.484742 89.271523) (xy 92.384254 89.271523) (xy 92.384254 92.0725)
-				)
-			)
